Commit message: URDF correction, code clean up and bug fixing

File: motoman_csda10f_support/urdf/arm_macro.xacro (robot description, xacro)
@@ -166,5 +166,5 @@
 		</joint>
     <joint name="${prefix}joint_tool0" type="fixed" >
-      <origin xyz="0 0 0.0" rpy="3.13 0 0"/>
+      <origin xyz="0 0 -0.057" rpy="3.13 0 0"/>
       <parent link="${prefix}link_7_t" />
       <child link="${prefix}link_tool0" />

Commit message: cleanup xacros and meshes
- switch everything to spaces
- lowercase file extensions for meshes
- correct name of tool0 link
- correct indentation levels
- remove trailing whitespace everywhere

File: motoman_csda10f_support/urdf/arm_macro.xacro (robot description, xacro)
@@ -1,174 +1,174 @@
 <?xml version="1.0" ?>
 <robot xmlns:xacro="http://ros.org/wiki/xacro">
-	<xacro:macro name="motoman_arm" params="name prefix parent *origin reflect">
-		<link name="${prefix}link_1_s">
-			<visual>
-				<origin rpy="0 0 0" xyz="0 0 0"/>
-				<geometry>
-					<mesh filename="package://motoman_csda10f_support/meshes/csda10f/visual/csda_axis_s.STL" />
-				</geometry>
-				<material name="silver">
-					<color rgba="0.8 0.8 0.8 1"/>
-				</material>
-			</visual>
-			<collision>
-				<origin rpy="0 0 0" xyz="0 0 0"/>
-				<geometry>
-					<mesh filename="package://motoman_csda10f_support/meshes/csda10f/collision/csda_axis_s.stl" />
-				</geometry>
-				<material name="yellow"/>
-			</collision>
-		</link>
-		<link name="${prefix}link_2_l">
-			<visual>
-				<origin rpy="0 0 0" xyz="0 0 0"/>
-				<geometry>
-					<mesh filename="package://motoman_csda10f_support/meshes/csda10f/visual/csda_axis_l.STL" />
-				</geometry>
-				<material name="silver"/>
-			</visual>
-			<collision>
-				<origin rpy="0 0 0" xyz="0 0 0"/>
-				<geometry>
-					<mesh filename="package://motoman_csda10f_support/meshes/csda10f/collision/csda_axis_l.stl" />
-				</geometry>
-				<material name="yellow"/>
-			</collision>
-		</link>
-		<link name="${prefix}link_3_e">
-			<visual>
-				<origin rpy="0 0 0" xyz="0 0 0"/>
-				<geometry>
-					<mesh filename="package://motoman_csda10f_support/meshes/csda10f/visual/csda_axis_e.STL" />
-				</geometry>
-				<material name="silver"/>
-			</visual>
-			<collision>
-				<origin rpy="0 0 0" xyz="0 0 0"/>
-				<geometry>
-					<mesh filename="package://motoman_csda10f_support/meshes/csda10f/collision/csda_axis_e.stl" />
-				</geometry>
-				<material name="yellow"/>
-			</collision>
-		</link>
-		<link name="${prefix}link_4_u">
-			<visual>
-				<origin rpy="0 0 0" xyz="0 0 0"/>
-				<geometry>
-					<mesh filename="package://motoman_csda10f_support/meshes/csda10f/visual/csda_axis_u.STL" />
-				</geometry>
-				<material name="silver"/>
-			</visual>
-			<collision>
-				<origin rpy="0 0 0" xyz="0 0 0"/>
-				<geometry>
-					<mesh filename="package://motoman_csda10f_support/meshes/csda10f/collision/csda_axis_u.stl" />
-				</geometry>
-				<material name="yellow"/>
-			</collision>
-		</link>
-		<link name="${prefix}link_5_r">
-			<visual>
-				<origin rpy="0 0 0" xyz="0 0 0"/>
-				<geometry>
-					<mesh filename="package://motoman_csda10f_support/meshes/csda10f/visual/csda_axis_r.STL" />
-				</geometry>
-				<material name="silver"/>
-			</visual>
-			<collision>
-				<origin rpy="0 0 0" xyz="0 0 0"/>
-				<geometry>
-					<mesh filename="package://motoman_csda10f_support/meshes/csda10f/collision/csda_axis_r.stl" />
-				</geometry>
-				<material name="yellow"/>
-			</collision>
-		</link>
-		<link name="${prefix}link_6_b">
-			<visual>
-				<origin rpy="0 0 0" xyz="0 0 0"/>
-				<geometry>
-					<mesh filename="package://motoman_csda10f_support/meshes/csda10f/visual/csda_axis_b.STL" />
-				</geometry>
-				<material name="silver"/>
-			</visual>
-			<collision>
-				<origin rpy="0 0 0" xyz="0 0 0"/>
-				<geometry>
-					<mesh filename="package://motoman_csda10f_support/meshes/csda10f/collision/csda_axis_b.stl" />
-				</geometry>
-				<material name="yellow"/>
-			</collision>
-		</link>
-		<link name="${prefix}link_7_t">
-			<visual>
-				<geometry>
-					<mesh filename="package://motoman_csda10f_support/meshes/csda10f/visual/csda_axis_t.STL" />
-				</geometry>
-				<material name="silver"/>
-			</visual>
-			<collision>
-                                <origin rpy="0 0 0" xyz="0 0 0"/>
-				<geometry>
-					<mesh filename="package://motoman_csda10f_support/meshes/csda10f/collision/csda_axis_t.stl" />
-				</geometry>
-				<material name="yellow"/>
-			</collision>
-		</link>
-	    <link name="${prefix}link_tool0" />
-		<joint name="${prefix}joint_1_s" type="revolute">
-			<parent link="torso_link_b1"/>
-			<child link="${prefix}link_1_s"/>
-			<origin xyz="0.1 ${reflect*0.023} 0.3381" rpy="1.57 0 ${(reflect-1)*1.57}"/>
-			<axis xyz="0 0 ${-reflect}" />
-			<limit lower="-2.95" upper="2.95" effort="0" velocity="2.95" />
-		</joint>
-		<joint name="${prefix}joint_2_l" type="revolute">
-			<parent link="${prefix}link_1_s"/>
-			<child link="${prefix}link_2_l"/>
-			<origin xyz="0 0.0454 -0.242" rpy="-1.57 0 0"/>
-			<axis xyz="0 0 ${-reflect}" />
-			<limit lower="-1.90" upper="1.90" effort="0" velocity="2.95" />
-		</joint>
-		<joint name="${prefix}joint_3_e" type="revolute">
-			<parent link="${prefix}link_2_l"/>
-			<child link="${prefix}link_3_e"/>
-			<origin xyz="0 0.175 -0.04540" rpy="1.57 0 0"/>
-			<axis xyz="0 0 ${-reflect}" />
-			<limit lower="-2.95" upper="2.95" effort="0" velocity="2.95" />
-		</joint>
-		<joint name="${prefix}joint_4_u" type="revolute">
-			<parent link="${prefix}link_3_e"/>
-			<child link="${prefix}link_4_u"/>
-			<origin xyz="0.00001 -0.0155 -0.185" rpy="-1.57 0 0"/>
-			<axis xyz="0 0 ${reflect}" />
-			<limit lower="-2.35" upper="2.35" effort="0" velocity="2.95" />
-		</joint>
-		<joint name="${prefix}joint_5_r" type="revolute">
-			<parent link="${prefix}link_4_u"/>
-			<child link="${prefix}link_5_r"/>
-			<origin xyz="0.00002 0.1487 0.0155" rpy="1.57 0 0"/>
-			<axis xyz="0 0 ${reflect}" />
-			<limit lower="-3.13" upper="3.13" effort="0" velocity="3.48" />
-		</joint>
-		<joint name="${prefix}joint_6_b" type="revolute">
-			<parent link="${prefix}link_5_r"/>
-			<child link="${prefix}link_6_b"/>
-			<origin xyz="0.00001 0.015 -0.2113" rpy="-1.57 0 0"/>
-			<axis xyz="0 0 ${reflect}" />
-			<limit lower="-1.90" upper="1.90" effort="0" velocity="3.48" />
-		</joint>
-		<joint name="${prefix}joint_7_t" type="revolute">
-			<parent link="${prefix}link_6_b"/>
-			<child link="${prefix}link_7_t"/>
-			<origin xyz="0 0.118 -0.015" rpy="1.57 0 0"/>
-			<axis xyz="0 0 ${reflect}" />
-			<limit lower="-3.13" upper="3.13" effort="0" velocity="6.97" />
-		</joint>
+  <xacro:macro name="motoman_arm" params="name prefix parent *origin reflect">
+    <link name="${prefix}link_1_s">
+      <visual>
+        <origin rpy="0 0 0" xyz="0 0 0"/>
+        <geometry>
+          <mesh filename="package://motoman_csda10f_support/meshes/csda10f/visual/csda_axis_s.stl" />
+        </geometry>
+        <material name="silver">
+          <color rgba="0.8 0.8 0.8 1"/>
+        </material>
+      </visual>
+      <collision>
+        <origin rpy="0 0 0" xyz="0 0 0"/>
+        <geometry>
+          <mesh filename="package://motoman_csda10f_support/meshes/csda10f/collision/csda_axis_s.stl" />
+        </geometry>
+        <material name="yellow"/>
+      </collision>
+    </link>
+    <link name="${prefix}link_2_l">
+      <visual>
+        <origin rpy="0 0 0" xyz="0 0 0"/>
+        <geometry>
+          <mesh filename="package://motoman_csda10f_support/meshes/csda10f/visual/csda_axis_l.stl" />
+        </geometry>
+        <material name="silver"/>
+      </visual>
+      <collision>
+        <origin rpy="0 0 0" xyz="0 0 0"/>
+        <geometry>
+          <mesh filename="package://motoman_csda10f_support/meshes/csda10f/collision/csda_axis_l.stl" />
+        </geometry>
+        <material name="yellow"/>
+      </collision>
+    </link>
+    <link name="${prefix}link_3_e">
+      <visual>
+        <origin rpy="0 0 0" xyz="0 0 0"/>
+        <geometry>
+          <mesh filename="package://motoman_csda10f_support/meshes/csda10f/visual/csda_axis_e.stl" />
+        </geometry>
+        <material name="silver"/>
+      </visual>
+      <collision>
+        <origin rpy="0 0 0" xyz="0 0 0"/>
+        <geometry>
+          <mesh filename="package://motoman_csda10f_support/meshes/csda10f/collision/csda_axis_e.stl" />
+        </geometry>
+        <material name="yellow"/>
+      </collision>
+    </link>
+    <link name="${prefix}link_4_u">
+      <visual>
+        <origin rpy="0 0 0" xyz="0 0 0"/>
+        <geometry>
+          <mesh filename="package://motoman_csda10f_support/meshes/csda10f/visual/csda_axis_u.stl" />
+        </geometry>
+        <material name="silver"/>
+      </visual>
+      <collision>
+        <origin rpy="0 0 0" xyz="0 0 0"/>
+        <geometry>
+          <mesh filename="package://motoman_csda10f_support/meshes/csda10f/collision/csda_axis_u.stl" />
+        </geometry>
+        <material name="yellow"/>
+      </collision>
+    </link>
+    <link name="${prefix}link_5_r">
+      <visual>
+        <origin rpy="0 0 0" xyz="0 0 0"/>
+        <geometry>
+          <mesh filename="package://motoman_csda10f_support/meshes/csda10f/visual/csda_axis_r.stl" />
+        </geometry>
+        <material name="silver"/>
+      </visual>
+      <collision>
+        <origin rpy="0 0 0" xyz="0 0 0"/>
+        <geometry>
+          <mesh filename="package://motoman_csda10f_support/meshes/csda10f/collision/csda_axis_r.stl" />
+        </geometry>
+        <material name="yellow"/>
+      </collision>
+    </link>
+    <link name="${prefix}link_6_b">
+      <visual>
+        <origin rpy="0 0 0" xyz="0 0 0"/>
+        <geometry>
+          <mesh filename="package://motoman_csda10f_support/meshes/csda10f/visual/csda_axis_b.stl" />
+        </geometry>
+        <material name="silver"/>
+      </visual>
+      <collision>
+        <origin rpy="0 0 0" xyz="0 0 0"/>
+        <geometry>
+          <mesh filename="package://motoman_csda10f_support/meshes/csda10f/collision/csda_axis_b.stl" />
+        </geometry>
+        <material name="yellow"/>
+      </collision>
+    </link>
+    <link name="${prefix}link_7_t">
+      <visual>
+        <geometry>
+          <mesh filename="package://motoman_csda10f_support/meshes/csda10f/visual/csda_axis_t.stl" />
+        </geometry>
+        <material name="silver"/>
+      </visual>
+      <collision>
+        <origin rpy="0 0 0" xyz="0 0 0"/>
+        <geometry>
+          <mesh filename="package://motoman_csda10f_support/meshes/csda10f/collision/csda_axis_t.stl" />
+        </geometry>
+        <material name="yellow"/>
+      </collision>
+    </link>
+    <link name="${prefix}tool0" />
+    <joint name="${prefix}joint_1_s" type="revolute">
+      <parent link="torso_link_b1"/>
+      <child link="${prefix}link_1_s"/>
+      <origin xyz="0.1 ${reflect*0.023} 0.3381" rpy="1.57 0 ${(reflect-1)*1.57}"/>
+      <axis xyz="0 0 ${-reflect}" />
+      <limit lower="-2.95" upper="2.95" effort="0" velocity="2.95" />
+    </joint>
+    <joint name="${prefix}joint_2_l" type="revolute">
+      <parent link="${prefix}link_1_s"/>
+      <child link="${prefix}link_2_l"/>
+      <origin xyz="0 0.0454 -0.242" rpy="-1.57 0 0"/>
+      <axis xyz="0 0 ${-reflect}" />
+      <limit lower="-1.90" upper="1.90" effort="0" velocity="2.95" />
+    </joint>
+    <joint name="${prefix}joint_3_e" type="revolute">
+      <parent link="${prefix}link_2_l"/>
+      <child link="${prefix}link_3_e"/>
+      <origin xyz="0 0.175 -0.04540" rpy="1.57 0 0"/>
+      <axis xyz="0 0 ${-reflect}" />
+      <limit lower="-2.95" upper="2.95" effort="0" velocity="2.95" />
+    </joint>
+    <joint name="${prefix}joint_4_u" type="revolute">
+      <parent link="${prefix}link_3_e"/>
+      <child link="${prefix}link_4_u"/>
+      <origin xyz="0.00001 -0.0155 -0.185" rpy="-1.57 0 0"/>
+      <axis xyz="0 0 ${reflect}" />
+      <limit lower="-2.35" upper="2.35" effort="0" velocity="2.95" />
+    </joint>
+    <joint name="${prefix}joint_5_r" type="revolute">
+      <parent link="${prefix}link_4_u"/>
+      <child link="${prefix}link_5_r"/>
+      <origin xyz="0.00002 0.1487 0.0155" rpy="1.57 0 0"/>
+      <axis xyz="0 0 ${reflect}" />
+      <limit lower="-3.13" upper="3.13" effort="0" velocity="3.48" />
+    </joint>
+    <joint name="${prefix}joint_6_b" type="revolute">
+      <parent link="${prefix}link_5_r"/>
+      <child link="${prefix}link_6_b"/>
+      <origin xyz="0.00001 0.015 -0.2113" rpy="-1.57 0 0"/>
+      <axis xyz="0 0 ${reflect}" />
+      <limit lower="-1.90" upper="1.90" effort="0" velocity="3.48" />
+    </joint>
+    <joint name="${prefix}joint_7_t" type="revolute">
+      <parent link="${prefix}link_6_b"/>
+      <child link="${prefix}link_7_t"/>
+      <origin xyz="0 0.118 -0.015" rpy="1.57 0 0"/>
+      <axis xyz="0 0 ${reflect}" />
+      <limit lower="-3.13" upper="3.13" effort="0" velocity="6.97" />
+    </joint>
     <joint name="${prefix}joint_tool0" type="fixed" >
       <origin xyz="0 0 -0.0569999" rpy="3.13 0 0"/>
       <parent link="${prefix}link_7_t" />
-      <child link="${prefix}link_tool0" />
+      <child link="${prefix}tool0" />
     </joint>
-		<!-- end of joint list -->
-	</xacro:macro>
+    <!-- end of joint list -->
+  </xacro:macro>
 </robot>

File: motoman_csda10f_support/urdf/common_torso_macro.xacro (robot description, xacro)
@@ -1,77 +1,77 @@
 <?xml version="1.0" ?>
 <robot xmlns:xacro="http://ros.org/wiki/xacro">
-	<xacro:macro name="torso" params="name prefix">
-		<!-- link list -->
-		<link name="base_link">
-			<visual>
-				<geometry>
-					<mesh filename="package://motoman_csda10f_support/meshes/csda10f/visual/csda_base.STL" />
-				</geometry>
-				<material name="blue">
-					<color rgba="0.8 0.8 0.8 1"/>
-				</material>
-			</visual>
-			<collision>
-				<geometry>
-					<mesh filename="package://motoman_csda10f_support/meshes/csda10f/collision/csda_base.stl" />
-				</geometry>
-				<material name="yellow">
-					<color rgba="0 1 1 1"/>
-				</material>
-			</collision>
-		</link>
-		<link name="${prefix}link_b1">
-			<visual>
-				<origin rpy="0 0 0" xyz="0 0 0"/>
-				<geometry>
-					<mesh filename="package://motoman_csda10f_support/meshes/csda10f/visual/csda_axis_b1.STL" />
-				</geometry>
-				<material name="silver">
-					<color rgba="0.8 0.8 0.8 1"/>
-				</material>
-			</visual>
-			<collision>
-				<origin rpy="0 0 0" xyz="0 0 0"/>
-				<geometry>
-					<mesh filename="package://motoman_csda10f_support/meshes/csda10f/collision/csda_axis_b1.stl" />
-				</geometry>
-				<material name="yellow"/>
-			</collision>
-		</link>
-		<link name="${prefix}link_b2">
-			<visual>
-				<origin rpy="0 0 0" xyz="0 0 0"/>
-				<geometry>
-					<mesh filename="package://motoman_csda10f_support/meshes/csda10f/visual/csda_axis_b1.STL" />
-				</geometry>
-				<material name="silver">
-					<color rgba="0.8 0.8 0.8 1"/>
-				</material>
-			</visual>
-			<collision>
-				<origin rpy="0 0 0" xyz="0 0 0"/>
-				<geometry>
-					<mesh filename="package://motoman_csda10f_support/meshes/csda10f/collision/csda_axis_b1.stl" />
-				</geometry>
-				<material name="yellow"/>
-			</collision>
-		</link>
-		<!-- joint list -->
-		<joint name="${prefix}joint_b1" type="revolute">
-			<parent link="base_link"/>
-			<child link="${prefix}link_b1"/>
-			<origin xyz="0.0925 0 0.8619" rpy="0 0 0"/>
-			<axis xyz="0 0 1" />
-			<limit lower="-2.9570" upper="2.9570" effort="100" velocity="2.26" />
-		</joint>
-		<joint name="${prefix}joint_b2" type="revolute">
-			<parent link="base_link"/>
-			<child link="${prefix}link_b2"/>
-			<origin xyz="0.0925 0 0.8619" rpy="0 0 0"/>
-			<axis xyz="0 0 1" />
-			<limit lower="-2.9570" upper="2.9570" effort="100" velocity="2.26" />
-			<mimic joint="${prefix}joint_b1" multiplier="1" offset="0"/>
-		</joint>
-		<!-- end of joint list -->
-	</xacro:macro>
+  <xacro:macro name="torso" params="name prefix">
+    <!-- link list -->
+    <link name="base_link">
+      <visual>
+        <geometry>
+          <mesh filename="package://motoman_csda10f_support/meshes/csda10f/visual/csda_base.stl" />
+        </geometry>
+        <material name="blue">
+          <color rgba="0.8 0.8 0.8 1"/>
+        </material>
+      </visual>
+      <collision>
+        <geometry>
+          <mesh filename="package://motoman_csda10f_support/meshes/csda10f/collision/csda_base.stl" />
+        </geometry>
+        <material name="yellow">
+          <color rgba="0 1 1 1"/>
+        </material>
+      </collision>
+    </link>
+    <link name="${prefix}link_b1">
+      <visual>
+        <origin rpy="0 0 0" xyz="0 0 0"/>
+        <geometry>
+          <mesh filename="package://motoman_csda10f_support/meshes/csda10f/visual/csda_axis_b1.stl" />
+        </geometry>
+        <material name="silver">
+          <color rgba="0.8 0.8 0.8 1"/>
+        </material>
+      </visual>
+      <collision>
+        <origin rpy="0 0 0" xyz="0 0 0"/>
+        <geometry>
+          <mesh filename="package://motoman_csda10f_support/meshes/csda10f/collision/csda_axis_b1.stl" />
+        </geometry>
+        <material name="yellow"/>
+      </collision>
+    </link>
+    <link name="${prefix}link_b2">
+      <visual>
+        <origin rpy="0 0 0" xyz="0 0 0"/>
+        <geometry>
+          <mesh filename="package://motoman_csda10f_support/meshes/csda10f/visual/csda_axis_b1.stl" />
+        </geometry>
+        <material name="silver">
+          <color rgba="0.8 0.8 0.8 1"/>
+        </material>
+      </visual>
+      <collision>
+        <origin rpy="0 0 0" xyz="0 0 0"/>
+        <geometry>
+          <mesh filename="package://motoman_csda10f_support/meshes/csda10f/collision/csda_axis_b1.stl" />
+        </geometry>
+        <material name="yellow"/>
+      </collision>
+    </link>
+    <!-- joint list -->
+    <joint name="${prefix}joint_b1" type="revolute">
+      <parent link="base_link"/>
+      <child link="${prefix}link_b1"/>
+      <origin xyz="0.0925 0 0.8619" rpy="0 0 0"/>
+      <axis xyz="0 0 1" />
+      <limit lower="-2.9570" upper="2.9570" effort="100" velocity="2.26" />
+    </joint>
+    <joint name="${prefix}joint_b2" type="revolute">
+      <parent link="base_link"/>
+      <child link="${prefix}link_b2"/>
+      <origin xyz="0.0925 0 0.8619" rpy="0 0 0"/>
+      <axis xyz="0 0 1" />
+      <limit lower="-2.9570" upper="2.9570" effort="100" velocity="2.26" />
+      <mimic joint="${prefix}joint_b1" multiplier="1" offset="0"/>
+    </joint>
+    <!-- end of joint list -->
+  </xacro:macro>
 </robot>

File: motoman_csda10f_support/urdf/csda10f.xacro (robot description, xacro)
@@ -1,5 +1,5 @@
 <?xml version="1.0" ?>
 <robot name="motoman_csda10f" xmlns:xacro="http://ros.org/wiki/xacro">
-	<xacro:include filename="$(find motoman_csda10f_support)/urdf/csda10f_macro.xacro" />
-	<xacro:motoman_csda10f prefix=""/>
+  <xacro:include filename="$(find motoman_csda10f_support)/urdf/csda10f_macro.xacro" />
+  <xacro:motoman_csda10f prefix=""/>
 </robot>

File: motoman_csda10f_support/urdf/csda10f_macro.xacro (robot description, xacro)
@@ -1,19 +1,19 @@
 <?xml version="1.0" ?>
 <robot xmlns:xacro="http://ros.org/wiki/xacro">
-        <!--Import torso and arm macros-->
-        <xacro:include filename="$(find motoman_csda10f_support)/urdf/common_torso_macro.xacro" />
-        <xacro:include filename="$(find motoman_csda10f_support)/urdf/arm_macro.xacro" />
-        <!--Robot instance-->
-        <xacro:macro name="motoman_csda10f" params="prefix">
-            <!--Torso instance-->
-            <xacro:torso name="torso" prefix="torso_"/>
-            <!--Arm instance joint parameters-->
-            <xacro:motoman_arm name="arm_left" prefix="arm_left_" parent="torso_link_b1" reflect="1">
-                <origin xyz="0.1 0.023 0.3381" rpy="1.57 0 0" />
-            </xacro:motoman_arm>
-            <!--Arm instance joint parameters-->
-            <xacro:motoman_arm name="arm_right" prefix="arm_right_" parent="torso_link_b1" reflect="-1">
-                <origin xyz="0.1 -0.023 0.3381" rpy="1.57 0 0" />
-            </xacro:motoman_arm>
-        </xacro:macro>
+  <!--Import torso and arm macros-->
+  <xacro:include filename="$(find motoman_csda10f_support)/urdf/common_torso_macro.xacro" />
+  <xacro:include filename="$(find motoman_csda10f_support)/urdf/arm_macro.xacro" />
+  <!--Robot instance-->
+  <xacro:macro name="motoman_csda10f" params="prefix">
+    <!--Torso instance-->
+    <xacro:torso name="torso" prefix="torso_"/>
+    <!--Arm instance joint parameters-->
+    <xacro:motoman_arm name="arm_left" prefix="arm_left_" parent="torso_link_b1" reflect="1">
+      <origin xyz="0.1 0.023 0.3381" rpy="1.57 0 0" />
+    </xacro:motoman_arm>
+    <!--Arm instance joint parameters-->
+    <xacro:motoman_arm name="arm_right" prefix="arm_right_" parent="torso_link_b1" reflect="-1">
+      <origin xyz="0.1 -0.023 0.3381" rpy="1.57 0 0" />
+    </xacro:motoman_arm>
+  </xacro:macro>
 </robot>
