Commit message: correct joint limits
Based on the manual.

File: motoman_csda10f_support/urdf/arm_macro.xacro (robot description, xacro)
@@ -121,5 +121,5 @@
       <origin xyz="0.1 ${reflect*0.023} 0.3381" rpy="1.57 0 ${(reflect-1)*1.57}"/>
       <axis xyz="0 0 ${-reflect}" />
-      <limit lower="-2.95" upper="2.95" effort="0" velocity="2.95" />
+      <limit lower="${radians(-170)}" upper="${radians(170)}" effort="0" velocity="${radians(130)}" />
     </joint>
     <joint name="${prefix}joint_2_l" type="revolute">
@@ -128,5 +128,5 @@
       <origin xyz="0 0.0454 -0.242" rpy="-1.57 0 0"/>
       <axis xyz="0 0 ${-reflect}" />
-      <limit lower="-1.90" upper="1.90" effort="0" velocity="2.95" />
+      <limit lower="${radians(-110)}" upper="${radians(110)}" effort="0" velocity="${radians(170)}" />
     </joint>
     <joint name="${prefix}joint_3_e" type="revolute">
@@ -135,5 +135,5 @@
       <origin xyz="0 0.175 -0.04540" rpy="1.57 0 0"/>
       <axis xyz="0 0 ${-reflect}" />
-      <limit lower="-2.95" upper="2.95" effort="0" velocity="2.95" />
+      <limit lower="${radians(-170)}" upper="${radians(170)}" effort="0" velocity="${radians(170)}" />
     </joint>
     <joint name="${prefix}joint_4_u" type="revolute">
@@ -142,5 +142,5 @@
       <origin xyz="0.00001 -0.0155 -0.185" rpy="-1.57 0 0"/>
       <axis xyz="0 0 ${reflect}" />
-      <limit lower="-2.35" upper="2.35" effort="0" velocity="2.95" />
+      <limit lower="${radians(-135)}" upper="${radians(135)}" effort="0" velocity="${radians(170)}" />
     </joint>
     <joint name="${prefix}joint_5_r" type="revolute">
@@ -149,5 +149,5 @@
       <origin xyz="0.00002 0.1487 0.0155" rpy="1.57 0 0"/>
       <axis xyz="0 0 ${reflect}" />
-      <limit lower="-3.13" upper="3.13" effort="0" velocity="3.48" />
+      <limit lower="-${radians(180)}" upper="${radians(180)}" effort="0" velocity="${radians(200)}" />
     </joint>
     <joint name="${prefix}joint_6_b" type="revolute">
@@ -156,5 +156,5 @@
       <origin xyz="0.00001 0.015 -0.2113" rpy="-1.57 0 0"/>
       <axis xyz="0 0 ${reflect}" />
-      <limit lower="-1.90" upper="1.90" effort="0" velocity="3.48" />
+      <limit lower="${radians(-110)}" upper="${radians(110)}" effort="0" velocity="${radians(200)}" />
     </joint>
     <joint name="${prefix}joint_7_t" type="revolute">
@@ -163,5 +163,5 @@
       <origin xyz="0 0.118 -0.015" rpy="1.57 0 0"/>
       <axis xyz="0 0 ${reflect}" />
-      <limit lower="-3.13" upper="3.13" effort="0" velocity="6.97" />
+      <limit lower="${radians(-180)}" upper="${radians(180)}" effort="0" velocity="${radians(400)}" />
     </joint>
     <joint name="${prefix}joint_tool0" type="fixed" >

File: motoman_csda10f_support/urdf/common_torso_macro.xacro (robot description, xacro)
@@ -63,5 +63,5 @@
       <origin xyz="0.0925 0 0.8619" rpy="0 0 0"/>
       <axis xyz="0 0 1" />
-      <limit lower="-2.9570" upper="2.9570" effort="100" velocity="2.26" />
+      <limit lower="${radians(-170)}" upper="${radians(170)}" effort="0" velocity="${radians(130)}" />
     </joint>
     <joint name="${prefix}joint_b2" type="revolute">
@@ -70,5 +70,5 @@
       <origin xyz="0.0925 0 0.8619" rpy="0 0 0"/>
       <axis xyz="0 0 1" />
-      <limit lower="-2.9570" upper="2.9570" effort="100" velocity="2.26" />
+      <limit lower="${radians(-170)}" upper="${radians(170)}" effort="0" velocity="${radians(130)}" />
       <mimic joint="${prefix}joint_b1" multiplier="1" offset="0"/>
     </joint>

Commit message: add max efforts
For the joints we have data on.

Based on https://github.com/ros-industrial/motoman/pull/646#issuecomment-3046257622.

File: motoman_csda10f_support/urdf/arm_macro.xacro (robot description, xacro)
@@ -121,5 +121,5 @@
       <origin xyz="0.1 ${reflect*0.023} 0.3381" rpy="1.57 0 ${(reflect-1)*1.57}"/>
       <axis xyz="0 0 ${-reflect}" />
-      <limit lower="${radians(-170)}" upper="${radians(170)}" effort="0" velocity="${radians(130)}" />
+      <limit lower="${radians(-170)}" upper="${radians(170)}" effort="268.36" velocity="${radians(130)}" />
     </joint>
     <joint name="${prefix}joint_2_l" type="revolute">
@@ -128,5 +128,5 @@
       <origin xyz="0 0.0454 -0.242" rpy="-1.57 0 0"/>
       <axis xyz="0 0 ${-reflect}" />
-      <limit lower="${radians(-110)}" upper="${radians(110)}" effort="0" velocity="${radians(170)}" />
+      <limit lower="${radians(-110)}" upper="${radians(110)}" effort="268.36" velocity="${radians(170)}" />
     </joint>
     <joint name="${prefix}joint_3_e" type="revolute">
@@ -135,5 +135,5 @@
       <origin xyz="0 0.175 -0.04540" rpy="1.57 0 0"/>
       <axis xyz="0 0 ${-reflect}" />
-      <limit lower="${radians(-170)}" upper="${radians(170)}" effort="0" velocity="${radians(170)}" />
+      <limit lower="${radians(-170)}" upper="${radians(170)}" effort="122.89" velocity="${radians(170)}" />
     </joint>
     <joint name="${prefix}joint_4_u" type="revolute">
@@ -142,5 +142,5 @@
       <origin xyz="0.00001 -0.0155 -0.185" rpy="-1.57 0 0"/>
       <axis xyz="0 0 ${reflect}" />
-      <limit lower="${radians(-135)}" upper="${radians(135)}" effort="0" velocity="${radians(170)}" />
+      <limit lower="${radians(-135)}" upper="${radians(135)}" effort="122.89" velocity="${radians(170)}" />
     </joint>
     <joint name="${prefix}joint_5_r" type="revolute">
@@ -149,5 +149,5 @@
       <origin xyz="0.00002 0.1487 0.0155" rpy="1.57 0 0"/>
       <axis xyz="0 0 ${reflect}" />
-      <limit lower="-${radians(180)}" upper="${radians(180)}" effort="0" velocity="${radians(200)}" />
+      <limit lower="-${radians(180)}" upper="${radians(180)}" effort="44.34" velocity="${radians(200)}" />
     </joint>
     <joint name="${prefix}joint_6_b" type="revolute">
@@ -156,5 +156,5 @@
       <origin xyz="0.00001 0.015 -0.2113" rpy="-1.57 0 0"/>
       <axis xyz="0 0 ${reflect}" />
-      <limit lower="${radians(-110)}" upper="${radians(110)}" effort="0" velocity="${radians(200)}" />
+      <limit lower="${radians(-110)}" upper="${radians(110)}" effort="44.34" velocity="${radians(200)}" />
     </joint>
     <joint name="${prefix}joint_7_t" type="revolute">
@@ -163,5 +163,5 @@
       <origin xyz="0 0.118 -0.015" rpy="1.57 0 0"/>
       <axis xyz="0 0 ${reflect}" />
-      <limit lower="${radians(-180)}" upper="${radians(180)}" effort="0" velocity="${radians(400)}" />
+      <limit lower="${radians(-180)}" upper="${radians(180)}" effort="39.04" velocity="${radians(400)}" />
     </joint>
     <joint name="${prefix}joint_tool0" type="fixed" >
