Commit message: Minor formatting corrections

File: motoman_gp25_support/urdf/gp25_20_macro.xacro (robot description, xacro)
@@ -1,5 +1,5 @@
 <?xml version="1.0" ?>
 <robot xmlns:xacro="http://ros.org/wiki/xacro">
-<xacro:macro name="motoman_gp25_20" params="prefix">
+  <xacro:macro name="motoman_gp25_20" params="prefix">
     <xacro:include filename="$(find motoman_resources)/urdf/common_materials.xacro"/>
     <!-- link list -->
@@ -161,4 +161,4 @@
         <child link="${prefix}base"/>
     </joint>
-    </xacro:macro>
+  </xacro:macro>
 </robot>
