Commit message: update references and reuse SDA10F artefacts as much as possible

File: motoman_sda10f_support/urdf/csda10f.xacro (robot description, xacro)
@@ -1,5 +1,5 @@
 <?xml version="1.0" ?>
 <robot name="motoman_csda10f" xmlns:xacro="http://ros.org/wiki/xacro">
-  <xacro:include filename="$(find motoman_csda10f_support)/urdf/csda10f_macro.xacro" />
+  <xacro:include filename="$(find motoman_sda10f_support)/urdf/csda10f_macro.xacro" />
   <xacro:motoman_csda10f prefix=""/>
 </robot>

File: motoman_sda10f_support/urdf/csda10f_arm_macro.xacro (robot description, xacro)
@@ -1,21 +1,18 @@
 <?xml version="1.0" ?>
 <robot xmlns:xacro="http://ros.org/wiki/xacro">
-  <xacro:macro name="motoman_arm" params="name prefix parent *origin reflect">
+  <xacro:macro name="csda10f_motoman_arm" params="name prefix parent *origin reflect">
     <link name="${prefix}link_1_s">
       <visual>
         <origin rpy="0 0 0" xyz="0 0 0"/>
         <geometry>
-          <mesh filename="package://motoman_csda10f_support/meshes/csda10f/visual/csda_axis_s.stl" />
+          <mesh filename="package://motoman_sda10f_support/meshes/sda10f/visual/link_s.stl"/>
         </geometry>
-        <material name="silver">
-          <color rgba="0.8 0.8 0.8 1"/>
-        </material>
+        <xacro:material_yaskawa_blue/>
       </visual>
       <collision>
         <origin rpy="0 0 0" xyz="0 0 0"/>
         <geometry>
-          <mesh filename="package://motoman_csda10f_support/meshes/csda10f/collision/csda_axis_s.stl" />
+          <mesh filename="package://motoman_sda10f_support/meshes/sda10f/collision/link_s.stl" />
         </geometry>
-        <material name="yellow"/>
       </collision>
     </link>
@@ -24,14 +21,13 @@
         <origin rpy="0 0 0" xyz="0 0 0"/>
         <geometry>
-          <mesh filename="package://motoman_csda10f_support/meshes/csda10f/visual/csda_axis_l.stl" />
+          <mesh filename="package://motoman_sda10f_support/meshes/sda10f/visual/link_l.stl"/>
         </geometry>
-        <material name="silver"/>
+        <xacro:material_yaskawa_white/>
       </visual>
       <collision>
         <origin rpy="0 0 0" xyz="0 0 0"/>
         <geometry>
-          <mesh filename="package://motoman_csda10f_support/meshes/csda10f/collision/csda_axis_l.stl" />
+          <mesh filename="package://motoman_sda10f_support/meshes/sda10f/collision/link_l.stl"/>
         </geometry>
-        <material name="yellow"/>
       </collision>
     </link>
@@ -40,14 +36,13 @@
         <origin rpy="0 0 0" xyz="0 0 0"/>
         <geometry>
-          <mesh filename="package://motoman_csda10f_support/meshes/csda10f/visual/csda_axis_e.stl" />
+          <mesh filename="package://motoman_sda10f_support/meshes/sda10f/visual/link_e.stl"/>
         </geometry>
-        <material name="silver"/>
+        <xacro:material_yaskawa_blue/>
       </visual>
       <collision>
         <origin rpy="0 0 0" xyz="0 0 0"/>
         <geometry>
-          <mesh filename="package://motoman_csda10f_support/meshes/csda10f/collision/csda_axis_e.stl" />
+          <mesh filename="package://motoman_sda10f_support/meshes/sda10f/collision/link_e.stl"/>
         </geometry>
-        <material name="yellow"/>
       </collision>
     </link>
@@ -56,14 +51,13 @@
         <origin rpy="0 0 0" xyz="0 0 0"/>
         <geometry>
-          <mesh filename="package://motoman_csda10f_support/meshes/csda10f/visual/csda_axis_u.stl" />
+          <mesh filename="package://motoman_sda10f_support/meshes/sda10f/visual/link_u.stl"/>
         </geometry>
-        <material name="silver"/>
+        <xacro:material_yaskawa_white/>
       </visual>
       <collision>
         <origin rpy="0 0 0" xyz="0 0 0"/>
         <geometry>
-          <mesh filename="package://motoman_csda10f_support/meshes/csda10f/collision/csda_axis_u.stl" />
+          <mesh filename="package://motoman_sda10f_support/meshes/sda10f/collision/link_u.stl"/>
         </geometry>
-        <material name="yellow"/>
       </collision>
     </link>
@@ -72,14 +66,13 @@
         <origin rpy="0 0 0" xyz="0 0 0"/>
         <geometry>
-          <mesh filename="package://motoman_csda10f_support/meshes/csda10f/visual/csda_axis_r.stl" />
+          <mesh filename="package://motoman_sda10f_support/meshes/sda10f/visual/link_r.stl"/>
         </geometry>
-        <material name="silver"/>
+        <xacro:material_yaskawa_blue/>
       </visual>
       <collision>
         <origin rpy="0 0 0" xyz="0 0 0"/>
         <geometry>
-          <mesh filename="package://motoman_csda10f_support/meshes/csda10f/collision/csda_axis_r.stl" />
+          <mesh filename="package://motoman_sda10f_support/meshes/sda10f/collision/link_r.stl"/>
         </geometry>
-        <material name="yellow"/>
       </collision>
     </link>
@@ -88,14 +81,13 @@
         <origin rpy="0 0 0" xyz="0 0 0"/>
         <geometry>
-          <mesh filename="package://motoman_csda10f_support/meshes/csda10f/visual/csda_axis_b.stl" />
+          <mesh filename="package://motoman_sda10f_support/meshes/sda10f/visual/link_b.stl"/>
         </geometry>
-        <material name="silver"/>
+        <xacro:material_yaskawa_white/>
       </visual>
       <collision>
         <origin rpy="0 0 0" xyz="0 0 0"/>
         <geometry>
-          <mesh filename="package://motoman_csda10f_support/meshes/csda10f/collision/csda_axis_b.stl" />
+          <mesh filename="package://motoman_sda10f_support/meshes/sda10f/collision/link_b.stl"/>
         </geometry>
-        <material name="yellow"/>
       </collision>
     </link>
@@ -103,28 +95,26 @@
       <visual>
         <geometry>
-          <mesh filename="package://motoman_csda10f_support/meshes/csda10f/visual/csda_axis_t.stl" />
+          <mesh filename="package://motoman_sda10f_support/meshes/sda10f/visual/link_t.stl" />
         </geometry>
-        <material name="silver"/>
+        <xacro:material_yaskawa_blue/>
       </visual>
       <collision>
-        <origin rpy="0 0 0" xyz="0 0 0"/>
         <geometry>
-          <mesh filename="package://motoman_csda10f_support/meshes/csda10f/collision/csda_axis_t.stl" />
+          <mesh filename="package://motoman_sda10f_support/meshes/sda10f/collision/link_t.stl" />
         </geometry>
-        <material name="yellow"/>
       </collision>
     </link>
     <link name="${prefix}tool0" />
     <joint name="${prefix}joint_1_s" type="revolute">
-      <parent link="torso_link_b1"/>
+      <parent link="${parent}"/>
       <child link="${prefix}link_1_s"/>
-      <origin xyz="0.1 ${reflect*0.023} 0.3381" rpy="1.57 0 ${(reflect-1)*1.57}"/>
+      <origin xyz="0.100 ${reflect*0.265} 0.0" rpy="${radians(90)} 0.0 ${(reflect-1)*radians(90)}"/>
       <axis xyz="0 0 ${-reflect}" />
-      <limit lower="${radians(-170)}" upper="${radians(170)}" effort="268.36" velocity="${radians(130)}" />
+      <limit lower="${radians(-170)}" upper="${radians(170)}" effort="268.36" velocity="${radians(170)}" />
     </joint>
     <joint name="${prefix}joint_2_l" type="revolute">
       <parent link="${prefix}link_1_s"/>
       <child link="${prefix}link_2_l"/>
-      <origin xyz="0 0.0454 -0.242" rpy="-1.57 0 0"/>
+      <origin xyz="0.0 0.0 0.0" rpy="${radians(-90)} 0.0 0.0"/>
       <axis xyz="0 0 ${-reflect}" />
       <limit lower="${radians(-110)}" upper="${radians(110)}" effort="268.36" velocity="${radians(170)}" />
@@ -133,5 +123,5 @@
       <parent link="${prefix}link_2_l"/>
       <child link="${prefix}link_3_e"/>
-      <origin xyz="0 0.175 -0.04540" rpy="1.57 0 0"/>
+      <origin xyz="0.0 0.360 0.0" rpy="${radians(90)} 0.0 0.0"/>
       <axis xyz="0 0 ${-reflect}" />
       <limit lower="${radians(-170)}" upper="${radians(170)}" effort="122.89" velocity="${radians(170)}" />
@@ -140,5 +130,5 @@
       <parent link="${prefix}link_3_e"/>
       <child link="${prefix}link_4_u"/>
-      <origin xyz="0.00001 -0.0155 -0.185" rpy="-1.57 0 0"/>
+      <origin xyz="0.0 0.0 0.0" rpy="${radians(-90)} 0.0 0.0"/>
       <axis xyz="0 0 ${reflect}" />
       <limit lower="${radians(-135)}" upper="${radians(135)}" effort="122.89" velocity="${radians(170)}" />
@@ -147,12 +137,12 @@
       <parent link="${prefix}link_4_u"/>
       <child link="${prefix}link_5_r"/>
-      <origin xyz="0.00002 0.1487 0.0155" rpy="1.57 0 0"/>
+      <origin xyz="0.0 0.360 0.0" rpy="${radians(90)} 0.0 0.0"/>
       <axis xyz="0 0 ${reflect}" />
-      <limit lower="-${radians(180)}" upper="${radians(180)}" effort="44.34" velocity="${radians(200)}" />
+      <limit lower="${radians(-180)}" upper="${radians(180)}" effort="44.34" velocity="${radians(200)}" />
     </joint>
     <joint name="${prefix}joint_6_b" type="revolute">
       <parent link="${prefix}link_5_r"/>
       <child link="${prefix}link_6_b"/>
-      <origin xyz="0.00001 0.015 -0.2113" rpy="-1.57 0 0"/>
+      <origin xyz="0.0 0.0 0.0" rpy="${radians(-90)} 0.0 0.0"/>
       <axis xyz="0 0 ${reflect}" />
       <limit lower="${radians(-110)}" upper="${radians(110)}" effort="44.34" velocity="${radians(200)}" />
@@ -161,12 +151,12 @@
       <parent link="${prefix}link_6_b"/>
       <child link="${prefix}link_7_t"/>
-      <origin xyz="0 0.118 -0.015" rpy="1.57 0 0"/>
-      <axis xyz="0 0 ${reflect}" />
+      <origin xyz="0.0 0.175 0.0" rpy="${radians(-90)} 0.0 0.0"/>
+      <axis xyz="0 0 ${-reflect}" />
       <limit lower="${radians(-180)}" upper="${radians(180)}" effort="39.04" velocity="${radians(400)}" />
     </joint>
     <joint name="${prefix}joint_tool0" type="fixed" >
-      <origin xyz="0 0 -0.0569999" rpy="3.13 0 0"/>
       <parent link="${prefix}link_7_t" />
       <child link="${prefix}tool0" />
+      <origin xyz="0 0 0" rpy="0 0 ${radians(180)}"/>
     </joint>
     <!-- end of joint list -->

File: motoman_sda10f_support/urdf/csda10f_macro.xacro (robot description, xacro)
@@ -1,19 +1,23 @@
 <?xml version="1.0" ?>
 <robot xmlns:xacro="http://ros.org/wiki/xacro">
-  <!--Import torso and arm macros-->
-  <xacro:include filename="$(find motoman_csda10f_support)/urdf/common_torso_macro.xacro" />
-  <xacro:include filename="$(find motoman_csda10f_support)/urdf/arm_macro.xacro" />
-  <!--Robot instance-->
+  <xacro:include filename="$(find motoman_resources)/urdf/common_materials.xacro"/>
+  <xacro:include filename="$(find motoman_sda10f_support)/urdf/common_torso_macro.xacro" />
+  <xacro:include filename="$(find motoman_sda10f_support)/urdf/csda10f_arm_macro.xacro" />
   <xacro:macro name="motoman_csda10f" params="prefix">
-    <!--Torso instance-->
-    <xacro:torso name="torso" prefix="torso_"/>
-    <!--Arm instance joint parameters-->
-    <xacro:motoman_arm name="arm_left" prefix="arm_left_" parent="torso_link_b1" reflect="1">
-      <origin xyz="0.1 0.023 0.3381" rpy="1.57 0 0" />
-    </xacro:motoman_arm>
-    <!--Arm instance joint parameters-->
-    <xacro:motoman_arm name="arm_right" prefix="arm_right_" parent="torso_link_b1" reflect="-1">
-      <origin xyz="0.1 -0.023 0.3381" rpy="1.57 0 0" />
-    </xacro:motoman_arm>
+    <xacro:torso name="${prefix}torso" prefix="${prefix}torso_"/>
+    <xacro:csda10f_motoman_arm name="${prefix}arm_left" prefix="${prefix}arm_left_" parent="${prefix}torso_link_b1" reflect="1">
+      <origin xyz="0 0 0" rpy="0 0 0" />
+    </xacro:csda10f_motoman_arm>
+    <xacro:csda10f_motoman_arm name="${prefix}arm_right" prefix="${prefix}arm_right_" parent="${prefix}torso_link_b1" reflect="-1">
+      <origin xyz="0 0 0" rpy="0 0 0" />
+    </xacro:csda10f_motoman_arm>
+    <!-- link list -->
+    <link name="${prefix}base_link" />
+    <!-- joint list -->
+    <joint name="${prefix}base_link_torso" type="fixed">
+      <parent link="${prefix}base_link"/>
+      <child link="${prefix}torso_base_link"/>
+      <origin xyz="0 0 1.2" rpy="0 0 0"/>
+    </joint>
   </xacro:macro>
 </robot>
