Commit message: change references to sda meshes

File: motoman_sda10f_support/urdf/arm_macro.xacro (robot description, xacro)
@@ -6,5 +6,5 @@
         <origin rpy="0 0 0" xyz="0 0 0"/>
         <geometry>
-          <mesh filename="package://motoman_sda10f_support/meshes/sda10f/visual/link_s.stl"/>
+          <mesh filename="package://motoman_sda10f_support/meshes/sda10f/visual/link_1.stl"/>
         </geometry>
         <xacro:material_yaskawa_blue/>
@@ -13,5 +13,5 @@
         <origin rpy="0 0 0" xyz="0 0 0"/>
         <geometry>
-          <mesh filename="package://motoman_sda10f_support/meshes/sda10f/collision/link_s.stl" />
+          <mesh filename="package://motoman_sda10f_support/meshes/sda10f/collision/link_1.stl" />
         </geometry>
       </collision>
@@ -21,5 +21,5 @@
         <origin rpy="0 0 0" xyz="0 0 0"/>
         <geometry>
-          <mesh filename="package://motoman_sda10f_support/meshes/sda10f/visual/link_l.stl"/>
+          <mesh filename="package://motoman_sda10f_support/meshes/sda10f/visual/link_2.stl"/>
         </geometry>
         <xacro:material_yaskawa_white/>
@@ -28,5 +28,5 @@
         <origin rpy="0 0 0" xyz="0 0 0"/>
         <geometry>
-          <mesh filename="package://motoman_sda10f_support/meshes/sda10f/collision/link_l.stl"/>
+          <mesh filename="package://motoman_sda10f_support/meshes/sda10f/collision/link_2.stl"/>
         </geometry>
       </collision>
@@ -36,5 +36,5 @@
         <origin rpy="0 0 0" xyz="0 0 0"/>
         <geometry>
-          <mesh filename="package://motoman_sda10f_support/meshes/sda10f/visual/link_e.stl"/>
+          <mesh filename="package://motoman_sda10f_support/meshes/sda10f/visual/link_3.stl"/>
         </geometry>
         <xacro:material_yaskawa_blue/>
@@ -43,5 +43,5 @@
         <origin rpy="0 0 0" xyz="0 0 0"/>
         <geometry>
-          <mesh filename="package://motoman_sda10f_support/meshes/sda10f/collision/link_e.stl"/>
+          <mesh filename="package://motoman_sda10f_support/meshes/sda10f/collision/link_3.stl"/>
         </geometry>
       </collision>
@@ -51,5 +51,5 @@
         <origin rpy="0 0 0" xyz="0 0 0"/>
         <geometry>
-          <mesh filename="package://motoman_sda10f_support/meshes/sda10f/visual/link_u.stl"/>
+          <mesh filename="package://motoman_sda10f_support/meshes/sda10f/visual/link_4.stl"/>
         </geometry>
         <xacro:material_yaskawa_white/>
@@ -58,5 +58,5 @@
         <origin rpy="0 0 0" xyz="0 0 0"/>
         <geometry>
-          <mesh filename="package://motoman_sda10f_support/meshes/sda10f/collision/link_u.stl"/>
+          <mesh filename="package://motoman_sda10f_support/meshes/sda10f/collision/link_4.stl"/>
         </geometry>
       </collision>
@@ -66,5 +66,5 @@
         <origin rpy="0 0 0" xyz="0 0 0"/>
         <geometry>
-          <mesh filename="package://motoman_sda10f_support/meshes/sda10f/visual/link_r.stl"/>
+          <mesh filename="package://motoman_sda10f_support/meshes/sda10f/visual/link_5.stl"/>
         </geometry>
         <xacro:material_yaskawa_blue/>
@@ -73,5 +73,5 @@
         <origin rpy="0 0 0" xyz="0 0 0"/>
         <geometry>
-          <mesh filename="package://motoman_sda10f_support/meshes/sda10f/collision/link_r.stl"/>
+          <mesh filename="package://motoman_sda10f_support/meshes/sda10f/collision/link_5.stl"/>
         </geometry>
       </collision>
@@ -81,5 +81,5 @@
         <origin rpy="0 0 0" xyz="0 0 0"/>
         <geometry>
-          <mesh filename="package://motoman_sda10f_support/meshes/sda10f/visual/link_b.stl"/>
+          <mesh filename="package://motoman_sda10f_support/meshes/sda10f/visual/link_6.stl"/>
         </geometry>
         <xacro:material_yaskawa_white/>
@@ -88,5 +88,5 @@
         <origin rpy="0 0 0" xyz="0 0 0"/>
         <geometry>
-          <mesh filename="package://motoman_sda10f_support/meshes/sda10f/collision/link_b.stl"/>
+          <mesh filename="package://motoman_sda10f_support/meshes/sda10f/collision/link_6.stl"/>
         </geometry>
       </collision>
@@ -95,5 +95,5 @@
       <visual>
         <geometry>
-          <mesh filename="package://motoman_sda10f_support/meshes/sda10f/visual/link_t.stl" />
+          <mesh filename="package://motoman_sda10f_support/meshes/sda10f/visual/link_7.stl" />
         </geometry>
         <xacro:material_yaskawa_blue/>
@@ -101,5 +101,5 @@
       <collision>
         <geometry>
-          <mesh filename="package://motoman_sda10f_support/meshes/sda10f/collision/link_t.stl" />
+          <mesh filename="package://motoman_sda10f_support/meshes/sda10f/collision/link_7.stl" />
         </geometry>
       </collision>

File: motoman_sda10f_support/urdf/common_torso_macro.xacro (robot description, xacro)
@@ -6,5 +6,5 @@
       <visual>
         <geometry>
-          <mesh filename="package://motoman_sda10f_support/meshes/sda10f/visual/base.stl" />
+          <mesh filename="package://motoman_sda10f_support/meshes/torso/visual/base_link.stl" />
         </geometry>
         <xacro:material_yaskawa_blue/>
@@ -12,5 +12,5 @@
       <collision>
         <geometry>
-          <mesh filename="package://motoman_sda10f_support/meshes/sda10f/collision/base.stl" />
+          <mesh filename="package://motoman_sda10f_support/meshes/torso/collision/base_link.stl" />
         </geometry>
       </collision>
@@ -20,5 +20,5 @@
         <origin rpy="0 0 0" xyz="0 0 0"/>
         <geometry>
-          <mesh filename="package://motoman_sda10f_support/meshes/sda10f/visual/link_b1.stl"/>
+          <mesh filename="package://motoman_sda10f_support/meshes/torso/visual/link_1.stl"/>
         </geometry>
         <xacro:material_yaskawa_white/>
@@ -27,5 +27,5 @@
         <origin rpy="0 0 0" xyz="0 0 0"/>
         <geometry>
-          <mesh filename="package://motoman_sda10f_support/meshes/sda10f/collision/link_b1.stl" />
+          <mesh filename="package://motoman_sda10f_support/meshes/torso/collision/link_1.stl" />
         </geometry>
       </collision>

File: motoman_sda10f_support/urdf/csda10f_arm_macro.xacro (robot description, xacro)
@@ -6,5 +6,5 @@
         <origin rpy="0 0 0" xyz="0 0 0"/>
         <geometry>
-          <mesh filename="package://motoman_sda10f_support/meshes/sda10f/visual/link_s.stl"/>
+          <mesh filename="package://motoman_sda10f_support/meshes/sda10f/visual/link_1.stl"/>
         </geometry>
         <xacro:material_yaskawa_blue/>
@@ -13,5 +13,5 @@
         <origin rpy="0 0 0" xyz="0 0 0"/>
         <geometry>
-          <mesh filename="package://motoman_sda10f_support/meshes/sda10f/collision/link_s.stl" />
+          <mesh filename="package://motoman_sda10f_support/meshes/sda10f/collision/link_1.stl" />
         </geometry>
       </collision>
@@ -21,5 +21,5 @@
         <origin rpy="0 0 0" xyz="0 0 0"/>
         <geometry>
-          <mesh filename="package://motoman_sda10f_support/meshes/sda10f/visual/link_l.stl"/>
+          <mesh filename="package://motoman_sda10f_support/meshes/sda10f/visual/link_2.stl"/>
         </geometry>
         <xacro:material_yaskawa_white/>
@@ -28,5 +28,5 @@
         <origin rpy="0 0 0" xyz="0 0 0"/>
         <geometry>
-          <mesh filename="package://motoman_sda10f_support/meshes/sda10f/collision/link_l.stl"/>
+          <mesh filename="package://motoman_sda10f_support/meshes/sda10f/collision/link_2.stl"/>
         </geometry>
       </collision>
@@ -36,5 +36,5 @@
         <origin rpy="0 0 0" xyz="0 0 0"/>
         <geometry>
-          <mesh filename="package://motoman_sda10f_support/meshes/sda10f/visual/link_e.stl"/>
+          <mesh filename="package://motoman_sda10f_support/meshes/sda10f/visual/link_3.stl"/>
         </geometry>
         <xacro:material_yaskawa_blue/>
@@ -43,5 +43,5 @@
         <origin rpy="0 0 0" xyz="0 0 0"/>
         <geometry>
-          <mesh filename="package://motoman_sda10f_support/meshes/sda10f/collision/link_e.stl"/>
+          <mesh filename="package://motoman_sda10f_support/meshes/sda10f/collision/link_3.stl"/>
         </geometry>
       </collision>
@@ -51,5 +51,5 @@
         <origin rpy="0 0 0" xyz="0 0 0"/>
         <geometry>
-          <mesh filename="package://motoman_sda10f_support/meshes/sda10f/visual/link_u.stl"/>
+          <mesh filename="package://motoman_sda10f_support/meshes/sda10f/visual/link_4.stl"/>
         </geometry>
         <xacro:material_yaskawa_white/>
@@ -58,5 +58,5 @@
         <origin rpy="0 0 0" xyz="0 0 0"/>
         <geometry>
-          <mesh filename="package://motoman_sda10f_support/meshes/sda10f/collision/link_u.stl"/>
+          <mesh filename="package://motoman_sda10f_support/meshes/sda10f/collision/link_4.stl"/>
         </geometry>
       </collision>
@@ -66,5 +66,5 @@
         <origin rpy="0 0 0" xyz="0 0 0"/>
         <geometry>
-          <mesh filename="package://motoman_sda10f_support/meshes/sda10f/visual/link_r.stl"/>
+          <mesh filename="package://motoman_sda10f_support/meshes/sda10f/visual/link_5.stl"/>
         </geometry>
         <xacro:material_yaskawa_blue/>
@@ -73,5 +73,5 @@
         <origin rpy="0 0 0" xyz="0 0 0"/>
         <geometry>
-          <mesh filename="package://motoman_sda10f_support/meshes/sda10f/collision/link_r.stl"/>
+          <mesh filename="package://motoman_sda10f_support/meshes/sda10f/collision/link_5.stl"/>
         </geometry>
       </collision>
@@ -81,5 +81,5 @@
         <origin rpy="0 0 0" xyz="0 0 0"/>
         <geometry>
-          <mesh filename="package://motoman_sda10f_support/meshes/sda10f/visual/link_b.stl"/>
+          <mesh filename="package://motoman_sda10f_support/meshes/sda10f/visual/link_6.stl"/>
         </geometry>
         <xacro:material_yaskawa_white/>
@@ -88,5 +88,5 @@
         <origin rpy="0 0 0" xyz="0 0 0"/>
         <geometry>
-          <mesh filename="package://motoman_sda10f_support/meshes/sda10f/collision/link_b.stl"/>
+          <mesh filename="package://motoman_sda10f_support/meshes/sda10f/collision/link_6.stl"/>
         </geometry>
       </collision>
@@ -95,5 +95,5 @@
       <visual>
         <geometry>
-          <mesh filename="package://motoman_sda10f_support/meshes/csda10f/visual/link_t.stl" />
+          <mesh filename="package://motoman_sda10f_support/meshes/csda10f/visual/link_7.stl" />
         </geometry>
         <xacro:material_yaskawa_blue/>
@@ -101,5 +101,5 @@
       <collision>
         <geometry>
-          <mesh filename="package://motoman_sda10f_support/meshes/csda10f/collision/link_t.stl" />
+          <mesh filename="package://motoman_sda10f_support/meshes/csda10f/collision/link_7.stl" />
         </geometry>
       </collision>
