Commit message: Change SDA link, joint names, and add new prefixes

File: motoman_sda10f_support/urdf/arm_macro.xacro (robot description, xacro)
@@ -2,5 +2,5 @@
 <robot xmlns:xacro="http://ros.org/wiki/xacro">
   <xacro:macro name="motoman_arm" params="name prefix parent *origin reflect">
-    <link name="${prefix}link_1_s">
+    <link name="${prefix}link_1">
       <visual>
         <origin rpy="0 0 0" xyz="0 0 0"/>
@@ -17,5 +17,5 @@
       </collision>
     </link>
-    <link name="${prefix}link_2_l">
+    <link name="${prefix}link_2">
       <visual>
         <origin rpy="0 0 0" xyz="0 0 0"/>
@@ -32,5 +32,5 @@
       </collision>
     </link>
-    <link name="${prefix}link_3_e">
+    <link name="${prefix}link_3">
       <visual>
         <origin rpy="0 0 0" xyz="0 0 0"/>
@@ -47,5 +47,5 @@
       </collision>
     </link>
-    <link name="${prefix}link_4_u">
+    <link name="${prefix}link_4">
       <visual>
         <origin rpy="0 0 0" xyz="0 0 0"/>
@@ -62,5 +62,5 @@
       </collision>
     </link>
-    <link name="${prefix}link_5_r">
+    <link name="${prefix}link_5">
       <visual>
         <origin rpy="0 0 0" xyz="0 0 0"/>
@@ -77,5 +77,5 @@
       </collision>
     </link>
-    <link name="${prefix}link_6_b">
+    <link name="${prefix}link_6">
       <visual>
         <origin rpy="0 0 0" xyz="0 0 0"/>
@@ -92,5 +92,5 @@
       </collision>
     </link>
-    <link name="${prefix}link_7_t">
+    <link name="${prefix}link_7">
       <visual>
         <geometry>
@@ -105,57 +105,57 @@
       </collision>
     </link>
-    <link name="${prefix}link_tool0" />
-    <joint name="${prefix}joint_1_s" type="revolute">
+    <link name="${prefix}tool0" />
+    <joint name="${prefix}joint_1" type="revolute">
       <parent link="${parent}"/>
-      <child link="${prefix}link_1_s"/>
+      <child link="${prefix}link_1"/>
       <origin xyz="0.100 ${reflect*0.265} 0.0" rpy="${radians(90)} 0.0 ${(reflect-1)*radians(90)}"/>
       <axis xyz="0 0 ${-reflect}" />
       <limit lower="${radians(-180)}" upper="${radians(180)}" effort="0" velocity="${radians(170)}" />
     </joint>
-    <joint name="${prefix}joint_2_l" type="revolute">
-      <parent link="${prefix}link_1_s"/>
-      <child link="${prefix}link_2_l"/>
+    <joint name="${prefix}joint_2" type="revolute">
+      <parent link="${prefix}link_1"/>
+      <child link="${prefix}link_2"/>
       <origin xyz="0.0 0.0 0.0" rpy="${radians(-90)} 0.0 0.0"/>
       <axis xyz="0 0 ${-reflect}" />
       <limit lower="${radians(-110)}" upper="${radians(110)}" effort="0" velocity="${radians(170)}" />
     </joint>
-    <joint name="${prefix}joint_3_e" type="revolute">
-      <parent link="${prefix}link_2_l"/>
-      <child link="${prefix}link_3_e"/>
+    <joint name="${prefix}joint_3" type="revolute">
+      <parent link="${prefix}link_2"/>
+      <child link="${prefix}link_3"/>
       <origin xyz="0.0 0.360 0.0" rpy="${radians(90)} 0.0 0.0"/>
       <axis xyz="0 0 ${-reflect}" />
       <limit lower="${radians(-170)}" upper="${radians(170)}" effort="0" velocity="${radians(170)}" />
     </joint>
-    <joint name="${prefix}joint_4_u" type="revolute">
-      <parent link="${prefix}link_3_e"/>
-      <child link="${prefix}link_4_u"/>
+    <joint name="${prefix}joint_4" type="revolute">
+      <parent link="${prefix}link_3"/>
+      <child link="${prefix}link_4"/>
       <origin xyz="0.0 0.0 0.0" rpy="${radians(-90)} 0.0 0.0"/>
       <axis xyz="0 0 ${reflect}" />
       <limit lower="${radians(-135)}" upper="${radians(135)}" effort="0" velocity="${radians(170)}" />
     </joint>
-    <joint name="${prefix}joint_5_r" type="revolute">
-      <parent link="${prefix}link_4_u"/>
-      <child link="${prefix}link_5_r"/>
+    <joint name="${prefix}joint_5" type="revolute">
+      <parent link="${prefix}link_4"/>
+      <child link="${prefix}link_5"/>
       <origin xyz="0.0 0.360 0.0" rpy="${radians(90)} 0.0 0.0"/>
       <axis xyz="0 0 ${reflect}" />
       <limit lower="${radians(-180)}" upper="${radians(180)}" effort="0" velocity="${radians(200)}" />
     </joint>
-    <joint name="${prefix}joint_6_b" type="revolute">
-      <parent link="${prefix}link_5_r"/>
-      <child link="${prefix}link_6_b"/>
+    <joint name="${prefix}joint_6" type="revolute">
+      <parent link="${prefix}link_5"/>
+      <child link="${prefix}link_6"/>
       <origin xyz="0.0 0.0 0.0" rpy="${radians(-90)} 0.0 0.0"/>
       <axis xyz="0 0 ${reflect}" />
       <limit lower="${radians(-110)}" upper="${radians(110)}" effort="0" velocity="${radians(200)}" />
     </joint>
-    <joint name="${prefix}joint_7_t" type="revolute">
-      <parent link="${prefix}link_6_b"/>
-      <child link="${prefix}link_7_t"/>
+    <joint name="${prefix}joint_7" type="revolute">
+      <parent link="${prefix}link_6"/>
+      <child link="${prefix}link_7"/>
       <origin xyz="0.0 0.155 0.0" rpy="${radians(-90)} 0.0 0.0"/>
       <axis xyz="0 0 ${-reflect}" />
       <limit lower="${radians(-180)}" upper="${radians(180)}" effort="0" velocity="${radians(400)}" />
     </joint>
-    <joint name="${prefix}joint_tool0" type="fixed" >
-      <parent link="${prefix}link_7_t" />
-      <child link="${prefix}link_tool0" />
+    <joint name="${prefix}joint_7-tool0" type="fixed" >
+      <parent link="${prefix}link_7" />
+      <child link="${prefix}tool0" />
       <origin xyz="0 0 0" rpy="0 0 ${radians(180)}"/>
     </joint>

File: motoman_sda10f_support/urdf/common_torso_macro.xacro (robot description, xacro)
@@ -1,7 +1,7 @@
 <?xml version="1.0" ?>
 <robot xmlns:xacro="http://ros.org/wiki/xacro">
-  <xacro:macro name="torso" params="name prefix">
+  <xacro:macro name="torso" params="name prefix left_base_prefix right_base_prefix">
     <!-- link list -->
-    <link name="${prefix}base_link">
+    <link name="${prefix}torso_base_link">
       <visual>
         <geometry>
@@ -16,5 +16,5 @@
       </collision>
     </link>
-    <link name="${prefix}link_b1">
+    <link name="${prefix}${left_base_prefix}base_link">
       <visual>
         <origin rpy="0 0 0" xyz="0 0 0"/>
@@ -31,20 +31,20 @@
       </collision>
     </link>
-    <link name="${prefix}link_b2"/>
+    <link name="${prefix}${right_base_prefix}base_link"/>
     <!-- joint list -->
-    <joint name="${prefix}joint_b1" type="revolute">
-      <parent link="${prefix}base_link"/>
-      <child link="${prefix}link_b1"/>
+    <joint name="${prefix}${left_base_prefix}joint_1" type="revolute">
+      <parent link="${prefix}torso_base_link"/>
+      <child link="${prefix}${left_base_prefix}base_link"/>
       <origin xyz="0 0 0" rpy="0 0 0"/>
       <axis xyz="0 0 1" />
       <limit lower="${radians(-170)}" upper="${radians(170)}" effort="100" velocity="${radians(130)}" />
     </joint>
-    <joint name="${prefix}joint_b2" type="revolute">
-      <parent link="${prefix}base_link"/>
-      <child link="${prefix}link_b2"/>
+    <joint name="${prefix}${right_base_prefix}joint_1" type="revolute">
+      <parent link="${prefix}torso_base_link"/>
+      <child link="${prefix}${right_base_prefix}base_link"/>
       <origin xyz="0 0 0" rpy="0 0 0"/>
       <axis xyz="0 0 1" />
       <limit lower="${radians(-170)}" upper="${radians(170)}" effort="100" velocity="${radians(130)}" />
-      <mimic joint="${prefix}joint_b1" multiplier="1" offset="0"/>
+      <mimic joint="${prefix}${left_base_prefix}joint_1" multiplier="1" offset="0"/>
     </joint>
     <!-- end of joint list -->

File: motoman_sda10f_support/urdf/csda10f_arm_macro.xacro (robot description, xacro)
@@ -2,5 +2,5 @@
 <robot xmlns:xacro="http://ros.org/wiki/xacro">
   <xacro:macro name="csda10f_motoman_arm" params="name prefix parent *origin reflect">
-    <link name="${prefix}link_1_s">
+    <link name="${prefix}link_1">
       <visual>
         <origin rpy="0 0 0" xyz="0 0 0"/>
@@ -17,5 +17,5 @@
       </collision>
     </link>
-    <link name="${prefix}link_2_l">
+    <link name="${prefix}link_2">
       <visual>
         <origin rpy="0 0 0" xyz="0 0 0"/>
@@ -32,5 +32,5 @@
       </collision>
     </link>
-    <link name="${prefix}link_3_e">
+    <link name="${prefix}link_3">
       <visual>
         <origin rpy="0 0 0" xyz="0 0 0"/>
@@ -47,5 +47,5 @@
       </collision>
     </link>
-    <link name="${prefix}link_4_u">
+    <link name="${prefix}link_4">
       <visual>
         <origin rpy="0 0 0" xyz="0 0 0"/>
@@ -62,5 +62,5 @@
       </collision>
     </link>
-    <link name="${prefix}link_5_r">
+    <link name="${prefix}link_5">
       <visual>
         <origin rpy="0 0 0" xyz="0 0 0"/>
@@ -77,5 +77,5 @@
       </collision>
     </link>
-    <link name="${prefix}link_6_b">
+    <link name="${prefix}link_6">
       <visual>
         <origin rpy="0 0 0" xyz="0 0 0"/>
@@ -92,5 +92,5 @@
       </collision>
     </link>
-    <link name="${prefix}link_7_t">
+    <link name="${prefix}link_7">
       <visual>
         <geometry>
@@ -106,55 +106,55 @@
     </link>
     <link name="${prefix}tool0" />
-    <joint name="${prefix}joint_1_s" type="revolute">
+    <joint name="${prefix}joint_1" type="revolute">
       <parent link="${parent}"/>
-      <child link="${prefix}link_1_s"/>
+      <child link="${prefix}link_1"/>
       <origin xyz="0.100 ${reflect*0.265} 0.0" rpy="${radians(90)} 0.0 ${(reflect-1)*radians(90)}"/>
       <axis xyz="0 0 ${-reflect}" />
       <limit lower="${radians(-170)}" upper="${radians(170)}" effort="268.36" velocity="${radians(170)}" />
     </joint>
-    <joint name="${prefix}joint_2_l" type="revolute">
-      <parent link="${prefix}link_1_s"/>
-      <child link="${prefix}link_2_l"/>
+    <joint name="${prefix}joint_2" type="revolute">
+      <parent link="${prefix}link_1"/>
+      <child link="${prefix}link_2"/>
       <origin xyz="0.0 0.0 0.0" rpy="${radians(-90)} 0.0 0.0"/>
       <axis xyz="0 0 ${-reflect}" />
       <limit lower="${radians(-110)}" upper="${radians(110)}" effort="268.36" velocity="${radians(170)}" />
     </joint>
-    <joint name="${prefix}joint_3_e" type="revolute">
-      <parent link="${prefix}link_2_l"/>
-      <child link="${prefix}link_3_e"/>
+    <joint name="${prefix}joint_3" type="revolute">
+      <parent link="${prefix}link_2"/>
+      <child link="${prefix}link_3"/>
       <origin xyz="0.0 0.360 0.0" rpy="${radians(90)} 0.0 0.0"/>
       <axis xyz="0 0 ${-reflect}" />
       <limit lower="${radians(-170)}" upper="${radians(170)}" effort="122.89" velocity="${radians(170)}" />
     </joint>
-    <joint name="${prefix}joint_4_u" type="revolute">
-      <parent link="${prefix}link_3_e"/>
-      <child link="${prefix}link_4_u"/>
+    <joint name="${prefix}joint_4" type="revolute">
+      <parent link="${prefix}link_3"/>
+      <child link="${prefix}link_4"/>
       <origin xyz="0.0 0.0 0.0" rpy="${radians(-90)} 0.0 0.0"/>
       <axis xyz="0 0 ${reflect}" />
       <limit lower="${radians(-135)}" upper="${radians(135)}" effort="122.89" velocity="${radians(170)}" />
     </joint>
-    <joint name="${prefix}joint_5_r" type="revolute">
-      <parent link="${prefix}link_4_u"/>
-      <child link="${prefix}link_5_r"/>
+    <joint name="${prefix}joint_5" type="revolute">
+      <parent link="${prefix}link_4"/>
+      <child link="${prefix}link_5"/>
       <origin xyz="0.0 0.360 0.0" rpy="${radians(90)} 0.0 0.0"/>
       <axis xyz="0 0 ${reflect}" />
       <limit lower="${radians(-180)}" upper="${radians(180)}" effort="44.34" velocity="${radians(200)}" />
     </joint>
-    <joint name="${prefix}joint_6_b" type="revolute">
-      <parent link="${prefix}link_5_r"/>
-      <child link="${prefix}link_6_b"/>
+    <joint name="${prefix}joint_6" type="revolute">
+      <parent link="${prefix}link_5"/>
+      <child link="${prefix}link_6"/>
       <origin xyz="0.0 0.0 0.0" rpy="${radians(-90)} 0.0 0.0"/>
       <axis xyz="0 0 ${reflect}" />
       <limit lower="${radians(-110)}" upper="${radians(110)}" effort="44.34" velocity="${radians(200)}" />
     </joint>
-    <joint name="${prefix}joint_7_t" type="revolute">
-      <parent link="${prefix}link_6_b"/>
-      <child link="${prefix}link_7_t"/>
+    <joint name="${prefix}joint_7" type="revolute">
+      <parent link="${prefix}link_6"/>
+      <child link="${prefix}link_7"/>
       <origin xyz="0.0 0.175 0.0" rpy="${radians(-90)} 0.0 0.0"/>
       <axis xyz="0 0 ${-reflect}" />
       <limit lower="${radians(-180)}" upper="${radians(180)}" effort="39.04" velocity="${radians(400)}" />
     </joint>
-    <joint name="${prefix}joint_tool0" type="fixed" >
-      <parent link="${prefix}link_7_t" />
+    <joint name="${prefix}joint_7-tool0" type="fixed" >
+      <parent link="${prefix}link_7" />
       <child link="${prefix}tool0" />
       <origin xyz="0 0 0" rpy="0 0 ${radians(180)}"/>

File: motoman_sda10f_support/urdf/sda10f_macro.xacro (robot description, xacro)
@@ -4,10 +4,10 @@
   <xacro:include filename="$(find motoman_sda10f_support)/urdf/common_torso_macro.xacro" />
   <xacro:include filename="$(find motoman_sda10f_support)/urdf/arm_macro.xacro" />
-  <xacro:macro name="motoman_sda10f" params="prefix">
-    <xacro:torso name="${prefix}torso" prefix="${prefix}torso_"/>
-    <xacro:motoman_arm name="${prefix}arm_left" prefix="${prefix}arm_left_" parent="${prefix}torso_link_b1" reflect="1">
+  <xacro:macro name="motoman_sda10f" params="prefix left_arm_prefix right_arm_prefix left_base_prefix right_base_prefix ">
+    <xacro:torso name="${prefix}torso" prefix="${prefix}"  left_base_prefix="${left_base_prefix}" right_base_prefix="${right_base_prefix}"/>
+    <xacro:motoman_arm name="${prefix}${left_arm_prefix}arm" prefix="${prefix}${left_arm_prefix}" parent="${prefix}${left_base_prefix}base_link" reflect="1">
       <origin xyz="0 0 0" rpy="0 0 0" />
     </xacro:motoman_arm>
-    <xacro:motoman_arm name="${prefix}arm_right" prefix="${prefix}arm_right_" parent="${prefix}torso_link_b1" reflect="-1">
+    <xacro:motoman_arm name="${prefix}${right_arm_prefix}arm" prefix="${prefix}${right_arm_prefix}" parent="${prefix}${right_base_prefix}base_link" reflect="-1">
       <origin xyz="0 0 0" rpy="0 0 0" />
     </xacro:motoman_arm>
@@ -15,5 +15,5 @@
     <link name="${prefix}base_link" />
     <!-- joint list -->
-    <joint name="${prefix}base_link_torso" type="fixed">
+    <joint name="${prefix}base_link_to_${prefix}torso_base_link" type="fixed">
       <parent link="${prefix}base_link"/>
       <child link="${prefix}torso_base_link"/>
