Commit message: Add base frames

File: motoman_sda10f_support/urdf/common_torso_macro.xacro (robot description, xacro)
@@ -32,4 +32,6 @@
     </link>
     <link name="${prefix}${right_base_prefix}base_link"/>
+    <link name="${prefix}${left_base_prefix}base"/>
+    <link name="${prefix}${right_base_prefix}base"/>
     <!-- joint list -->
     <joint name="${prefix}${left_base_prefix}joint_1" type="revolute">
@@ -48,4 +50,14 @@
       <mimic joint="${prefix}${left_base_prefix}joint_1" multiplier="1" offset="0"/>
     </joint>
+    <joint name="${prefix}${left_base_prefix}base_link-${prefix}${left_base_prefix}base" type="fixed">
+      <parent link="${prefix}${left_base_prefix}base_link"/>
+      <child link="${prefix}${left_base_prefix}base"/>
+      <origin xyz="0 0 0" rpy="0 0 0"/>
+    </joint>
+    <joint name="${prefix}${right_base_prefix}base_link-${prefix}${right_base_prefix}base" type="fixed">
+      <parent link="${prefix}${right_base_prefix}base_link"/>
+      <child link="${prefix}${right_base_prefix}base"/>
+      <origin xyz="0 0 0" rpy="0 0 0"/>
+    </joint>
     <!-- end of joint list -->
   </xacro:macro>
