Commit message: Remove outdated xacro

File: motoman_sda10f_support/urdf/sda10f_macro.xacro (robot description, xacro)
@@ -21,8 +21,3 @@
     </joint>
   </xacro:macro>
-  <!-- The following xacro is kept for backwards compatibility, it should not be used -->
-  <!-- see: https://github.com/ros-industrial/motoman/issues/166 -->
-  <xacro:macro name="sda10f">
-    <xacro:motoman_sda10f prefix=""/>
-  </xacro:macro>
 </robot>
