Commit message: csda10f: use model-specific mesh for link T
It's different from the base model's link T.

File: motoman_sda10f_support/urdf/csda10f_arm_macro.xacro (robot description, xacro)
@@ -95,5 +95,5 @@
       <visual>
         <geometry>
-          <mesh filename="package://motoman_sda10f_support/meshes/sda10f/visual/link_t.stl" />
+          <mesh filename="package://motoman_sda10f_support/meshes/csda10f/visual/link_t.stl" />
         </geometry>
         <xacro:material_yaskawa_blue/>
@@ -101,5 +101,5 @@
       <collision>
         <geometry>
-          <mesh filename="package://motoman_sda10f_support/meshes/sda10f/collision/link_t.stl" />
+          <mesh filename="package://motoman_sda10f_support/meshes/csda10f/collision/link_t.stl" />
         </geometry>
       </collision>

Commit message: Revert "fix csda10f joint limits"

File: motoman_sda10f_support/urdf/csda10f_arm_macro.xacro (robot description, xacro)
@@ -111,5 +111,5 @@
       <origin xyz="0.100 ${reflect*0.265} 0" rpy="${radians(90)} 0 ${(reflect-1)*radians(90)}"/>
       <axis xyz="0 0 ${-reflect}" />
-      <limit lower="${radians(-180)}" upper="${radians(180)}" effort="268.36" velocity="${radians(170)}" />
+      <limit lower="${radians(-170)}" upper="${radians(170)}" effort="268.36" velocity="${radians(170)}" />
     </joint>
     <joint name="${prefix}joint_2" type="revolute">
