Commit message: Add `flange` and `tool0` for single-arm robots and positioners

File: motoman_es_support/urdf/es165_macro.xacro (robot description, xacro)
@@ -120,5 +120,4 @@
       </collision>
     </link>
-    <link name="${prefix}tool0"/>
     <!--
       Balancer and rod are disabled as without a mimic joint they will not update
@@ -206,9 +205,4 @@
       <limit lower="${radians(-360)}" upper="${radians(360)}" effort="0" velocity="${radians(velocities['joint_6_t'])}"/>
     </joint>
-    <joint name="${prefix}joint_t-tool0" type="fixed">
-      <origin xyz="0 0 0" rpy="0 ${pi} 0"/>
-      <parent link="${prefix}link_t"/>
-      <child link="${prefix}tool0"/>
-    </joint>
     <!--
       See earlier comment about balancer and piston.
@@ -224,4 +218,18 @@
     </joint>
     -->
+    <!-- ROS-Industrial 'flange' frame: attachment point for EEF models -->
+    <link name="${prefix}flange"/>
+    <joint name="${prefix}link_t-flange" type="fixed">
+      <origin xyz="0 0 0" rpy="0 ${radians(90)} 0"/>
+      <parent link="${prefix}link_t"/>
+      <child link="${prefix}flange"/>
+    </joint>
+    <!-- ROS-Industrial 'tool0' frame: all-zeros tool frame -->
+    <link name="${prefix}tool0"/>
+    <joint name="${prefix}flange-tool0" type="fixed">
+      <origin xyz="0 0 0" rpy="${radians(180)} ${radians(-90)} 0"/>
+      <parent link="${prefix}flange"/>
+      <child link="${prefix}tool0"/>
+    </joint>
     <!-- end of joint list -->
     <!-- ROS base_link to Robot Manufacturer World Coordinates transform -->

File: motoman_es_support/urdf/es200_120_macro.xacro (robot description, xacro)
@@ -120,5 +120,4 @@
       </collision>
     </link>
-    <link name="${prefix}tool0"/>
     <!--
       Balancer and rod are disabled as without a mimic joint they will not update
@@ -204,9 +203,4 @@
       <limit lower="${radians(-360)}" upper="${radians(360)}" effort="0" velocity="${radians(velocities['joint_6_t'])}"/>
     </joint>
-    <joint name="${prefix}joint_t-tool0" type="fixed">
-      <origin xyz="0 0 0" rpy="0 ${radians(180)} 0"/>
-      <parent link="${prefix}link_t"/>
-      <child link="${prefix}tool0"/>
-    </joint>
     <!--
       See earlier comment about balancer and piston.
@@ -222,4 +216,18 @@
     </joint>
     -->
+    <!-- ROS-Industrial 'flange' frame: attachment point for EEF models -->
+    <link name="${prefix}flange"/>
+    <joint name="${prefix}joint_t-flange" type="fixed">
+      <origin xyz="0 0 0" rpy="0 ${radians(90)} 0"/>
+      <parent link="${prefix}link_t"/>
+      <child link="${prefix}flange"/>
+    </joint>
+    <!-- ROS-Industrial 'tool0' frame: all-zeros tool frame -->
+    <link name="${prefix}tool0"/>
+    <joint name="${prefix}flange-tool0" type="fixed">
+      <origin xyz="0 0 0" rpy="${radians(180)} ${radians(-90)} 0"/>
+      <parent link="${prefix}flange"/>
+      <child link="${prefix}tool0"/>
+    </joint>
     <!-- end of joint list -->
     <!-- ROS base_link to Robot Manufacturer World Coordinates transform -->

File: motoman_gp12_support/urdf/gp12_macro.xacro (robot description, xacro)
@@ -95,5 +95,4 @@
         </collision>
     </link>
-    <link name="${prefix}tool0"/>
     <!-- end of link list -->
     <!-- joint list -->
@@ -140,8 +139,17 @@
         <limit lower="-7.9412" upper="7.9412" effort="33.30" velocity="12.2143"/>
     </joint>
-    <joint name="${prefix}joint_6_t-tool0" type="fixed">
-        <origin xyz="0.100 0 0" rpy="3.1415926 -1.570796 0"/>
-        <parent link="${prefix}link_6_t"/>
-        <child link="${prefix}tool0"/>
+    <!-- ROS-Industrial 'flange' frame: attachment point for EEF models -->
+    <link name="${prefix}flange"/>
+    <joint name="${prefix}joint_6_t-flange" type="fixed">
+      <origin xyz="0.100 0 0" rpy="0 0 0"/>
+      <parent link="${prefix}link_6_t"/>
+      <child link="${prefix}flange"/>
+    </joint>
+    <!-- ROS-Industrial 'tool0' frame: all-zeros tool frame -->
+    <link name="${prefix}tool0"/>
+    <joint name="${prefix}flange-tool0" type="fixed">
+      <origin xyz="0 0 0" rpy="3.1415926 -1.570796 0"/>
+      <parent link="${prefix}flange"/>
+      <child link="${prefix}tool0"/>
     </joint>
     <!-- end of joint list -->

File: motoman_gp180_support/urdf/gp180_120_macro.xacro (robot description, xacro)
@@ -95,5 +95,4 @@
         </collision>
     </link>
-    <link name="${prefix}tool0"/>
     <!-- end of link list -->
     <!-- joint list -->
@@ -140,8 +139,17 @@
         <limit lower="${radians(-360)}" upper="${radians(360)}" effort="926.73" velocity="${radians(265)}"/>
     </joint>
-    <joint name="${prefix}joint_6_t-tool0" type="fixed">
-        <origin xyz="0 0 0" rpy="${radians(180)} ${radians(-90)} 0"/>
-        <parent link="${prefix}link_6_t"/>
-        <child link="${prefix}tool0"/>
+    <!-- ROS-Industrial 'flange' frame: attachment point for EEF models -->
+    <link name="${prefix}flange" />
+    <joint name="${prefix}joint_6_t-flange" type="fixed">
+        <origin xyz="0 0 0" rpy="0 0 0" />
+        <parent link="${prefix}link_6_t" />
+        <child link="${prefix}flange" />
+    </joint>
+    <!-- ROS-Industrial 'tool0' frame: all-zeros tool frame -->
+    <link name="${prefix}tool0" />
+    <joint name="${prefix}flange-tool0" type="fixed">
+        <origin xyz="0 0 0" rpy="${radians(180)} ${radians(-90)} 0" />
+        <parent link="${prefix}flange" />
+        <child link="${prefix}tool0" />
     </joint>
     <!-- end of joint list -->

File: motoman_gp50_support/urdf/gp50_macro.xacro (robot description, xacro)
@@ -95,5 +95,4 @@
         </collision>
     </link>
-    <link name="${prefix}tool0"/>
     <!-- end of link list -->
     <!-- joint list -->
@@ -140,8 +139,17 @@
         <limit lower="${radians(-360)}" upper="${radians(360)}" effort="375" velocity="${radians(360)}"/>
     </joint>
-    <joint name="${prefix}joint_6_t-tool0" type="fixed">
-        <origin xyz="0.175 0 0" rpy="3.1415926 -1.570796 0"/>
-        <parent link="${prefix}link_6_t"/>
-        <child link="${prefix}tool0"/>
+    <!-- ROS-Industrial 'flange' frame: attachment point for EEF models -->
+    <link name="${prefix}flange" />
+    <joint name="${prefix}joint_6_t-flange" type="fixed">
+        <origin xyz="0.175 0 0" rpy="0 0 0" />
+        <parent link="${prefix}link_6_t" />
+        <child link="${prefix}flange" />
+    </joint>
+    <!-- ROS-Industrial 'tool0' frame: all-zeros tool frame -->
+    <link name="${prefix}tool0" />
+    <joint name="${prefix}flange-tool0" type="fixed">
+        <origin xyz="0 0 0" rpy="${radians(180)} ${radians(-90)} 0" />
+        <parent link="${prefix}flange" />
+        <child link="${prefix}tool0" />
     </joint>
     <!-- end of joint list -->

File: motoman_hc10_support/urdf/hc10_macro.xacro (robot description, xacro)
@@ -95,5 +95,4 @@
       </collision>
     </link>
-    <link name="${prefix}tool0"/>
     <!-- end of link list -->
     <!-- joint list -->
@@ -140,8 +139,17 @@
       <limit lower="${radians(-180)}" upper="${radians(180)}" effort="31.36" velocity="${radians(250)}"/>
     </joint>
-    <joint name="${prefix}joint_6_t-tool0" type="fixed">
-      <origin xyz="0 0 -0.130" rpy="${pi} 0 0"/>
-      <parent link="${prefix}link_6_t"/>
-      <child link="${prefix}tool0"/>
+    <!-- ROS-Industrial 'flange' frame: attachment point for EEF models -->
+    <link name="${prefix}flange" />
+    <joint name="${prefix}joint_6_t-flange" type="fixed">
+        <origin xyz="0 0 -0.130" rpy="0 ${radians(90)} 0" />
+        <parent link="${prefix}link_6_t" />
+        <child link="${prefix}flange" />
+    </joint>
+    <!-- ROS-Industrial 'tool0' frame: all-zeros tool frame -->
+    <link name="${prefix}tool0" />
+    <joint name="${prefix}flange-tool0" type="fixed">
+        <origin xyz="0 0 0" rpy="${radians(180)} ${radians(-90)} 0" />
+        <parent link="${prefix}flange" />
+        <child link="${prefix}tool0" />
     </joint>
     <!-- end of joint list -->

File: motoman_hc10_support/urdf/hc10dt_macro.xacro (robot description, xacro)
@@ -95,5 +95,4 @@
       </collision>
     </link>
-    <link name="${prefix}tool0"/>
     <!-- end of link list -->
     <!-- joint list -->
@@ -140,7 +139,16 @@
       <limit lower="${radians(-180)}" upper="${radians(180)}" effort="31.36" velocity="${radians(250)}"/>
     </joint>
-    <joint name="${prefix}joint_6_t-tool0" type="fixed">
-      <origin xyz="0 0 -0.170" rpy="${pi} 0 0"/>
+    <!-- ROS-Industrial 'flange' frame: attachment point for EEF models -->
+    <link name="${prefix}flange"/>
+    <joint name="${prefix}joint_6_t-flange" type="fixed">
+      <origin xyz="0 0 -0.170" rpy="0 ${radians(90)} 0"/>
       <parent link="${prefix}link_6_t"/>
+      <child link="${prefix}flange"/>
+    </joint>
+    <!-- ROS-Industrial 'tool0' frame: all-zeros tool frame -->
+    <link name="${prefix}tool0"/>
+    <joint name="${prefix}flange-tool0" type="fixed">
+      <origin xyz="0 0 0" rpy="${radians(180)} ${radians(-90)} 0"/>
+      <parent link="${prefix}flange"/>
       <child link="${prefix}tool0"/>
     </joint>

File: motoman_ma2010_support/urdf/ma2010_macro.xacro (robot description, xacro)
@@ -139,4 +139,18 @@
       <limit lower="-3.6652" upper="3.6652" effort="29.6" velocity="10.6465"/>
     </joint>
+    <!-- ROS-Industrial 'flange' frame: attachment point for EEF models -->
+    <link name="${prefix}flange"/>
+    <joint name="${prefix}joint_6_t-flange" type="fixed">
+      <origin xyz="0.100 0 0" rpy="0 0 0"/>
+      <parent link="${prefix}link_6_t"/>
+      <child link="${prefix}flange"/>
+    </joint>
+    <!-- ROS-Industrial 'tool0' frame: all-zeros tool frame -->
+    <link name="${prefix}tool0"/>
+    <joint name="${prefix}flange-tool0" type="fixed">
+      <origin xyz="0 0 0" rpy="3.1415926 -1.5707963 0"/>
+      <parent link="${prefix}flange"/>
+      <child link="${prefix}tool0"/>
+    </joint>
     <!-- end of joint list -->
     <!-- ROS base_link to Robot Manufacturer World Coordinates transform -->
@@ -147,11 +161,4 @@
       <child link="${prefix}base"/>
     </joint>
-    <!-- ROS-Industrial 'tool0' frame: all-zeros tool frame -->
-    <link name="${prefix}tool0"/>
-    <joint name="${prefix}joint_6_t-tool0" type="fixed">
-      <origin xyz="0.100 0 0" rpy="0 0 0"/>
-      <parent link="${prefix}link_6_t"/>
-      <child link="${prefix}tool0"/>
-    </joint>
   </xacro:macro>
 </robot>

File: motoman_mh12_support/urdf/mh12_macro.xacro (robot description, xacro)
@@ -95,5 +95,4 @@
         </collision>
     </link>
-    <link name="${prefix}tool0"/>
     <!-- end of link list -->
     <!-- joint list -->
@@ -140,8 +139,17 @@
         <limit lower="${radians(-360)}" upper="${radians(360)}" effort="14.80" velocity="${radians(610)}"/>
     </joint>
-    <joint name="${prefix}joint_6_t-tool0" type="fixed">
-        <origin xyz="0.100 0 0" rpy="3.1415926 -1.570796 0"/>
-        <parent link="${prefix}link_6_t"/>
-        <child link="${prefix}tool0"/>
+    <!-- ROS-Industrial 'flange' frame: attachment point for EEF models -->
+    <link name="${prefix}flange"/>
+    <joint name="${prefix}joint_6_t-flange" type="fixed">
+      <origin xyz="0.100 0 0" rpy="0 0 0"/>
+      <parent link="${prefix}link_6_t"/>
+      <child link="${prefix}flange"/>
+    </joint>
+    <!-- ROS-Industrial 'tool0' frame: all-zeros tool frame -->
+    <link name="${prefix}tool0"/>
+    <joint name="${prefix}flange-tool0" type="fixed">
+      <origin xyz="0 0 0" rpy="3.1415926 -1.570796 0"/>
+      <parent link="${prefix}flange"/>
+      <child link="${prefix}tool0"/>
     </joint>
     <!-- end of joint list -->

File: motoman_mh50_support/urdf/mh50_macro.xacro (robot description, xacro)
@@ -95,5 +95,4 @@
         </collision>
     </link>
-    <link name="${prefix}tool0"/>
     <!-- end of link list -->
     <!-- joint list -->
@@ -140,8 +139,17 @@
         <limit lower="-6.2831" upper="6.2831" effort="333.43" velocity="6.283"/>
     </joint>
-    <joint name="${prefix}joint_6_t-tool0" type="fixed">
-        <origin xyz="0.175 0 0" rpy="3.1415926 -1.570796 0"/>
-        <parent link="${prefix}link_6_t"/>
-        <child link="${prefix}tool0"/>
+    <!-- ROS-Industrial 'flange' frame: attachment point for EEF models -->
+    <link name="${prefix}flange"/>
+    <joint name="${prefix}joint_6_t-flange" type="fixed">
+      <origin xyz="0.175 0 0" rpy="0 0 0"/>
+      <parent link="${prefix}link_6_t"/>
+      <child link="${prefix}flange"/>
+    </joint>
+    <!-- ROS-Industrial 'tool0' frame: all-zeros tool frame -->
+    <link name="${prefix}tool0"/>
+    <joint name="${prefix}flange-tool0" type="fixed">
+      <origin xyz="0 0 0" rpy="3.1415926 -1.570796 0"/>
+      <parent link="${prefix}flange"/>
+      <child link="${prefix}tool0"/>
     </joint>
     <!-- end of joint list -->

File: motoman_motomini_support/urdf/motomini_macro.xacro (robot description, xacro)
@@ -95,5 +95,4 @@
     </collision>
   </link>
-  <link name="${prefix}tool0"/>
   <!-- end of link list -->
   <!-- joint list -->
@@ -140,9 +139,18 @@
     <limit lower="-6.2831" upper="6.2831" effort="0.07" velocity="10.4719"/>
   </joint>
-  <joint name="${prefix}joint_6_t-tool0" type="fixed">
-    <origin xyz="0 0 -0.040 " rpy="${pi} 0 0"/>
-    <parent link="${prefix}link_6_t"/>
-    <child link="${prefix}tool0"/>
-  </joint>
+  <!-- ROS-Industrial 'flange' frame: attachment point for EEF models -->
+    <link name="${prefix}flange"/>
+    <joint name="${prefix}joint_6_t-flange" type="fixed">
+      <origin xyz="0 0 -0.040" rpy="0 ${pi/2} 0"/>
+      <parent link="${prefix}link_6_t"/>
+      <child link="${prefix}flange"/>
+    </joint>
+    <!-- ROS-Industrial 'tool0' frame: all-zeros tool frame -->
+    <link name="${prefix}tool0"/>
+    <joint name="${prefix}flange-tool0" type="fixed">
+      <origin xyz="0 0 0 " rpy="${pi} ${-pi/2} 0"/>
+      <parent link="${prefix}flange"/>
+      <child link="${prefix}tool0"/>
+    </joint>
   <!-- end of joint list -->
   <!-- ROS base_link to Robot Manufacturer World Coordinates transform -->

File: motoman_motopos_d500_support/urdf/motopos_d500_macro.xacro (robot description, xacro)
@@ -68,8 +68,14 @@
     </joint>
     <!-- ROS-Industrial 'tool0' frame: all-zeros tool frame -->
+    <link name="${prefix}flange"/>
+    <joint name="${prefix}joint_2-flange" type="fixed">
+      <origin xyz="0 0 0.150 " rpy="0 -1.57079632679 0"/>
+      <parent link="${prefix}link_2"/>
+      <child link="${prefix}flange"/>
+    </joint>
     <link name="${prefix}tool0"/>
-    <joint name="${prefix}joint_2-tool0" type="fixed">
-      <origin xyz="0 0 0.150 " rpy="0 0 0"/>
-      <parent link="${prefix}link_2"/>
+    <joint name="${prefix}flange-tool0" type="fixed">
+      <origin xyz="0 0 0 " rpy="0 -1.57079632679 3.14159265359"/>
+      <parent link="${prefix}flange"/>
       <child link="${prefix}tool0"/>
     </joint>

File: motoman_ms210_support/urdf/ms210_macro.xacro (robot description, xacro)
@@ -153,4 +153,18 @@
     <limit lower="${radians(-210)}" upper="${radians(210)}" effort="1800.5" velocity="${radians(220)}" />
   </joint>
+  <!-- ROS-Industrial 'flange' frame: attachment point for EEF models -->
+  <link name="${prefix}flange"/>
+  <joint name="${prefix}joint_6_t-flange" type="fixed">
+    <origin xyz="0 0 0" rpy="0 0 0"/>
+    <parent link="${prefix}link_6_t"/>
+    <child link="${prefix}flange"/>
+  </joint>
+  <!-- ROS-Industrial 'tool0' frame: all-zeros tool frame -->
+  <link name="${prefix}tool0"/>
+  <joint name="${prefix}flange-tool0" type="fixed">
+    <origin xyz="0 0 0 " rpy="${radians(180)} ${radians(-90)} 0"/>
+    <parent link="${prefix}flange"/>
+    <child link="${prefix}tool0"/>
+  </joint>
   <!-- end of joint list -->
   <!-- ROS base_link to Robot Manufacturer World Coordinates transform -->
@@ -161,11 +175,4 @@
     <child link="${prefix}base"/>
   </joint>
-    <!-- ROS-Industrial 'tool0' frame: all-zeros tool frame -->
-  <link name="${prefix}tool0"/>
-  <joint name="${prefix}joint_6_t-tool0" type="fixed">
-    <parent link="${prefix}link_6_t"/>
-    <child link="${prefix}tool0"/>
-    <origin xyz="0 0 0 " rpy="${radians(180)} ${radians(-90)} 0"/>
-  </joint>
 </xacro:macro>
 </robot>

File: motoman_sia10d_support/urdf/sia10d_macro.xacro (robot description, xacro)
@@ -263,4 +263,18 @@
             <axis xyz="0 0 -1" />
             <limit lower="-3.1415" upper="3.1415" effort="100" velocity="6.9813" />
+        </joint>
+        <!-- ROS-Industrial 'flange' frame: attachment point for EEF models -->
+        <link name="${prefix}flange"/>
+        <joint name="${prefix}joint_t-flange" type="fixed">
+            <origin xyz="0 0 0" rpy="0 -1.57079632679 0"/>
+            <parent link="${prefix}link_t"/>
+            <child link="${prefix}flange"/>
+        </joint>
+        <!-- ROS-Industrial 'tool0' frame: all-zeros tool frame -->
+        <link name="${prefix}tool0"/>
+        <joint name="${prefix}flange-tool0" type="fixed">
+            <origin xyz="0 0 0 " rpy="0 -1.57079632679 3.1415296"/>
+            <parent link="${prefix}flange"/>
+            <child link="${prefix}tool0"/>
         </joint>
         <!-- end of joint list -->

File: motoman_sia10f_support/urdf/sia10f_macro.xacro (robot description, xacro)
@@ -128,5 +128,4 @@
             </collision>
         </link>
-        <link name="${prefix}link_tool0" />
         <!-- end of link list -->
         <!-- joint list -->
@@ -180,9 +179,18 @@
             <limit lower="-3.1415" upper="3.1415" effort="0" velocity="6.9813" />
         </joint>
-    <joint name="${prefix}joint_tool0" type="fixed" >
-      <origin xyz="0 0 0.0" rpy="0 0 -3.1415926535"/>
-      <parent link="${prefix}link_7_t" />
-      <child link="${prefix}link_tool0" />
-    </joint>
+        <!-- ROS-Industrial 'flange' frame: attachment point for EEF models -->
+        <link name="${prefix}flange"/>
+        <joint name="${prefix}joint_7_t-flange" type="fixed">
+            <origin xyz="0 0 0" rpy="0 -1.57079632679 0"/>
+            <parent link="${prefix}link_7_t"/>
+            <child link="${prefix}flange"/>
+        </joint>
+        <!-- ROS-Industrial 'tool0' frame: all-zeros tool frame -->
+        <link name="${prefix}tool0"/>
+        <joint name="${prefix}flange-tool0" type="fixed">
+            <origin xyz="0 0 0 " rpy="0 -1.57079632679 3.1415296"/>
+            <parent link="${prefix}flange"/>
+            <child link="${prefix}tool0"/>
+        </joint>
         <!-- end of joint list -->
         <!-- ROS base_link (via base_link) to Motoman Robot (not Base) Frame transform -->

File: motoman_sia20d_support/urdf/sia20d_macro.xacro (robot description, xacro)
@@ -128,5 +128,4 @@
             </collision>
         </link>
-    <link name="${prefix}tool0" />
         <!-- end of link list -->
         <!-- joint list -->
@@ -180,9 +179,18 @@
             <limit lower="-3.1415" upper="3.1415" effort="100" velocity="6.9813" />
         </joint>
-    <joint name="${prefix}link_t-tool0" type="fixed" >
-      <origin xyz="0 0 0.0" rpy="0 0 -3.1415926535"/>
-      <parent link="${prefix}link_t" />
-      <child link="${prefix}tool0" />
-    </joint>
+    <!-- ROS-Industrial 'flange' frame: attachment point for EEF models -->
+        <link name="${prefix}flange"/>
+        <joint name="${prefix}link_t-flange" type="fixed">
+            <origin xyz="0 0 0" rpy="0 -1.57079632679 0"/>
+            <parent link="${prefix}link_t"/>
+            <child link="${prefix}flange"/>
+        </joint>
+        <!-- ROS-Industrial 'tool0' frame: all-zeros tool frame -->
+        <link name="${prefix}tool0"/>
+        <joint name="${prefix}flange-tool0" type="fixed">
+            <origin xyz="0 0 0 " rpy="0 -1.57079632679 3.1415296"/>
+            <parent link="${prefix}flange"/>
+            <child link="${prefix}tool0"/>
+        </joint>
         <!-- end of joint list -->
         <!-- ROS base_link (via base_link) to Motoman Robot (not Base) Frame transform -->

File: motoman_sia30d_support/urdf/sia30d_macro.xacro (robot description, xacro)
@@ -159,4 +159,18 @@
       <limit lower="${radians(-180)}" upper="${radians(180)}" effort="77" velocity="${radians(200)}"/>
     </joint>
+    <!-- ROS-Industrial 'flange' frame: attachment point for EEF models -->
+    <link name="${prefix}flange"/>
+    <joint name="${prefix}joint_7_t-flange" type="fixed">
+        <origin xyz="0 0 0.217" rpy="0 ${radians(-90)} 0"/>
+        <parent link="${prefix}link_7_t"/>
+        <child link="${prefix}flange"/>
+    </joint>
+    <!-- ROS-Industrial 'tool0' frame: all-zeros tool frame -->
+    <link name="${prefix}tool0"/>
+    <joint name="${prefix}flange-tool0" type="fixed">
+        <origin xyz="0 0 0 " rpy="0 ${radians(-90)} ${radians(180)}"/>
+        <parent link="${prefix}flange"/>
+        <child link="${prefix}tool0"/>
+    </joint>
     <!-- end of joint list -->
     <!-- ROS base_link to Robot Manufacturer World Coordinates transform -->
@@ -167,11 +181,4 @@
       <child link="${prefix}base"/>
     </joint>
-    <!-- ROS-Industrial 'tool0' frame: all-zeros tool frame -->
-    <link name="${prefix}tool0" />
-    <joint name="${prefix}link_7_t-tool0" type="fixed">
-      <origin xyz="0 0 0.217" rpy="0 0 ${pi}"/>
-      <parent link="${prefix}link_7_t" />
-      <child link="${prefix}tool0" />
-    </joint>
   </xacro:macro>
 </robot>

File: motoman_sia50_support/urdf/sia50_macro.xacro (robot description, xacro)
@@ -128,5 +128,4 @@
       </collision>
     </link>
-    <link name="${prefix}tool0" />
     <!-- end of link list -->
     <!-- joint list -->
@@ -180,8 +179,17 @@
       <limit lower="${radians(-180)}" upper="${radians(180)}" effort="255.76" velocity="${radians(200)}" />
     </joint>
-    <joint name="${prefix}link_t-tool0" type="fixed">
-      <origin xyz="0 0 0.0" rpy="0 0 ${radians(-180)}"/>
-      <parent link="${prefix}link_t" />
-      <child link="${prefix}tool0" />
+    <!-- ROS-Industrial 'flange' frame: attachment point for EEF models -->
+    <link name="${prefix}flange"/>
+    <joint name="${prefix}joint_t-flange" type="fixed">
+        <origin xyz="0 0 0" rpy="0 0 0"/>
+        <parent link="${prefix}link_t"/>
+        <child link="${prefix}flange"/>
+    </joint>
+    <!-- ROS-Industrial 'tool0' frame: all-zeros tool frame -->
+    <link name="${prefix}tool0"/>
+    <joint name="${prefix}flange-tool0" type="fixed">
+        <origin xyz="0 0 0 " rpy="${radians(180)} ${radians(-90)} 0"/>
+        <parent link="${prefix}flange"/>
+        <child link="${prefix}tool0"/>
     </joint>
     <!-- end of joint list -->
