Commit message: Add `flange` and `tool0` for single-arm robots and positioners

File: motoman_sia5d_support/urdf/sia5d_macro.xacro (robot description, xacro)
@@ -165,9 +165,17 @@
     <limit lower="${-90*deg}" upper="${90*deg}" effort="0" velocity="${350*deg}" />
   </joint>
-  <link name="${prefix}tool0" />
-  <joint name="${prefix}link_t-tool0" type="fixed" >
-    <origin xyz="0.011 0 0" rpy="${-90*deg} ${-90*deg} ${-90*deg}"/>
-    <parent link="${prefix}link_t" />
-    <child link="${prefix}tool0" />
+  <!-- ROS-Industrial 'flange' frame: attachment point for EEF models -->
+  <link name="${prefix}flange"/>
+  <joint name="${prefix}joint_t-flange" type="fixed">
+    <origin xyz="0.011 0 0" rpy="0 0 0"/>
+    <parent link="${prefix}link_t"/>
+    <child link="${prefix}flange"/>
+  </joint>
+  <!-- ROS-Industrial 'tool0' frame: all-zeros tool frame -->
+  <link name="${prefix}tool0"/>
+  <joint name="${prefix}flange-tool0" type="fixed">
+    <origin xyz="0 0 0 " rpy="${180*deg} ${-90*deg} 0"/>
+    <parent link="${prefix}flange"/>
+    <child link="${prefix}tool0"/>
   </joint>
     <!-- ROS base_link (via base_link) to Motoman Robot (not Base) Frame transform -->

Commit message: Standardize formatting of fixed transforms

File: motoman_es_support/urdf/es165_macro.xacro (robot description, xacro)
@@ -218,18 +218,4 @@
     </joint>
     -->
-    <!-- ROS-Industrial 'flange' frame: attachment point for EEF models -->
-    <link name="${prefix}flange"/>
-    <joint name="${prefix}link_t-flange" type="fixed">
-      <origin xyz="0 0 0" rpy="0 ${radians(90)} 0"/>
-      <parent link="${prefix}link_t"/>
-      <child link="${prefix}flange"/>
-    </joint>
-    <!-- ROS-Industrial 'tool0' frame: all-zeros tool frame -->
-    <link name="${prefix}tool0"/>
-    <joint name="${prefix}flange-tool0" type="fixed">
-      <origin xyz="0 0 0" rpy="${radians(180)} ${radians(-90)} 0"/>
-      <parent link="${prefix}flange"/>
-      <child link="${prefix}tool0"/>
-    </joint>
     <!-- end of joint list -->
     <!-- ROS base_link to Robot Manufacturer World Coordinates transform -->
@@ -240,4 +226,18 @@
       <child link="${prefix}base"/>
     </joint>
+    <!-- ROS-Industrial 'flange' frame: attachment point for EEF models -->
+    <link name="${prefix}flange"/>
+    <joint name="${prefix}link_t-flange" type="fixed">
+      <origin xyz="0 0 0" rpy="0 ${radians(90)} 0"/>
+      <parent link="${prefix}link_t"/>
+      <child link="${prefix}flange"/>
+    </joint>
+    <!-- ROS-Industrial 'tool0' frame: all-zeros tool frame -->
+    <link name="${prefix}tool0"/>
+    <joint name="${prefix}flange-tool0" type="fixed">
+      <origin xyz="0 0 0" rpy="${radians(180)} ${radians(-90)} 0"/>
+      <parent link="${prefix}flange"/>
+      <child link="${prefix}tool0"/>
+    </joint>
   </xacro:macro>
 </robot>

File: motoman_es_support/urdf/es200_120_macro.xacro (robot description, xacro)
@@ -216,18 +216,4 @@
     </joint>
     -->
-    <!-- ROS-Industrial 'flange' frame: attachment point for EEF models -->
-    <link name="${prefix}flange"/>
-    <joint name="${prefix}joint_t-flange" type="fixed">
-      <origin xyz="0 0 0" rpy="0 ${radians(90)} 0"/>
-      <parent link="${prefix}link_t"/>
-      <child link="${prefix}flange"/>
-    </joint>
-    <!-- ROS-Industrial 'tool0' frame: all-zeros tool frame -->
-    <link name="${prefix}tool0"/>
-    <joint name="${prefix}flange-tool0" type="fixed">
-      <origin xyz="0 0 0" rpy="${radians(180)} ${radians(-90)} 0"/>
-      <parent link="${prefix}flange"/>
-      <child link="${prefix}tool0"/>
-    </joint>
     <!-- end of joint list -->
     <!-- ROS base_link to Robot Manufacturer World Coordinates transform -->
@@ -238,4 +224,18 @@
       <child link="${prefix}base"/>
     </joint>
+    <!-- ROS-Industrial 'flange' frame: attachment point for EEF models -->
+    <link name="${prefix}flange"/>
+    <joint name="${prefix}joint_t-flange" type="fixed">
+      <origin xyz="0 0 0" rpy="0 ${radians(90)} 0"/>
+      <parent link="${prefix}link_t"/>
+      <child link="${prefix}flange"/>
+    </joint>
+    <!-- ROS-Industrial 'tool0' frame: all-zeros tool frame -->
+    <link name="${prefix}tool0"/>
+    <joint name="${prefix}flange-tool0" type="fixed">
+      <origin xyz="0 0 0" rpy="${radians(180)} ${radians(-90)} 0"/>
+      <parent link="${prefix}flange"/>
+      <child link="${prefix}tool0"/>
+    </joint>
   </xacro:macro>
 </robot>

File: motoman_gp110_support/urdf/gp110_macro.xacro (robot description, xacro)
@@ -140,4 +140,11 @@
     </joint>
     <!-- end of joint list -->
+    <!-- ROS base_link to Robot Manufacturer World Coordinates transform -->
+    <link name="${prefix}base" />
+    <joint name="${prefix}base_link-base" type="fixed">
+      <origin xyz="0 0 0.540" rpy="0 0 0"/>
+      <parent link="${prefix}base_link"/>
+      <child link="${prefix}base"/>
+    </joint>
     <!-- ROS-Industrial 'flange' frame: attachment point for EEF models -->
     <link name="${prefix}flange"/>
@@ -154,11 +161,4 @@
       <child link="${prefix}tool0"/>
     </joint>
-    <!-- ROS base_link to Robot Manufacturer World Coordinates transform -->
-    <link name="${prefix}base" />
-    <joint name="${prefix}base_link-base" type="fixed">
-      <origin xyz="0 0 0.540" rpy="0 0 0"/>
-      <parent link="${prefix}base_link"/>
-      <child link="${prefix}base"/>
-    </joint>
   </xacro:macro>
 </robot>

File: motoman_gp12_support/urdf/gp12_macro.xacro (robot description, xacro)
@@ -139,4 +139,12 @@
         <limit lower="-7.9412" upper="7.9412" effort="33.30" velocity="12.2143"/>
     </joint>
+    <!-- end of joint list -->
+    <!-- ROS base_link to Robot Manufacturer World Coordinates transform -->
+    <link name="${prefix}base" />
+    <joint name="${prefix}base_link-base" type="fixed">
+        <origin xyz="0 0 0.450" rpy="0 0 0"/>
+        <parent link="${prefix}base_link"/>
+        <child link="${prefix}base"/>
+    </joint>
     <!-- ROS-Industrial 'flange' frame: attachment point for EEF models -->
     <link name="${prefix}flange"/>
@@ -153,12 +161,4 @@
       <child link="${prefix}tool0"/>
     </joint>
-    <!-- end of joint list -->
-    <!-- ROS base_link to Robot Manufacturer World Coordinates transform -->
-    <link name="${prefix}base" />
-    <joint name="${prefix}base_link-base" type="fixed">
-        <origin xyz="0 0 0.450" rpy="0 0 0"/>
-        <parent link="${prefix}base_link"/>
-        <child link="${prefix}base"/>
-    </joint>
     </xacro:macro>
 </robot>

File: motoman_gp180_support/urdf/gp180_120_macro.xacro (robot description, xacro)
@@ -139,4 +139,12 @@
         <limit lower="${radians(-360)}" upper="${radians(360)}" effort="926.73" velocity="${radians(265)}"/>
     </joint>
+    <!-- end of joint list -->
+    <!-- ROS base_link to Robot Manufacturer World Coordinates transform -->
+    <link name="${prefix}base" />
+    <joint name="${prefix}base_link-base" type="fixed">
+        <origin xyz="0 0 0.650" rpy="0 0 0"/>
+        <parent link="${prefix}base_link"/>
+        <child link="${prefix}base"/>
+    </joint>
     <!-- ROS-Industrial 'flange' frame: attachment point for EEF models -->
     <link name="${prefix}flange" />
@@ -153,12 +161,4 @@
         <child link="${prefix}tool0" />
     </joint>
-    <!-- end of joint list -->
-    <!-- ROS base_link to Robot Manufacturer World Coordinates transform -->
-    <link name="${prefix}base" />
-    <joint name="${prefix}base_link-base" type="fixed">
-        <origin xyz="0 0 0.650" rpy="0 0 0"/>
-        <parent link="${prefix}base_link"/>
-        <child link="${prefix}base"/>
-    </joint>
 </xacro:macro>
 </robot>

File: motoman_gp20hl_support/urdf/gp20hl_macro.xacro (robot description, xacro)
@@ -140,4 +140,11 @@
     </joint>
     <!-- end of joint list -->
+    <!-- ROS base_link to Robot Manufacturer World Coordinates transform -->
+    <link name="${prefix}base" />
+    <joint name="${prefix}base_link-base" type="fixed">
+      <origin xyz="0 0 0.540" rpy="0 0 0"/>
+      <parent link="${prefix}base_link"/>
+      <child link="${prefix}base"/>
+    </joint>
     <!-- ROS-Industrial 'flange' frame: attachment point for EEF models -->
     <link name="${prefix}flange"/>
@@ -154,11 +161,4 @@
       <child link="${prefix}tool0"/>
     </joint>
-    <!-- ROS base_link to Robot Manufacturer World Coordinates transform -->
-    <link name="${prefix}base" />
-    <joint name="${prefix}base_link-base" type="fixed">
-      <origin xyz="0 0 0.540" rpy="0 0 0"/>
-      <parent link="${prefix}base_link"/>
-      <child link="${prefix}base"/>
-    </joint>
   </xacro:macro>
 </robot>

File: motoman_gp215_support/urdf/gp215_macro.xacro (robot description, xacro)
@@ -140,4 +140,11 @@
     </joint>
     <!-- end of joint list -->
+    <!-- ROS base_link to Robot Manufacturer World Coordinates transform -->
+    <link name="${prefix}base" />
+    <joint name="${prefix}base_link-base" type="fixed">
+      <origin xyz="0 0 0.640" rpy="0 0 0"/>
+      <parent link="${prefix}base_link"/>
+      <child link="${prefix}base"/>
+    </joint>
     <!-- ROS-Industrial 'flange' frame: attachment point for EEF models -->
     <link name="${prefix}flange"/>
@@ -154,11 +161,4 @@
       <child link="${prefix}tool0"/>
     </joint>
-    <!-- ROS base_link to Robot Manufacturer World Coordinates transform -->
-    <link name="${prefix}base" />
-    <joint name="${prefix}base_link-base" type="fixed">
-      <origin xyz="0 0 0.640" rpy="0 0 0"/>
-      <parent link="${prefix}base_link"/>
-      <child link="${prefix}base"/>
-    </joint>
   </xacro:macro>
 </robot>

File: motoman_gp225_support/urdf/gp225_macro.xacro (robot description, xacro)
@@ -139,5 +139,4 @@
         <limit lower="${radians(-360)}" upper="${radians(360)}" effort="2250.6" velocity="${radians(220)}"/>
     </joint>
-    <!-- end of joint list -->
     <!-- balancer -->
     <link name="${prefix}link_1_s_2">
@@ -179,4 +178,5 @@
         <mimic joint="${prefix}joint_2_l" multiplier="-0.2366"/>
     </joint>
+    <!-- end of joint list -->
     <!-- ROS base_link to Robot Manufacturer World Coordinates transform -->
     <link name="${prefix}base" />

File: motoman_gp250_support/urdf/gp250_macro.xacro (robot description, xacro)
@@ -140,4 +140,11 @@
     </joint>
     <!-- end of joint list -->
+    <!-- ROS base_link to Robot Manufacturer World Coordinates transform -->
+    <link name="${prefix}base" />
+    <joint name="${prefix}base_link-base" type="fixed">
+      <origin xyz="0 0 0.640" rpy="0 0 0"/>
+      <parent link="${prefix}base_link"/>
+      <child link="${prefix}base"/>
+    </joint>
     <!-- ROS-Industrial 'flange' frame: attachment point for EEF models -->
     <link name="${prefix}flange"/>
@@ -154,11 +161,4 @@
       <child link="${prefix}tool0"/>
     </joint>
-    <!-- ROS base_link to Robot Manufacturer World Coordinates transform -->
-    <link name="${prefix}base" />
-    <joint name="${prefix}base_link-base" type="fixed">
-      <origin xyz="0 0 0.640" rpy="0 0 0"/>
-      <parent link="${prefix}base_link"/>
-      <child link="${prefix}base"/>
-    </joint>
   </xacro:macro>
 </robot>

File: motoman_gp25_support/urdf/gp25_12_macro.xacro (robot description, xacro)
@@ -140,4 +140,11 @@
     </joint>
     <!-- end of joint list -->
+    <!-- ROS base_link to Robot Manufacturer World Coordinates transform -->
+    <link name="${prefix}base" />
+    <joint name="${prefix}base_link-base" type="fixed">
+        <origin xyz="0 0 0.505" rpy="0 0 0"/>
+        <parent link="${prefix}base_link"/>
+        <child link="${prefix}base"/>
+    </joint>
     <!-- ROS-Industrial 'flange' frame: attachment point for EEF models -->
     <link name="${prefix}flange"/>
@@ -154,11 +161,4 @@
       <child link="${prefix}tool0"/>
     </joint>
-    <!-- ROS base_link to Robot Manufacturer World Coordinates transform -->
-    <link name="${prefix}base" />
-    <joint name="${prefix}base_link-base" type="fixed">
-        <origin xyz="0 0 0.505" rpy="0 0 0"/>
-        <parent link="${prefix}base_link"/>
-        <child link="${prefix}base"/>
-    </joint>
     </xacro:macro>
 </robot>

File: motoman_gp25_support/urdf/gp25_20_macro.xacro (robot description, xacro)
@@ -140,4 +140,11 @@
     </joint>
     <!-- end of joint list -->
+    <!-- ROS base_link to Robot Manufacturer World Coordinates transform -->
+    <link name="${prefix}base" />
+    <joint name="${prefix}base_link-base" type="fixed">
+        <origin xyz="0 0 0.505" rpy="0 0 0"/>
+        <parent link="${prefix}base_link"/>
+        <child link="${prefix}base"/>
+    </joint>
     <!-- ROS-Industrial 'flange' frame: attachment point for EEF models -->
     <link name="${prefix}flange"/>
@@ -154,11 +161,4 @@
       <child link="${prefix}tool0"/>
     </joint>
-    <!-- ROS base_link to Robot Manufacturer World Coordinates transform -->
-    <link name="${prefix}base" />
-    <joint name="${prefix}base_link-base" type="fixed">
-        <origin xyz="0 0 0.505" rpy="0 0 0"/>
-        <parent link="${prefix}base_link"/>
-        <child link="${prefix}base"/>
-    </joint>
   </xacro:macro>
 </robot>

File: motoman_gp25_support/urdf/gp25_macro.xacro (robot description, xacro)
@@ -140,4 +140,11 @@
     </joint>
     <!-- end of joint list -->
+    <!-- ROS base_link to Robot Manufacturer World Coordinates transform -->
+    <link name="${prefix}base" />
+    <joint name="${prefix}base_link-base" type="fixed">
+        <origin xyz="0 0 0.505" rpy="0 0 0"/>
+        <parent link="${prefix}base_link"/>
+        <child link="${prefix}base"/>
+    </joint>
     <!-- ROS-Industrial 'flange' frame: attachment point for EEF models -->
     <link name="${prefix}flange"/>
@@ -154,11 +161,4 @@
       <child link="${prefix}tool0"/>
     </joint>
-    <!-- ROS base_link to Robot Manufacturer World Coordinates transform -->
-    <link name="${prefix}base" />
-    <joint name="${prefix}base_link-base" type="fixed">
-        <origin xyz="0 0 0.505" rpy="0 0 0"/>
-        <parent link="${prefix}base_link"/>
-        <child link="${prefix}base"/>
-    </joint>
     </xacro:macro>
 </robot>

File: motoman_gp35l_support/urdf/gp35l_macro.xacro (robot description, xacro)
@@ -140,4 +140,11 @@
     </joint>
     <!-- end of joint list -->
+    <!-- ROS base_link to Robot Manufacturer World Coordinates transform -->
+    <link name="${prefix}base" />
+    <joint name="${prefix}base_link-base" type="fixed">
+      <origin xyz="0 0 0.540" rpy="0 0 0"/>
+      <parent link="${prefix}base_link"/>
+      <child link="${prefix}base"/>
+    </joint>
     <!-- ROS-Industrial 'flange' frame: attachment point for EEF models -->
     <link name="${prefix}flange"/>
@@ -154,11 +161,4 @@
       <child link="${prefix}tool0"/>
     </joint>
-    <!-- ROS base_link to Robot Manufacturer World Coordinates transform -->
-    <link name="${prefix}base" />
-    <joint name="${prefix}base_link-base" type="fixed">
-      <origin xyz="0 0 0.540" rpy="0 0 0"/>
-      <parent link="${prefix}base_link"/>
-      <child link="${prefix}base"/>
-    </joint>
   </xacro:macro>
 </robot>

File: motoman_gp4_support/urdf/gp4_macro.xacro (robot description, xacro)
@@ -140,4 +140,11 @@
     </joint>
     <!-- end of joint list -->
+    <!-- ROS base_link to Robot Manufacturer World Coordinates transform -->
+    <link name="${prefix}base" />
+    <joint name="${prefix}base_link-base" type="fixed">
+      <origin xyz="0 0 0.330" rpy="0 0 0"/>
+      <parent link="${prefix}base_link"/>
+      <child link="${prefix}base"/>
+    </joint>
     <!-- ROS-Industrial 'flange' frame: attachment point for EEF models -->
     <link name="${prefix}flange"/>
@@ -154,11 +161,4 @@
       <child link="${prefix}tool0"/>
     </joint>
-    <!-- ROS base_link to Robot Manufacturer World Coordinates transform -->
-    <link name="${prefix}base" />
-    <joint name="${prefix}base_link-base" type="fixed">
-      <origin xyz="0 0 0.330" rpy="0 0 0"/>
-      <parent link="${prefix}base_link"/>
-      <child link="${prefix}base"/>
-    </joint>
   </xacro:macro>
 </robot>

File: motoman_gp50_support/urdf/gp50_macro.xacro (robot description, xacro)
@@ -139,4 +139,12 @@
         <limit lower="${radians(-360)}" upper="${radians(360)}" effort="375" velocity="${radians(360)}"/>
     </joint>
+    <!-- end of joint list -->
+    <!-- ROS base_link to Robot Manufacturer World Coordinates transform -->
+    <link name="${prefix}base" />
+    <joint name="${prefix}base_link-base" type="fixed">
+        <origin xyz="0 0 0.540" rpy="0 0 0"/>
+        <parent link="${prefix}base_link"/>
+        <child link="${prefix}base"/>
+    </joint>
     <!-- ROS-Industrial 'flange' frame: attachment point for EEF models -->
     <link name="${prefix}flange" />
@@ -153,12 +161,4 @@
         <child link="${prefix}tool0" />
     </joint>
-    <!-- end of joint list -->
-    <!-- ROS base_link to Robot Manufacturer World Coordinates transform -->
-    <link name="${prefix}base" />
-    <joint name="${prefix}base_link-base" type="fixed">
-        <origin xyz="0 0 0.540" rpy="0 0 0"/>
-        <parent link="${prefix}base_link"/>
-        <child link="${prefix}base"/>
-    </joint>
   </xacro:macro>
 </robot>

File: motoman_gp70l_support/urdf/gp70l_macro.xacro (robot description, xacro)
@@ -140,4 +140,11 @@
     </joint>
     <!-- end of joint list -->
+    <!-- ROS base_link to Robot Manufacturer World Coordinates transform -->
+    <link name="${prefix}base" />
+    <joint name="${prefix}base_link-base" type="fixed">
+      <origin xyz="0 0 0.540" rpy="0 0 0"/>
+      <parent link="${prefix}base_link"/>
+      <child link="${prefix}base"/>
+    </joint>
     <!-- ROS-Industrial 'flange' frame: attachment point for EEF models -->
     <link name="${prefix}flange"/>
@@ -154,11 +161,4 @@
       <child link="${prefix}tool0"/>
     </joint>
-    <!-- ROS base_link to Robot Manufacturer World Coordinates transform -->
-    <link name="${prefix}base" />
-    <joint name="${prefix}base_link-base" type="fixed">
-      <origin xyz="0 0 0.540" rpy="0 0 0"/>
-      <parent link="${prefix}base_link"/>
-      <child link="${prefix}base"/>
-    </joint>
   </xacro:macro>
 </robot>

File: motoman_gp7_support/urdf/gp7_macro.xacro (robot description, xacro)
@@ -140,4 +140,11 @@
     </joint>
     <!-- end of joint list -->
+    <!-- ROS base_link to Robot Manufacturer World Coordinates transform -->
+    <link name="${prefix}base" />
+    <joint name="${prefix}base_link-base" type="fixed">
+        <origin xyz="0 0 0.330" rpy="0 0 0"/>
+        <parent link="${prefix}base_link"/>
+        <child link="${prefix}base"/>
+    </joint>
     <!-- ROS-Industrial 'flange' frame: attachment point for EEF models -->
     <link name="${prefix}flange"/>
@@ -154,11 +161,4 @@
         <child link="${prefix}tool0"/>
     </joint>
-    <!-- ROS base_link to Robot Manufacturer World Coordinates transform -->
-    <link name="${prefix}base" />
-    <joint name="${prefix}base_link-base" type="fixed">
-        <origin xyz="0 0 0.330" rpy="0 0 0"/>
-        <parent link="${prefix}base_link"/>
-        <child link="${prefix}base"/>
-    </joint>
     </xacro:macro>
 </robot>

File: motoman_gp8_support/urdf/gp8_macro.xacro (robot description, xacro)
@@ -140,4 +140,11 @@
     </joint>
     <!-- end of joint list -->
+    <!-- ROS base_link to Robot Manufacturer World Coordinates transform -->
+    <link name="${prefix}base" />
+    <joint name="${prefix}base_link-base" type="fixed">
+      <origin xyz="0 0 0.330" rpy="0 0 0"/>
+      <parent link="${prefix}base_link"/>
+      <child link="${prefix}base"/>
+    </joint>
     <!-- ROS-Industrial 'flange' frame: attachment point for EEF models -->
     <link name="${prefix}flange"/>
@@ -154,11 +161,4 @@
       <child link="${prefix}tool0"/>
     </joint>
-    <!-- ROS base_link to Robot Manufacturer World Coordinates transform -->
-    <link name="${prefix}base" />
-    <joint name="${prefix}base_link-base" type="fixed">
-      <origin xyz="0 0 0.330" rpy="0 0 0"/>
-      <parent link="${prefix}base_link"/>
-      <child link="${prefix}base"/>
-    </joint>
   </xacro:macro>
 </robot>

File: motoman_gp8l_support/urdf/gp8l_macro.xacro (robot description, xacro)
@@ -140,4 +140,11 @@
     </joint>
     <!-- end of joint list -->
+    <!-- ROS base_link to Robot Manufacturer World Coordinates transform -->
+    <link name="${prefix}base" />
+    <joint name="${prefix}base_link-base" type="fixed">
+      <origin xyz="0 0 0.450" rpy="0 0 0"/>
+      <parent link="${prefix}base_link"/>
+      <child link="${prefix}base"/>
+    </joint>
     <!-- ROS-Industrial 'flange' frame: attachment point for EEF models -->
     <link name="${prefix}flange"/>
@@ -154,11 +161,4 @@
       <child link="${prefix}tool0"/>
     </joint>
-    <!-- ROS base_link to Robot Manufacturer World Coordinates transform -->
-    <link name="${prefix}base" />
-    <joint name="${prefix}base_link-base" type="fixed">
-      <origin xyz="0 0 0.450" rpy="0 0 0"/>
-      <parent link="${prefix}base_link"/>
-      <child link="${prefix}base"/>
-    </joint>
   </xacro:macro>
 </robot>

File: motoman_hc10_support/urdf/hc10_macro.xacro (robot description, xacro)
@@ -139,4 +139,12 @@
       <limit lower="${radians(-180)}" upper="${radians(180)}" effort="31.36" velocity="${radians(250)}"/>
     </joint>
+    <!-- end of joint list -->
+    <!-- ROS base_link to Robot Manufacturer World Coordinates transform -->
+    <link name="${prefix}base" />
+    <joint name="${prefix}base_link-base" type="fixed">
+      <origin xyz="0 0 0.275" rpy="0 0 0"/>
+      <parent link="${prefix}base_link"/>
+      <child link="${prefix}base"/>
+    </joint>
     <!-- ROS-Industrial 'flange' frame: attachment point for EEF models -->
     <link name="${prefix}flange" />
@@ -153,12 +161,4 @@
         <child link="${prefix}tool0" />
     </joint>
-    <!-- end of joint list -->
-    <!-- ROS base_link to Robot Manufacturer World Coordinates transform -->
-    <link name="${prefix}base" />
-    <joint name="${prefix}base_link-base" type="fixed">
-      <origin xyz="0 0 0.275" rpy="0 0 0"/>
-      <parent link="${prefix}base_link"/>
-      <child link="${prefix}base"/>
-    </joint>
   </xacro:macro>
 </robot>
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