Commit message: Change es mesh materials

File: motoman_es_support/urdf/es165_macro.xacro (robot description, xacro)
@@ -2,14 +2,13 @@
 <robot xmlns:xacro="http://ros.org/wiki/xacro">
   <xacro:macro name="motoman_es165" params="prefix joint_velocities_file">
+    <xacro:include filename="$(find motoman_resources)/urdf/common_materials.xacro"/>
     <!-- link list -->
     <link name="${prefix}base_link">
       <visual>
         <origin xyz="0 0 0" rpy="0 0 0"/>
-          <geometry>
-            <mesh filename="package://motoman_es_support/meshes/es/visual/base_link.stl"/>
-          </geometry>
-          <material name="blue">
-            <color rgba="0 0 1 1"/>
-          </material>
+        <geometry>
+          <mesh filename="package://motoman_es_support/meshes/es/visual/base_link.stl"/>
+        </geometry>
+        <xacro:material_yaskawa_blue/>
       </visual>
       <collision>
@@ -17,7 +16,4 @@
           <mesh filename="package://motoman_es_support/meshes/es/collision/base_link.stl"/>
         </geometry>
-        <material name="yellow">
-          <color rgba="0 1 1 1"/>
-        </material>
       </collision>
     </link>
@@ -28,5 +24,5 @@
           <mesh filename="package://motoman_es_support/meshes/es/visual/link_1.stl"/>
         </geometry>
-        <material name="blue"/>
+        <xacro:material_yaskawa_blue/>
       </visual>
       <collision>
@@ -35,5 +31,4 @@
           <mesh filename="package://motoman_es_support/meshes/es/collision/link_1.stl"/>
         </geometry>
-        <material name="yellow"/>
       </collision>
     </link>
@@ -44,5 +39,5 @@
           <mesh filename="package://motoman_es_support/meshes/es/visual/link_2.stl"/>
         </geometry>
-        <material name="blue"/>
+        <xacro:material_yaskawa_blue/>
       </visual>
       <collision>
@@ -51,5 +46,4 @@
           <mesh filename="package://motoman_es_support/meshes/es/collision/link_2.stl"/>
         </geometry>
-        <material name="yellow"/>
       </collision>
     </link>
@@ -60,5 +54,5 @@
           <mesh filename="package://motoman_es_support/meshes/es/visual/link_3.stl"/>
         </geometry>
-        <material name="blue"/>
+        <xacro:material_yaskawa_blue/>
       </visual>
       <collision>
@@ -67,5 +61,4 @@
           <mesh filename="package://motoman_es_support/meshes/es/collision/link_3.stl"/>
         </geometry>
-        <material name="yellow"/>
       </collision>
     </link>
@@ -73,8 +66,8 @@
       <visual>
         <origin xyz="0 0 0" rpy="0 0 0"/>
-      <geometry>
-        <mesh filename="package://motoman_es_support/meshes/es165/visual/link_4.stl"/>
-      </geometry>
-      <material name="blue"/>
+        <geometry>
+          <mesh filename="package://motoman_es_support/meshes/es165/visual/link_4.stl"/>
+        </geometry>
+        <xacro:material_yaskawa_blue/>
       </visual>
       <collision>
@@ -83,5 +76,4 @@
           <mesh filename="package://motoman_es_support/meshes/es165/collision/link_4.stl"/>
         </geometry>
-        <material name="yellow"/>
       </collision>
     </link>
@@ -92,5 +84,5 @@
           <mesh filename="package://motoman_es_support/meshes/es/visual/link_5.stl"/>
         </geometry>
-        <material name="blue"/>
+        <xacro:material_yaskawa_blue/>
       </visual>
       <collision>
@@ -99,5 +91,4 @@
           <mesh filename="package://motoman_es_support/meshes/es/collision/link_5.stl"/>
         </geometry>
-        <material name="yellow"/>
       </collision>
     </link>
@@ -105,10 +96,8 @@
       <visual>
         <origin xyz="0 0 0" rpy="0 0 0"/>
-          <geometry>
-            <mesh filename="package://motoman_es_support/meshes/es/visual/link_6.stl"/>
-          </geometry>
-          <material name="black">
-            <color rgba="0 0 0 1"/>
-          </material>
+        <geometry>
+          <mesh filename="package://motoman_es_support/meshes/es/visual/link_6.stl"/>
+        </geometry>
+        <xacro:material_yaskawa_silver/>
       </visual>
       <collision>
@@ -117,5 +106,4 @@
           <mesh filename="package://motoman_es_support/meshes/es/collision/link_6.stl"/>
         </geometry>
-        <material name="black"/>
       </collision>
     </link>
@@ -131,5 +119,5 @@
           <mesh filename="package://motoman_es_support/meshes/es/visual/balancer_piston.stl"/>
         </geometry>
-        <material name="blue"/>
+        <xacro:material_yaskawa_blue/>
       </visual>
       <collision>
@@ -138,5 +126,4 @@
           <mesh filename="package://motoman_es_support/meshes/es/collision/balancer_piston.stl"/>
         </geometry>
-        <material name="yellow"/>
       </collision>
     </link>
@@ -147,7 +134,5 @@
           <mesh filename="package://motoman_es_support/meshes/es/visual/balancer_rod.stl"/>
         </geometry>
-        <material name="blue">
-          <color rgba="1 1 1 1"/>
-        </material>
+        <xacro:material_yaskawa_blue/>
       </visual>
       <collision>
@@ -156,5 +141,4 @@
           <mesh filename="package://motoman_es_support/meshes/es/collision/balancer_rod.stl"/>
         </geometry>
-        <material name="yellow"/>
       </collision>
     </link>

File: motoman_es_support/urdf/es200_120_macro.xacro (robot description, xacro)
@@ -2,4 +2,5 @@
 <robot xmlns:xacro="http://ros.org/wiki/xacro">
   <xacro:macro name="motoman_es200_120" params="prefix joint_velocities_file">
+    <xacro:include filename="$(find motoman_resources)/urdf/common_materials.xacro"/>
     <!-- link list -->
     <link name="${prefix}base_link">
@@ -9,7 +10,5 @@
           <mesh filename="package://motoman_es_support/meshes/es/visual/base_link.stl"/>
         </geometry>
-        <material name="blue">
-          <color rgba="0 0 1 1"/>
-        </material>
+        <xacro:material_yaskawa_blue/>
       </visual>
       <collision>
@@ -17,7 +16,4 @@
           <mesh filename="package://motoman_es_support/meshes/es/collision/base_link.stl"/>
         </geometry>
-        <material name="yellow">
-          <color rgba="0 1 1 1"/>
-        </material>
       </collision>
     </link>
@@ -28,5 +24,5 @@
           <mesh filename="package://motoman_es_support/meshes/es/visual/link_1.stl"/>
         </geometry>
-        <material name="blue"/>
+        <xacro:material_yaskawa_blue/>
       </visual>
       <collision>
@@ -35,5 +31,4 @@
           <mesh filename="package://motoman_es_support/meshes/es/collision/link_1.stl"/>
         </geometry>
-        <material name="yellow"/>
       </collision>
     </link>
@@ -44,5 +39,5 @@
           <mesh filename="package://motoman_es_support/meshes/es/visual/link_2.stl"/>
         </geometry>
-        <material name="blue"/>
+        <xacro:material_yaskawa_blue/>
       </visual>
       <collision>
@@ -51,5 +46,4 @@
           <mesh filename="package://motoman_es_support/meshes/es/collision/link_2.stl"/>
         </geometry>
-        <material name="yellow"/>
       </collision>
     </link>
@@ -60,5 +54,5 @@
           <mesh filename="package://motoman_es_support/meshes/es200_120/visual/link_3.stl"/>
         </geometry>
-        <material name="blue"/>
+        <xacro:material_yaskawa_blue/>
       </visual>
       <collision>
@@ -67,5 +61,4 @@
           <mesh filename="package://motoman_es_support/meshes/es200_120/collision/link_3.stl"/>
         </geometry>
-        <material name="yellow"/>
       </collision>
     </link>
@@ -76,5 +69,5 @@
           <mesh filename="package://motoman_es_support/meshes/es200_120/visual/link_4.stl"/>
         </geometry>
-        <material name="blue"/>
+        <xacro:material_yaskawa_blue/>
       </visual>
       <collision>
@@ -83,5 +76,4 @@
           <mesh filename="package://motoman_es_support/meshes/es200_120/collision/link_4.stl"/>
         </geometry>
-        <material name="yellow"/>
       </collision>
     </link>
@@ -92,5 +84,5 @@
           <mesh filename="package://motoman_es_support/meshes/es/visual/link_5.stl"/>
         </geometry>
-        <material name="blue"/>
+        <xacro:material_yaskawa_blue/>
       </visual>
       <collision>
@@ -99,5 +91,4 @@
           <mesh filename="package://motoman_es_support/meshes/es/collision/link_5.stl"/>
         </geometry>
-        <material name="yellow"/>
       </collision>
     </link>
@@ -108,7 +99,5 @@
           <mesh filename="package://motoman_es_support/meshes/es/visual/link_6.stl"/>
         </geometry>
-        <material name="black">
-          <color rgba="0 0 0 1"/>
-        </material>
+        <xacro:material_yaskawa_silver/>
       </visual>
       <collision>
@@ -117,5 +106,4 @@
           <mesh filename="package://motoman_es_support/meshes/es/collision/link_6.stl"/>
         </geometry>
-        <material name="black"/>
       </collision>
     </link>
@@ -131,5 +119,5 @@
           <mesh filename="package://motoman_es_support/meshes/es/visual/balancer_piston.stl"/>
         </geometry>
-        <material name="blue"/>
+        <xacro:material_yaskawa_blue/>
       </visual>
       <collision>
@@ -138,5 +126,4 @@
           <mesh filename="package://motoman_es_support/meshes/es/collision/balancer_piston.stl"/>
         </geometry>
-        <material name="yellow"/>
       </collision>
     </link>
@@ -147,5 +134,5 @@
           <mesh filename="package://motoman_es_support/meshes/es/visual/balancer_rod.stl"/>
         </geometry>
-        <material name="blue"/>
+        <xacro:material_yaskawa_blue/>
       </visual>
       <collision>
@@ -154,5 +141,4 @@
           <mesh filename="package://motoman_es_support/meshes/es/collision/balancer_rod.stl"/>
         </geometry>
-        <material name="yellow"/>
       </collision>
     </link>

Commit message: Fix broken joint_3 limits on es robots

File: motoman_es_support/urdf/es165_macro.xacro (robot description, xacro)
@@ -166,5 +166,5 @@
       <child link="${prefix}link_3"/>
       <axis xyz="0 -1 0"/>
-      <limit lower="${radians(-112)}" upper="${radians(208)}" effort="${limits['joint_3']['effort']}" velocity="${radians(limits['joint_3']['velocity'])}"/>
+      <limit lower="${radians(-79.4)}" upper="${radians(78)}" effort="${limits['joint_3']['effort']}" velocity="${radians(limits['joint_3']['velocity'])}"/>
     </joint>
     <joint name="${prefix}joint_4" type="revolute">

File: motoman_es_support/urdf/es200_120_macro.xacro (robot description, xacro)
@@ -166,5 +166,5 @@
       <child link="${prefix}link_3"/>
       <axis xyz="0 -1 0"/>
-      <limit lower="${radians(-107)}" upper="${radians(190)}" effort="${limits['joint_3']['effort']}" velocity="${radians(limits['joint_3']['velocity'])}"/>
+      <limit lower="${radians(-78.4)}" upper="${radians(90)}" effort="${limits['joint_3']['effort']}" velocity="${radians(limits['joint_3']['velocity'])}"/>
     </joint>
     <joint name="${prefix}joint_4" type="revolute">
