Commit message: es_changes

File: motoman_es_support/urdf/es165rd_macro.xacro (robot description, xacro)
@@ -1,15 +1,15 @@
 <?xml version="1.0"?>
 <robot xmlns:xacro="http://ros.org/wiki/xacro">
-  <xacro:macro name="motoman_es200_120" params="prefix joint_velocities_file">
+  <xacro:macro name="motoman_es165" params="prefix joint_velocities_file">
     <!-- link list -->
     <link name="${prefix}base_link">
       <visual>
         <origin xyz="0 0 0" rpy="0 0 0"/>
-        <geometry>
-          <mesh filename="package://motoman_es_support/meshes/es/visual/base_link.stl"/>
-        </geometry>
-        <material name="blue">
-          <color rgba="0 0 1 1"/>
-        </material>
+          <geometry>
+            <mesh filename="package://motoman_es_support/meshes/es/visual/base_link.stl"/>
+          </geometry>
+          <material name="blue">
+            <color rgba="0 0 1 1"/>
+          </material>
       </visual>
       <collision>
@@ -58,12 +58,12 @@
         <origin xyz="0 0 0" rpy="0 0 0"/>
         <geometry>
-          <mesh filename="package://motoman_es_support/meshes/es200_120/visual/link_3.stl"/>
-        </geometry>
-        <material name="blue"/>
-      </visual>
-      <collision>
-        <origin xyz="0 0 0" rpy="0 0 0"/>
-        <geometry>
-          <mesh filename="package://motoman_es_support/meshes/es200_120/collision/link_3.stl"/>
+          <mesh filename="package://motoman_es_support/meshes/es/visual/link_3.stl"/>
+        </geometry>
+        <material name="blue"/>
+      </visual>
+      <collision>
+        <origin xyz="0 0 0" rpy="0 0 0"/>
+        <geometry>
+          <mesh filename="package://motoman_es_support/meshes/es/collision/link_3.stl"/>
         </geometry>
         <material name="yellow"/>
@@ -73,13 +73,13 @@
       <visual>
         <origin xyz="0 0 0" rpy="0 0 0"/>
-        <geometry>
-          <mesh filename="package://motoman_es_support/meshes/es200_120/visual/link_4.stl"/>
-        </geometry>
-        <material name="blue"/>
-      </visual>
-      <collision>
-        <origin xyz="0 0 0" rpy="0 0 0"/>
-        <geometry>
-          <mesh filename="package://motoman_es_support/meshes/es200_120/collision/link_4.stl"/>
+      <geometry>
+        <mesh filename="package://motoman_es_support/meshes/es165/visual/link_4.stl"/>
+      </geometry>
+      <material name="blue"/>
+      </visual>
+      <collision>
+        <origin xyz="0 0 0" rpy="0 0 0"/>
+        <geometry>
+          <mesh filename="package://motoman_es_support/meshes/es165/collision/link_4.stl"/>
         </geometry>
         <material name="yellow"/>
@@ -105,10 +105,10 @@
       <visual>
         <origin xyz="0 0 0" rpy="0 0 0"/>
-        <geometry>
-          <mesh filename="package://motoman_es_support/meshes/es/visual/link_6.stl"/>
-        </geometry>
-        <material name="black">
-          <color rgba="0 0 0 1"/>
-        </material>
+          <geometry>
+            <mesh filename="package://motoman_es_support/meshes/es/visual/link_6.stl"/>
+          </geometry>
+          <material name="black">
+            <color rgba="0 0 0 1"/>
+          </material>
       </visual>
       <collision>
@@ -147,5 +147,7 @@
           <mesh filename="package://motoman_es_support/meshes/es/visual/balancer_rod.stl"/>
         </geometry>
-        <material name="blue"/>
+        <material name="blue">
+          <color rgba="1 1 1 1"/>
+        </material>
       </visual>
       <collision>
@@ -166,5 +168,5 @@
       <child link="${prefix}link_1"/>
       <axis xyz="0 0 1"/>
-      <limit lower="${radians(-180)}" upper="${radians(180)}" effort="0" velocity="${radians(velocities['joint_1'])}"/>
+      <limit lower="${radians(-180)}" upper="${radians(180)}" effort="6354.71" velocity="${radians(velocities['joint_1'])}"/>
     </joint>
     <joint name="${prefix}joint_2" type="revolute">
@@ -173,5 +175,5 @@
       <child link="${prefix}link_2"/>
       <axis xyz="0 1 0"/>
-      <limit lower="${radians(-130)}" upper="${radians(80)}" effort="0" velocity="${radians(velocities['joint_2'])}"/>
+      <limit lower="${radians(-130)}" upper="${radians(80)}" effort="8825.98" velocity="${radians(velocities['joint_2'])}"/>
     </joint>
     <joint name="${prefix}joint_3" type="revolute">
@@ -180,5 +182,5 @@
       <child link="${prefix}link_3"/>
       <axis xyz="0 -1 0"/>
-      <limit lower="${radians(-107)}" upper="${radians(190)}" effort="0" velocity="${radians(velocities['joint_3'])}"/>
+      <limit lower="${radians(-79.4)}" upper="${radians(78)}" effort="6276.26" velocity="${radians(velocities['joint_3'])}"/>
     </joint>
     <joint name="${prefix}joint_4" type="revolute">
@@ -187,12 +189,12 @@
       <child link="${prefix}link_4"/>
       <axis xyz="0 0 1"/>
-      <limit lower="${radians(-360)}" upper="${radians(360)}" effort="0" velocity="${radians(velocities['joint_4'])}"/>
+      <limit lower="${radians(-360)}" upper="${radians(360)}" effort="1253.29" velocity="${radians(velocities['joint_4'])}"/>
     </joint>
     <joint name="${prefix}joint_5" type="revolute">
-      <origin xyz="0 0 -2.100" rpy="0 0 0"/>
+      <origin xyz="0 0 -1.225" rpy="0 0 0"/>
       <parent link="${prefix}link_4"/>
       <child link="${prefix}link_5"/>
       <axis xyz="0 -1 0"/>
-      <limit lower="${radians(-130)}" upper="${radians(130)}" effort="0" velocity="${radians(velocities['joint_5'])}"/>
+      <limit lower="${radians(-130)}" upper="${radians(130)}" effort="1725.97" velocity="${radians(velocities['joint_5'])}"/>
     </joint>
     <joint name="${prefix}joint_6" type="revolute">
@@ -201,5 +203,5 @@
       <child link="${prefix}link_6"/>
       <axis xyz="0 0 1"/>
-      <limit lower="${radians(-360)}" upper="${radians(360)}" effort="0" velocity="${radians(velocities['joint_6'])}"/>
+      <limit lower="${radians(-360)}" upper="${radians(360)}" effort="638.41" velocity="${radians(velocities['joint_6'])}"/>
     </joint>
     <!--
@@ -218,5 +220,5 @@
     <!-- end of joint list -->
     <!-- ROS base_link to Robot Manufacturer World Coordinates transform -->
-    <link name="${prefix}base"/>
+    <link name="${prefix}base" />
     <joint name="${prefix}base_link-base" type="fixed">
       <origin xyz="0 0 0.450" rpy="0 0 0"/>

File: motoman_es_support/urdf/es200rd_120_macro.xacro (robot description, xacro)
@@ -1,15 +1,15 @@
 <?xml version="1.0"?>
 <robot xmlns:xacro="http://ros.org/wiki/xacro">
-  <xacro:macro name="motoman_es165" params="prefix joint_velocities_file">
+  <xacro:macro name="motoman_es200_120" params="prefix joint_velocities_file">
     <!-- link list -->
     <link name="${prefix}base_link">
       <visual>
         <origin xyz="0 0 0" rpy="0 0 0"/>
-          <geometry>
-            <mesh filename="package://motoman_es_support/meshes/es/visual/base_link.stl"/>
-          </geometry>
-          <material name="blue">
-            <color rgba="0 0 1 1"/>
-          </material>
+        <geometry>
+          <mesh filename="package://motoman_es_support/meshes/es/visual/base_link.stl"/>
+        </geometry>
+        <material name="blue">
+          <color rgba="0 0 1 1"/>
+        </material>
       </visual>
       <collision>
@@ -58,12 +58,12 @@
         <origin xyz="0 0 0" rpy="0 0 0"/>
         <geometry>
-          <mesh filename="package://motoman_es_support/meshes/es/visual/link_3.stl"/>
-        </geometry>
-        <material name="blue"/>
-      </visual>
-      <collision>
-        <origin xyz="0 0 0" rpy="0 0 0"/>
-        <geometry>
-          <mesh filename="package://motoman_es_support/meshes/es/collision/link_3.stl"/>
+          <mesh filename="package://motoman_es_support/meshes/es200_120/visual/link_3.stl"/>
+        </geometry>
+        <material name="blue"/>
+      </visual>
+      <collision>
+        <origin xyz="0 0 0" rpy="0 0 0"/>
+        <geometry>
+          <mesh filename="package://motoman_es_support/meshes/es200_120/collision/link_3.stl"/>
         </geometry>
         <material name="yellow"/>
@@ -73,13 +73,13 @@
       <visual>
         <origin xyz="0 0 0" rpy="0 0 0"/>
-      <geometry>
-        <mesh filename="package://motoman_es_support/meshes/es165/visual/link_4.stl"/>
-      </geometry>
-      <material name="blue"/>
-      </visual>
-      <collision>
-        <origin xyz="0 0 0" rpy="0 0 0"/>
-        <geometry>
-          <mesh filename="package://motoman_es_support/meshes/es165/collision/link_4.stl"/>
+        <geometry>
+          <mesh filename="package://motoman_es_support/meshes/es200_120/visual/link_4.stl"/>
+        </geometry>
+        <material name="blue"/>
+      </visual>
+      <collision>
+        <origin xyz="0 0 0" rpy="0 0 0"/>
+        <geometry>
+          <mesh filename="package://motoman_es_support/meshes/es200_120/collision/link_4.stl"/>
         </geometry>
         <material name="yellow"/>
@@ -105,10 +105,10 @@
       <visual>
         <origin xyz="0 0 0" rpy="0 0 0"/>
-          <geometry>
-            <mesh filename="package://motoman_es_support/meshes/es/visual/link_6.stl"/>
-          </geometry>
-          <material name="black">
-            <color rgba="0 0 0 1"/>
-          </material>
+        <geometry>
+          <mesh filename="package://motoman_es_support/meshes/es/visual/link_6.stl"/>
+        </geometry>
+        <material name="black">
+          <color rgba="0 0 0 1"/>
+        </material>
       </visual>
       <collision>
@@ -147,7 +147,5 @@
           <mesh filename="package://motoman_es_support/meshes/es/visual/balancer_rod.stl"/>
         </geometry>
-        <material name="blue">
-          <color rgba="1 1 1 1"/>
-        </material>
+        <material name="blue"/>
       </visual>
       <collision>
@@ -168,5 +166,5 @@
       <child link="${prefix}link_1"/>
       <axis xyz="0 0 1"/>
-      <limit lower="${radians(-180)}" upper="${radians(180)}" effort="0" velocity="${radians(velocities['joint_1'])}"/>
+      <limit lower="${radians(-180)}" upper="${radians(180)}" effort="0" velocity="${radians(90)}"/>
     </joint>
     <joint name="${prefix}joint_2" type="revolute">
@@ -175,5 +173,5 @@
       <child link="${prefix}link_2"/>
       <axis xyz="0 1 0"/>
-      <limit lower="${radians(-130)}" upper="${radians(80)}" effort="0" velocity="${radians(velocities['joint_2'])}"/>
+      <limit lower="${radians(-130)}" upper="${radians(80)}" effort="0" velocity="${radians(85)}"/>
     </joint>
     <joint name="${prefix}joint_3" type="revolute">
@@ -182,5 +180,5 @@
       <child link="${prefix}link_3"/>
       <axis xyz="0 -1 0"/>
-      <limit lower="${radians(-112)}" upper="${radians(208)}" effort="0" velocity="${radians(velocities['joint_3'])}"/>
+      <limit lower="${radians(-78.4)}" upper="${radians(90)}" effort="0" velocity="${radians(85)}"/>
     </joint>
     <joint name="${prefix}joint_4" type="revolute">
@@ -189,12 +187,12 @@
       <child link="${prefix}link_4"/>
       <axis xyz="0 0 1"/>
-      <limit lower="${radians(-360)}" upper="${radians(360)}" effort="0" velocity="${radians(velocities['joint_4'])}"/>
+      <limit lower="${radians(-360)}" upper="${radians(360)}" effort="0" velocity="${radians(175)}"/>
     </joint>
     <joint name="${prefix}joint_5" type="revolute">
-      <origin xyz="0 0 -1.225" rpy="0 0 0"/>
+      <origin xyz="0 0 -2.100" rpy="0 0 0"/>
       <parent link="${prefix}link_4"/>
       <child link="${prefix}link_5"/>
       <axis xyz="0 -1 0"/>
-      <limit lower="${radians(-130)}" upper="${radians(130)}" effort="0" velocity="${radians(velocities['joint_5'])}"/>
+      <limit lower="${radians(-130)}" upper="${radians(130)}" effort="0" velocity="${radians(140)}"/>
     </joint>
     <joint name="${prefix}joint_6" type="revolute">
@@ -203,5 +201,5 @@
       <child link="${prefix}link_6"/>
       <axis xyz="0 0 1"/>
-      <limit lower="${radians(-360)}" upper="${radians(360)}" effort="0" velocity="${radians(velocities['joint_6'])}"/>
+      <limit lower="${radians(-360)}" upper="${radians(360)}" effort="0" velocity="${radians(240)}"/>
     </joint>
     <!--
@@ -220,5 +218,5 @@
     <!-- end of joint list -->
     <!-- ROS base_link to Robot Manufacturer World Coordinates transform -->
-    <link name="${prefix}base" />
+    <link name="${prefix}base"/>
     <joint name="${prefix}base_link-base" type="fixed">
       <origin xyz="0 0 0.450" rpy="0 0 0"/>
