Commit message: Reference new es config files

File: motoman_es_support/urdf/es165.xacro (robot description, xacro)
@@ -2,5 +2,5 @@
 <robot name="motoman_es165" xmlns:xacro="http://ros.org/wiki/xacro">
   <xacro:include filename="$(find motoman_es_support)/urdf/es165_macro.xacro"/>
-  <xacro:arg name="joint_velocities_file" default=""/>
-  <xacro:motoman_es165 prefix="" joint_velocities_file="$(arg joint_velocities_file)"/>
+  <xacro:arg name="joint_limits_file" default=""/>
+  <xacro:motoman_es165 prefix="" joint_limits_file="$(arg joint_limits_file)"/>
 </robot>

File: motoman_es_support/urdf/es165_macro.xacro (robot description, xacro)
@@ -1,5 +1,5 @@
 <?xml version="1.0"?>
 <robot xmlns:xacro="http://ros.org/wiki/xacro">
-  <xacro:macro name="motoman_es165" params="prefix joint_velocities_file">
+  <xacro:macro name="motoman_es165" params="prefix joint_limits_file">
     <xacro:include filename="$(find motoman_resources)/urdf/common_materials.xacro"/>
     <!-- link list -->
@@ -146,5 +146,5 @@
     <!-- end of link list -->
     <!-- joint list -->
-    <xacro:property name="velocities" value="${xacro.load_yaml(joint_velocities_file)}" />
+    <xacro:property name="limits" value="${xacro.load_yaml(joint_limits_file)}" />
     <joint name="${prefix}joint_1" type="revolute">
       <origin xyz="0 0 0.450" rpy="0 0 0"/>
@@ -152,5 +152,5 @@
       <child link="${prefix}link_1"/>
       <axis xyz="0 0 1"/>
-      <limit lower="${radians(-180)}" upper="${radians(180)}" effort="0" velocity="${radians(velocities['joint_1'])}"/>
+      <limit lower="${radians(-180)}" upper="${radians(180)}" effort="${limits['joint_1']['effort']}" velocity="${radians(limits['joint_1']['velocity'])}"/>
     </joint>
     <joint name="${prefix}joint_2" type="revolute">
@@ -159,5 +159,5 @@
       <child link="${prefix}link_2"/>
       <axis xyz="0 1 0"/>
-      <limit lower="${radians(-130)}" upper="${radians(80)}" effort="0" velocity="${radians(velocities['joint_2'])}"/>
+      <limit lower="${radians(-130)}" upper="${radians(80)}" effort="${limits['joint_2']['effort']}" velocity="${radians(limits['joint_2']['velocity'])}"/>
     </joint>
     <joint name="${prefix}joint_3" type="revolute">
@@ -166,5 +166,5 @@
       <child link="${prefix}link_3"/>
       <axis xyz="0 -1 0"/>
-      <limit lower="${radians(-112)}" upper="${radians(208)}" effort="0" velocity="${radians(velocities['joint_3'])}"/>
+      <limit lower="${radians(-112)}" upper="${radians(208)}" effort="${limits['joint_3']['effort']}" velocity="${radians(limits['joint_3']['velocity'])}"/>
     </joint>
     <joint name="${prefix}joint_4" type="revolute">
@@ -173,5 +173,5 @@
       <child link="${prefix}link_4"/>
       <axis xyz="0 0 1"/>
-      <limit lower="${radians(-360)}" upper="${radians(360)}" effort="0" velocity="${radians(velocities['joint_4'])}"/>
+      <limit lower="${radians(-360)}" upper="${radians(360)}" effort="${limits['joint_4']['effort']}" velocity="${radians(limits['joint_4']['velocity'])}"/>
     </joint>
     <joint name="${prefix}joint_5" type="revolute">
@@ -180,5 +180,5 @@
       <child link="${prefix}link_5"/>
       <axis xyz="0 -1 0"/>
-      <limit lower="${radians(-130)}" upper="${radians(130)}" effort="0" velocity="${radians(velocities['joint_5'])}"/>
+      <limit lower="${radians(-130)}" upper="${radians(130)}" effort="${limits['joint_5']['effort']}" velocity="${radians(limits['joint_5']['velocity'])}"/>
     </joint>
     <joint name="${prefix}joint_6" type="revolute">
@@ -187,5 +187,5 @@
       <child link="${prefix}link_6"/>
       <axis xyz="0 0 1"/>
-      <limit lower="${radians(-360)}" upper="${radians(360)}" effort="0" velocity="${radians(velocities['joint_6'])}"/>
+      <limit lower="${radians(-360)}" upper="${radians(360)}" effort="${limits['joint_6']['effort']}" velocity="${radians(limits['joint_6']['velocity'])}"/>
     </joint>
     <!--

File: motoman_es_support/urdf/es200_120.xacro (robot description, xacro)
@@ -2,5 +2,5 @@
 <robot name="motoman_es200_120" xmlns:xacro="http://ros.org/wiki/xacro">
   <xacro:include filename="$(find motoman_es_support)/urdf/es200_120_macro.xacro"/>
-  <xacro:arg name="joint_velocities_file" default=""/>
-  <xacro:motoman_es200_120 prefix="" joint_velocities_file="$(arg joint_velocities_file)"/>
+  <xacro:arg name="joint_limits_file" default=""/>
+  <xacro:motoman_es200_120 prefix="" joint_limits_file="$(arg joint_limits_file)"/>
 </robot>

File: motoman_es_support/urdf/es200_120_macro.xacro (robot description, xacro)
@@ -1,5 +1,5 @@
 <?xml version="1.0"?>
 <robot xmlns:xacro="http://ros.org/wiki/xacro">
-  <xacro:macro name="motoman_es200_120" params="prefix joint_velocities_file">
+  <xacro:macro name="motoman_es200_120" params="prefix joint_limits_file">
     <xacro:include filename="$(find motoman_resources)/urdf/common_materials.xacro"/>
     <!-- link list -->
@@ -146,5 +146,5 @@
     <!-- end of link list -->
     <!-- joint list -->
-    <xacro:property name="velocities" value="${xacro.load_yaml(joint_velocities_file)}" />
+    <xacro:property name="limits" value="${xacro.load_yaml(joint_limits_file)}" />
     <joint name="${prefix}joint_1" type="revolute">
       <origin xyz="0 0 0.450" rpy="0 0 0"/>
@@ -152,5 +152,5 @@
       <child link="${prefix}link_1"/>
       <axis xyz="0 0 1"/>
-      <limit lower="${radians(-180)}" upper="${radians(180)}" effort="0" velocity="${radians(velocities['joint_1'])}"/>
+      <limit lower="${radians(-180)}" upper="${radians(180)}" effort="${limits['joint_1']['effort']}" velocity="${radians(limits['joint_1']['velocity'])}"/>
     </joint>
     <joint name="${prefix}joint_2" type="revolute">
@@ -159,5 +159,5 @@
       <child link="${prefix}link_2"/>
       <axis xyz="0 1 0"/>
-      <limit lower="${radians(-130)}" upper="${radians(80)}" effort="0" velocity="${radians(velocities['joint_2'])}"/>
+      <limit lower="${radians(-130)}" upper="${radians(80)}" effort="${limits['joint_2']['effort']}" velocity="${radians(limits['joint_2']['velocity'])}"/>
     </joint>
     <joint name="${prefix}joint_3" type="revolute">
@@ -166,5 +166,5 @@
       <child link="${prefix}link_3"/>
       <axis xyz="0 -1 0"/>
-      <limit lower="${radians(-107)}" upper="${radians(190)}" effort="0" velocity="${radians(velocities['joint_3'])}"/>
+      <limit lower="${radians(-107)}" upper="${radians(190)}" effort="${limits['joint_3']['effort']}" velocity="${radians(limits['joint_3']['velocity'])}"/>
     </joint>
     <joint name="${prefix}joint_4" type="revolute">
@@ -173,5 +173,5 @@
       <child link="${prefix}link_4"/>
       <axis xyz="0 0 1"/>
-      <limit lower="${radians(-360)}" upper="${radians(360)}" effort="0" velocity="${radians(velocities['joint_4'])}"/>
+      <limit lower="${radians(-360)}" upper="${radians(360)}" effort="${limits['joint_4']['effort']}" velocity="${radians(limits['joint_4']['velocity'])}"/>
     </joint>
     <joint name="${prefix}joint_5" type="revolute">
@@ -180,5 +180,5 @@
       <child link="${prefix}link_5"/>
       <axis xyz="0 -1 0"/>
-      <limit lower="${radians(-130)}" upper="${radians(130)}" effort="0" velocity="${radians(velocities['joint_5'])}"/>
+      <limit lower="${radians(-130)}" upper="${radians(130)}" effort="${limits['joint_5']['effort']}" velocity="${radians(limits['joint_5']['velocity'])}"/>
     </joint>
     <joint name="${prefix}joint_6" type="revolute">
@@ -187,5 +187,5 @@
       <child link="${prefix}link_6"/>
       <axis xyz="0 0 1"/>
-      <limit lower="${radians(-360)}" upper="${radians(360)}" effort="0" velocity="${radians(velocities['joint_6'])}"/>
+      <limit lower="${radians(-360)}" upper="${radians(360)}" effort="${limits['joint_6']['effort']}" velocity="${radians(limits['joint_6']['velocity'])}"/>
     </joint>
     <!--
