Commit message: Change references to all renamed mesh files

File: motoman_gp225_support/urdf/gp225_macro.xacro (robot description, xacro)
@@ -20,11 +20,11 @@
         <visual>
             <geometry>
-                <mesh filename="package://motoman_gp225_support/meshes/gp225/visual/link_1_s.dae"/>
-            </geometry>
-            <xacro:material_yaskawa_blue/>
-        </visual>
-        <collision>
-            <geometry>
-                <mesh filename="package://motoman_gp225_support/meshes/gp225/collision/link_1_s.stl"/>
+                <mesh filename="package://motoman_gp225_support/meshes/gp225/visual/link_1.dae"/>
+            </geometry>
+            <xacro:material_yaskawa_blue/>
+        </visual>
+        <collision>
+            <geometry>
+                <mesh filename="package://motoman_gp225_support/meshes/gp225/collision/link_1.stl"/>
             </geometry>
         </collision>
@@ -33,11 +33,11 @@
         <visual>
             <geometry>
-                <mesh filename="package://motoman_gp225_support/meshes/gp225/visual/link_2_l.dae"/>
-            </geometry>
-            <xacro:material_yaskawa_blue/>
-        </visual>
-        <collision>
-            <geometry>
-                <mesh filename="package://motoman_gp225_support/meshes/gp225/collision/link_2_l.stl"/>
+                <mesh filename="package://motoman_gp225_support/meshes/gp225/visual/link_2.dae"/>
+            </geometry>
+            <xacro:material_yaskawa_blue/>
+        </visual>
+        <collision>
+            <geometry>
+                <mesh filename="package://motoman_gp225_support/meshes/gp225/collision/link_2.stl"/>
             </geometry>
         </collision>
@@ -46,11 +46,11 @@
         <visual>
             <geometry>
-                <mesh filename="package://motoman_gp225_support/meshes/gp225/visual/link_3_u.dae"/>
-            </geometry>
-            <xacro:material_yaskawa_blue/>
-        </visual>
-        <collision>
-            <geometry>
-                <mesh filename="package://motoman_gp225_support/meshes/gp225/collision/link_3_u.stl"/>
+                <mesh filename="package://motoman_gp225_support/meshes/gp225/visual/link_3.dae"/>
+            </geometry>
+            <xacro:material_yaskawa_blue/>
+        </visual>
+        <collision>
+            <geometry>
+                <mesh filename="package://motoman_gp225_support/meshes/gp225/collision/link_3.stl"/>
             </geometry>
         </collision>
@@ -64,11 +64,11 @@
         <visual>
             <geometry>
-                <mesh filename="package://motoman_gp225_support/meshes/gp225/visual/link_4_r.dae"/>
-            </geometry>
-            <xacro:material_yaskawa_blue/>
-        </visual>
-        <collision>
-            <geometry>
-                <mesh filename="package://motoman_gp225_support/meshes/gp225/collision/link_4_r.stl"/>
+                <mesh filename="package://motoman_gp225_support/meshes/gp225/visual/link_4.dae"/>
+            </geometry>
+            <xacro:material_yaskawa_blue/>
+        </visual>
+        <collision>
+            <geometry>
+                <mesh filename="package://motoman_gp225_support/meshes/gp225/collision/link_4.stl"/>
             </geometry>
         </collision>
@@ -77,11 +77,11 @@
         <visual>
             <geometry>
-                <mesh filename="package://motoman_gp225_support/meshes/gp225/visual/link_5_b.dae"/>
-            </geometry>
-            <xacro:material_yaskawa_blue/>
-        </visual>
-        <collision>
-            <geometry>
-                <mesh filename="package://motoman_gp225_support/meshes/gp225/collision/link_5_b.stl"/>
+                <mesh filename="package://motoman_gp225_support/meshes/gp225/visual/link_5.dae"/>
+            </geometry>
+            <xacro:material_yaskawa_blue/>
+        </visual>
+        <collision>
+            <geometry>
+                <mesh filename="package://motoman_gp225_support/meshes/gp225/collision/link_5.stl"/>
             </geometry>
         </collision>
@@ -90,11 +90,11 @@
         <visual>
             <geometry>
-                <mesh filename="package://motoman_gp225_support/meshes/gp225/visual/link_6_t.dae"/>
-            </geometry>
-            <xacro:material_yaskawa_blue/>
-        </visual>
-        <collision>
-            <geometry>
-                <mesh filename="package://motoman_gp225_support/meshes/gp225/collision/link_6_t.stl"/>
+                <mesh filename="package://motoman_gp225_support/meshes/gp225/visual/link_6.dae"/>
+            </geometry>
+            <xacro:material_yaskawa_blue/>
+        </visual>
+        <collision>
+            <geometry>
+                <mesh filename="package://motoman_gp225_support/meshes/gp225/collision/link_6.stl"/>
             </geometry>
         </collision>
@@ -148,11 +148,11 @@
         <visual>
             <geometry>
-                <mesh filename="package://motoman_gp225_support/meshes/gp225/visual/link_1_s_2.dae"/>
-            </geometry>
-            <xacro:material_yaskawa_blue/>
-        </visual>
-        <collision>
-            <geometry>
-                <mesh filename="package://motoman_gp225_support/meshes/gp225/collision/link_1_s_2.stl"/>
+                <mesh filename="package://motoman_gp225_support/meshes/gp225/visual/balancer_1.dae"/>
+            </geometry>
+            <xacro:material_yaskawa_blue/>
+        </visual>
+        <collision>
+            <geometry>
+                <mesh filename="package://motoman_gp225_support/meshes/gp225/collision/balancer_1.stl"/>
             </geometry>
         </collision>
@@ -161,5 +161,5 @@
         <visual>
             <geometry>
-                <mesh filename="package://motoman_gp225_support/meshes/gp225/visual/link_2_l_2.dae"/>
+                <mesh filename="package://motoman_gp225_support/meshes/gp225/visual/balancer_2.dae"/>
             </geometry>
             <xacro:material_yaskawa_blue/>

File: motoman_sia10d_support/urdf/sia10d_macro.xacro (robot description, xacro)
@@ -10,11 +10,11 @@
             <visual>
                 <geometry>
-                    <mesh filename="package://motoman_sia10d_support/meshes/sia10d/visual/MOTOMAN_BASE.stl" />
-                </geometry>
-                <xacro:material_yaskawa_blue/>
-            </visual>
-            <collision>
-                <geometry>
-                    <mesh filename="package://motoman_sia10d_support/meshes/sia10d/collision/MOTOMAN_BASE.stl" />
+                    <mesh filename="package://motoman_sia10d_support/meshes/sia10d/visual/base_link.stl" />
+                </geometry>
+                <xacro:material_yaskawa_blue/>
+            </visual>
+            <collision>
+                <geometry>
+                    <mesh filename="package://motoman_sia10d_support/meshes/sia10d/collision/base_link.stl" />
                 </geometry>
                 <xacro:material_yaskawa_yellow/>
@@ -24,11 +24,11 @@
             <visual>
                 <geometry>
-                    <mesh filename="package://motoman_sia10d_support/meshes/sia10d/visual/MOTOMAN_AXIS_S.stl"/>
-                </geometry>
-                <xacro:material_yaskawa_silver/>
-            </visual>
-            <collision>
-                <geometry>
-                    <mesh filename="package://motoman_sia10d_support/meshes/sia10d/collision/MOTOMAN_AXIS_S.stl" />
+                    <mesh filename="package://motoman_sia10d_support/meshes/sia10d/visual/link_1.stl"/>
+                </geometry>
+                <xacro:material_yaskawa_silver/>
+            </visual>
+            <collision>
+                <geometry>
+                    <mesh filename="package://motoman_sia10d_support/meshes/sia10d/collision/link_1.stl" />
                 </geometry>
                 <xacro:material_yaskawa_yellow/>
@@ -39,5 +39,5 @@
                 <origin rpy="1.57 3.1416 0" xyz="0 0 0"/>
                 <geometry>
-                    <mesh filename="package://motoman_sia10d_support/meshes/sia10d/visual/MOTOMAN_AXIS_L.stl"/>
+                    <mesh filename="package://motoman_sia10d_support/meshes/sia10d/visual/link_2.stl"/>
                 </geometry>
                 <xacro:material_yaskawa_blue/>
@@ -46,5 +46,5 @@
                 <origin rpy="1.57 3.1416 0" xyz="0 0 0"/>
                 <geometry>
-                    <mesh filename="package://motoman_sia10d_support/meshes/sia10d/collision/MOTOMAN_AXIS_L.stl" />
+                    <mesh filename="package://motoman_sia10d_support/meshes/sia10d/collision/link_2.stl" />
                 </geometry>
                 <xacro:material_yaskawa_yellow/>
@@ -55,5 +55,5 @@
                 <origin rpy="0 0 3.1415" xyz="0 0 0"/>
                 <geometry>
-                    <mesh filename="package://motoman_sia10d_support/meshes/sia10d/visual/MOTOMAN_AXIS_E.stl"/>
+                    <mesh filename="package://motoman_sia10d_support/meshes/sia10d/visual/link_3.stl"/>
                 </geometry>
                 <xacro:material_yaskawa_silver/>
@@ -62,5 +62,5 @@
                 <origin rpy="0 0 3.1415" xyz="0 0 0"/>
                 <geometry>
-                    <mesh filename="package://motoman_sia10d_support/meshes/sia10d/collision/MOTOMAN_AXIS_E.stl" />
+                    <mesh filename="package://motoman_sia10d_support/meshes/sia10d/collision/link_3.stl" />
                 </geometry>
                 <xacro:material_yaskawa_yellow/>
@@ -71,5 +71,5 @@
                 <origin rpy="1.57 -3.1415 0" xyz="0 0 0"/>
                 <geometry>
-                    <mesh filename="package://motoman_sia10d_support/meshes/sia10d/visual/MOTOMAN_AXIS_U.stl"/>
+                    <mesh filename="package://motoman_sia10d_support/meshes/sia10d/visual/link_4.stl"/>
                 </geometry>
                 <xacro:material_yaskawa_blue/>
@@ -78,5 +78,5 @@
                 <origin rpy="1.57 -3.1415 0" xyz="0 0 0"/>
                 <geometry>
-                    <mesh filename="package://motoman_sia10d_support/meshes/sia10d/collision/MOTOMAN_AXIS_U.stl" />
+                    <mesh filename="package://motoman_sia10d_support/meshes/sia10d/collision/link_4.stl" />
                 </geometry>
                 <xacro:material_yaskawa_yellow/>
@@ -87,5 +87,5 @@
                 <origin rpy="0 0 3.1416" xyz="0 0 0"/>
                 <geometry>
-                    <mesh filename="package://motoman_sia10d_support/meshes/sia10d/visual/MOTOMAN_AXIS_R.stl"/>
+                    <mesh filename="package://motoman_sia10d_support/meshes/sia10d/visual/link_5.stl"/>
                 </geometry>
                 <xacro:material_yaskawa_silver/>
@@ -94,5 +94,5 @@
                 <origin rpy="0 0 3.1416" xyz="0 0 0"/>
                 <geometry>
-                    <mesh filename="package://motoman_sia10d_support/meshes/sia10d/collision/MOTOMAN_AXIS_R.stl" />
+                    <mesh filename="package://motoman_sia10d_support/meshes/sia10d/collision/link_5.stl" />
                 </geometry>
                 <xacro:material_yaskawa_yellow/>
@@ -103,5 +103,5 @@
                 <origin rpy="-1.57 0 3.1416" xyz="0 0 0"/>
                 <geometry>
-                    <mesh filename="package://motoman_sia10d_support/meshes/sia10d/visual/MOTOMAN_AXIS_B.stl"/>
+                    <mesh filename="package://motoman_sia10d_support/meshes/sia10d/visual/link_6.stl"/>
                 </geometry>
                 <xacro:material_yaskawa_blue/>
@@ -110,5 +110,5 @@
                 <origin rpy="-1.57 0 3.1416" xyz="0 0 0"/>
                 <geometry>
-                    <mesh filename="package://motoman_sia10d_support/meshes/sia10d/collision/MOTOMAN_AXIS_B.stl" />
+                    <mesh filename="package://motoman_sia10d_support/meshes/sia10d/collision/link_6.stl" />
                 </geometry>
                 <xacro:material_yaskawa_yellow/>
@@ -118,11 +118,11 @@
             <visual>
                 <geometry>
-                    <mesh filename="package://motoman_sia10d_support/meshes/sia10d/visual/MOTOMAN_AXIS_T.stl" />
-                </geometry>
-                <xacro:material_yaskawa_silver/>
-            </visual>
-            <collision>
-                <geometry>
-                    <mesh filename="package://motoman_sia10d_support/meshes/sia10d/collision/MOTOMAN_AXIS_T.stl" />
+                    <mesh filename="package://motoman_sia10d_support/meshes/sia10d/visual/link_7.stl" />
+                </geometry>
+                <xacro:material_yaskawa_silver/>
+            </visual>
+            <collision>
+                <geometry>
+                    <mesh filename="package://motoman_sia10d_support/meshes/sia10d/collision/link_7.stl" />
                 </geometry>
                 <xacro:material_yaskawa_yellow/>

File: motoman_sia5d_support/urdf/sia5d_macro.xacro (robot description, xacro)
@@ -8,5 +8,5 @@
       <origin xyz="0 0 0" rpy="0 0 0" />
       <geometry>
-        <mesh filename="package://motoman_sia5d_support/meshes/sia5d/visual/base.dae" />
+        <mesh filename="package://motoman_sia5d_support/meshes/sia5d/visual/base_link.dae" />
       </geometry>
     </visual>
@@ -14,5 +14,5 @@
       <origin xyz="0 0 0" rpy="0 0 0" />
       <geometry>
-        <mesh filename="package://motoman_sia5d_support/meshes/sia5d/collision/base.dae" />
+        <mesh filename="package://motoman_sia5d_support/meshes/sia5d/collision/base_link.dae" />
       </geometry>
     </collision>
@@ -22,5 +22,5 @@
       <origin xyz="0 0 0" rpy="0 0 0" />
       <geometry>
-        <mesh filename="package://motoman_sia5d_support/meshes/sia5d/visual/link_s.dae" />
+        <mesh filename="package://motoman_sia5d_support/meshes/sia5d/visual/link_1.dae" />
       </geometry>
     </visual>
@@ -28,5 +28,5 @@
       <origin xyz="0 0 0" rpy="0 0 0" />
       <geometry>
-        <mesh filename="package://motoman_sia5d_support/meshes/sia5d/collision/link_s.dae" />
+        <mesh filename="package://motoman_sia5d_support/meshes/sia5d/collision/link_1.dae" />
       </geometry>
     </collision>
@@ -43,5 +43,5 @@
       <origin xyz="0 0 0" rpy="0 0 0" />
       <geometry>
-        <mesh filename="package://motoman_sia5d_support/meshes/sia5d/visual/link_l.dae" />
+        <mesh filename="package://motoman_sia5d_support/meshes/sia5d/visual/link_2.dae" />
       </geometry>
     </visual>
@@ -49,5 +49,5 @@
       <origin xyz="0 0 0" rpy="0 0 0" />
       <geometry>
-        <mesh filename="package://motoman_sia5d_support/meshes/sia5d/collision/link_l.dae" />
+        <mesh filename="package://motoman_sia5d_support/meshes/sia5d/collision/link_2.dae" />
       </geometry>
     </collision>
@@ -64,5 +64,5 @@
       <origin xyz="0 0 0" rpy="0 0 0" />
       <geometry>
-        <mesh filename="package://motoman_sia5d_support/meshes/sia5d/visual/link_e.dae" />
+        <mesh filename="package://motoman_sia5d_support/meshes/sia5d/visual/link_3.dae" />
       </geometry>
     </visual>
@@ -70,5 +70,5 @@
       <origin xyz="0 0 0" rpy="0 0 0" />
       <geometry>
-        <mesh filename="package://motoman_sia5d_support/meshes/sia5d/collision/link_e.dae" />
+        <mesh filename="package://motoman_sia5d_support/meshes/sia5d/collision/link_3.dae" />
       </geometry>
     </collision>
@@ -85,5 +85,5 @@
       <origin xyz="0 0 0" rpy="0 0 0" />
       <geometry>
-        <mesh filename="package://motoman_sia5d_support/meshes/sia5d/visual/link_u.dae" />
+        <mesh filename="package://motoman_sia5d_support/meshes/sia5d/visual/link_4.dae" />
       </geometry>
     </visual>
@@ -91,5 +91,5 @@
       <origin xyz="0 0 0" rpy="0 0 0" />
       <geometry>
-        <mesh filename="package://motoman_sia5d_support/meshes/sia5d/collision/link_u.dae" />
+        <mesh filename="package://motoman_sia5d_support/meshes/sia5d/collision/link_4.dae" />
       </geometry>
     </collision>
@@ -106,5 +106,5 @@
       <origin xyz="0 0 0" rpy="0 0 0" />
       <geometry>
-        <mesh filename="package://motoman_sia5d_support/meshes/sia5d/visual/link_r.dae" />
+        <mesh filename="package://motoman_sia5d_support/meshes/sia5d/visual/link_5.dae" />
       </geometry>
     </visual>
@@ -112,5 +112,5 @@
       <origin xyz="0 0 0" rpy="0 0 0" />
       <geometry>
-        <mesh filename="package://motoman_sia5d_support/meshes/sia5d/collision/link_r.dae" />
+        <mesh filename="package://motoman_sia5d_support/meshes/sia5d/collision/link_5.dae" />
       </geometry>
     </collision>
@@ -127,5 +127,5 @@
       <origin xyz="0 0 0" rpy="0 0 0" />
       <geometry>
-        <mesh filename="package://motoman_sia5d_support/meshes/sia5d/visual/link_b.dae" />
+        <mesh filename="package://motoman_sia5d_support/meshes/sia5d/visual/link_6.dae" />
       </geometry>
     </visual>
@@ -133,5 +133,5 @@
       <origin xyz="0 0 0" rpy="0 0 0" />
       <geometry>
-        <mesh filename="package://motoman_sia5d_support/meshes/sia5d/collision/link_b.dae" />
+        <mesh filename="package://motoman_sia5d_support/meshes/sia5d/collision/link_6.dae" />
       </geometry>
     </collision>
@@ -148,5 +148,5 @@
       <origin xyz="0 0 0" rpy="0 0 0" />
       <geometry>
-        <mesh filename="package://motoman_sia5d_support/meshes/sia5d/visual/link_t.dae" />
+        <mesh filename="package://motoman_sia5d_support/meshes/sia5d/visual/link_7.dae" />
       </geometry>
     </visual>
@@ -154,5 +154,5 @@
       <origin xyz="0 0 0" rpy="0 0 0" />
       <geometry>
-        <mesh filename="package://motoman_sia5d_support/meshes/sia5d/collision/link_t.dae" />
+        <mesh filename="package://motoman_sia5d_support/meshes/sia5d/collision/link_7.dae" />
       </geometry>
     </collision>
