Commit message: Update link and joint names in `xacro` files

File: motoman_gp225_support/urdf/gp225_macro.xacro (robot description, xacro)
@@ -17,5 +17,5 @@
         </collision>
     </link>
-    <link name="${prefix}link_1_s">
+    <link name="${prefix}link_1">
         <visual>
             <geometry>
@@ -30,5 +30,5 @@
         </collision>
     </link>
-    <link name="${prefix}link_2_l">
+    <link name="${prefix}link_2">
         <visual>
             <geometry>
@@ -43,5 +43,5 @@
         </collision>
     </link>
-    <link name="${prefix}link_3_u">
+    <link name="${prefix}link_3">
         <visual>
             <geometry>
@@ -61,5 +61,5 @@
         </collision>
     </link>
-    <link name="${prefix}link_4_r">
+    <link name="${prefix}link_4">
         <visual>
             <geometry>
@@ -74,5 +74,5 @@
         </collision>
     </link>
-    <link name="${prefix}link_5_b">
+    <link name="${prefix}link_5">
         <visual>
             <geometry>
@@ -87,5 +87,5 @@
         </collision>
     </link>
-    <link name="${prefix}link_6_t">
+    <link name="${prefix}link_6">
         <visual>
             <geometry>
@@ -102,42 +102,42 @@
     <!-- end of link list -->
     <!-- joint list -->
-    <joint name="${prefix}joint_1_s" type="revolute">
+    <joint name="${prefix}joint_1" type="revolute">
         <parent link="${prefix}base_link"/>
-        <child link="${prefix}link_1_s"/>
+        <child link="${prefix}link_1"/>
         <origin xyz="0 0 0.650" rpy="0 0 0" />
         <axis xyz="0 0 1" />
         <limit lower="${radians(-180)}" upper="${radians(180)}" effort="7845.3" velocity="${radians(120)}"/>
     </joint>
-    <joint name="${prefix}joint_2_l" type="revolute">
-        <parent link="${prefix}link_1_s"/>
-        <child link="${prefix}link_2_l"/>
+    <joint name="${prefix}joint_2" type="revolute">
+        <parent link="${prefix}link_1"/>
+        <child link="${prefix}link_2"/>
         <origin xyz="0.325 0 0" rpy="0 0 0" />
         <axis xyz="0 1 0" />
         <limit lower="${radians(-60)}" upper="${radians(76)}" effort="11522.8" velocity="${radians(97)}"/>
     </joint>
-    <joint name="${prefix}joint_3_u" type="revolute">
-        <parent link="${prefix}link_2_l"/>
-        <child link="${prefix}link_3_u"/>
+    <joint name="${prefix}joint_3" type="revolute">
+        <parent link="${prefix}link_2"/>
+        <child link="${prefix}link_3"/>
         <origin xyz="0 0 1.150" rpy="0 0 0" />
         <axis xyz="0 -1 0" />
         <limit lower="${radians(-86)}" upper="${radians(90)}" effort="12258.3" velocity="${radians(115)}"/>
     </joint>
-    <joint name="${prefix}joint_4_r" type="revolute">
-        <parent link="${prefix}link_3_u"/>
-        <child link="${prefix}link_4_r"/>
+    <joint name="${prefix}joint_4" type="revolute">
+        <parent link="${prefix}link_3"/>
+        <child link="${prefix}link_4"/>
         <origin xyz="1.225 0 0.300" rpy="0 0 0" />
         <axis xyz="-1 0 0" />
         <limit lower="${radians(-360)}" upper="${radians(360)}" effort="3064.5" velocity="${radians(145)}"/>
     </joint>
-    <joint name="${prefix}joint_5_b" type="revolute">
-        <parent link="${prefix}link_4_r"/>
-        <child link="${prefix}link_5_b"/>
+    <joint name="${prefix}joint_5" type="revolute">
+        <parent link="${prefix}link_4"/>
+        <child link="${prefix}link_5"/>
         <origin xyz="0 0 0" rpy="0 0 0" />
         <axis xyz="0 -1 0" />
         <limit lower="${radians(-125)}" upper="${radians(125)}" effort="3432.3" velocity="${radians(145)}"/>
     </joint>
-    <joint name="${prefix}joint_6_t" type="revolute">
-        <parent link="${prefix}link_5_b"/>
-        <child link="${prefix}link_6_t"/>
+    <joint name="${prefix}joint_6" type="revolute">
+        <parent link="${prefix}link_5"/>
+        <child link="${prefix}link_6"/>
         <origin xyz="0 0 0" rpy="0 0 0" />
         <axis xyz="-1 0 0" />
@@ -145,41 +145,41 @@
     </joint>
     <!-- balancer -->
-    <link name="${prefix}link_1_s_2">
-        <visual>
-            <geometry>
-                <mesh filename="package://motoman_gp225_support/meshes/gp225/visual/balancer_1.dae"/>
-            </geometry>
-            <xacro:material_yaskawa_blue/>
-        </visual>
-        <collision>
-            <geometry>
-                <mesh filename="package://motoman_gp225_support/meshes/gp225/collision/balancer_1.stl"/>
-            </geometry>
-        </collision>
-    </link>
-    <link name="${prefix}link_2_l_2">
-        <visual>
-            <geometry>
-                <mesh filename="package://motoman_gp225_support/meshes/gp225/visual/balancer_2.dae"/>
-            </geometry>
-            <xacro:material_yaskawa_blue/>
-        </visual>
-        <!-- collision mesh is fully contained within link_2_l -->
-    </link>
-    <joint name="${prefix}joint_1_s_2" type="revolute">
-        <parent link="${prefix}link_1_s"/>
-        <child link="${prefix}link_1_s_2"/>
+    <link name="${prefix}balancer_link_1">
+        <visual>
+            <geometry>
+                <mesh filename="package://motoman_gp225_support/meshes/gp225/visual/balancer_link_1.dae"/>
+            </geometry>
+            <xacro:material_yaskawa_blue/>
+        </visual>
+        <collision>
+            <geometry>
+                <mesh filename="package://motoman_gp225_support/meshes/gp225/collision/balancer_link_1.stl"/>
+            </geometry>
+        </collision>
+    </link>
+    <link name="${prefix}balancer_link_2">
+        <visual>
+            <geometry>
+                <mesh filename="package://motoman_gp225_support/meshes/gp225/visual/balancer_link_2.dae"/>
+            </geometry>
+            <xacro:material_yaskawa_blue/>
+        </visual>
+        <!-- collision mesh is fully contained within link_2 -->
+    </link>
+    <joint name="${prefix}balancer_joint_1" type="revolute">
+        <parent link="${prefix}link_1"/>
+        <child link="${prefix}balancer_link_1"/>
         <origin xyz="0.3989 0 -0.2576" rpy="0 0 0" />
         <axis xyz="0 1 0" />
         <limit lower="${radians(-60)}" upper="${radians(76)}" effort="11522.8" velocity="${radians(97)}"/>
-        <mimic joint="${prefix}joint_2_l" multiplier="0.7634"/>
-    </joint>
-    <joint name="${prefix}joint_2_l_2" type="revolute">
-        <parent link="${prefix}link_2_l"/>
-        <child link="${prefix}link_2_l_2"/>
+        <mimic joint="${prefix}joint_2" multiplier="0.7634"/>
+    </joint>
+    <joint name="${prefix}balancer_joint_2" type="revolute">
+        <parent link="${prefix}link_2"/>
+        <child link="${prefix}balancer_link_2"/>
         <origin xyz="0 0 0.720" rpy="0 0 0" />
         <axis xyz="0 1 0" />
         <limit lower="${radians(-60)}" upper="${radians(76)}" effort="11522.8" velocity="${radians(97)}"/>
-        <mimic joint="${prefix}joint_2_l" multiplier="-0.2366"/>
+        <mimic joint="${prefix}joint_2" multiplier="-0.2366"/>
     </joint>
     <!-- end of joint list -->
@@ -193,7 +193,7 @@
     <!-- ROS-Industrial 'flange' frame: attachment point for EEF models -->
     <link name="${prefix}flange" />
-    <joint name="${prefix}joint_6_t-flange" type="fixed">
+    <joint name="${prefix}joint_6-flange" type="fixed">
         <origin xyz="0.250 0 0" rpy="0 0 0" />
-        <parent link="${prefix}link_6_t" />
+        <parent link="${prefix}link_6" />
         <child link="${prefix}flange" />
     </joint>

File: motoman_sia10d_support/urdf/sia10d_macro.xacro (robot description, xacro)
@@ -21,5 +21,5 @@
             </collision>
         </link>
-        <link name="${prefix}link_s">
+        <link name="${prefix}link_1">
             <visual>
                 <geometry>
@@ -35,5 +35,5 @@
             </collision>
         </link>
-        <link name="${prefix}link_l">
+        <link name="${prefix}link_2">
             <visual>
                 <origin rpy="1.57 3.1416 0" xyz="0 0 0"/>
@@ -51,5 +51,5 @@
             </collision>
         </link>
-        <link name="${prefix}link_e">
+        <link name="${prefix}link_3">
             <visual>
                 <origin rpy="0 0 3.1415" xyz="0 0 0"/>
@@ -67,5 +67,5 @@
             </collision>
         </link>
-        <link name="${prefix}link_u">
+        <link name="${prefix}link_4">
             <visual>
                 <origin rpy="1.57 -3.1415 0" xyz="0 0 0"/>
@@ -83,5 +83,5 @@
             </collision>
         </link>
-        <link name="${prefix}link_r">
+        <link name="${prefix}link_5">
             <visual>
                 <origin rpy="0 0 3.1416" xyz="0 0 0"/>
@@ -99,5 +99,5 @@
             </collision>
         </link>
-        <link name="${prefix}link_b">
+        <link name="${prefix}link_6">
             <visual>
                 <origin rpy="-1.57 0 3.1416" xyz="0 0 0"/>
@@ -115,5 +115,5 @@
             </collision>
         </link>
-        <link name="${prefix}link_t">
+        <link name="${prefix}link_7">
             <visual>
                 <geometry>
@@ -136,49 +136,49 @@
             <child link="base_link"/>
         </joint>
-        <joint name="${prefix}joint_s" type="revolute">
+        <joint name="${prefix}joint_1" type="revolute">
             <parent link="${prefix}base_link"/>
-            <child link="${prefix}link_s"/>
+            <child link="${prefix}link_1"/>
             <origin xyz="0 0 0.36" rpy="0 0 0"/>
             <axis xyz="0 0 1" />
             <limit lower="-3.1415" upper="3.1415" effort="100" velocity="2.9670" />
         </joint>
-        <joint name="${prefix}joint_l" type="revolute">
-            <parent link="${prefix}link_s"/>
-            <child link="${prefix}link_l"/>
+        <joint name="${prefix}joint_2" type="revolute">
+            <parent link="${prefix}link_1"/>
+            <child link="${prefix}link_2"/>
             <origin xyz="0 0 0" rpy="0 0 0"/>
             <axis xyz="0 1 0" />
             <limit lower="-1.9198" upper="1.9198" effort="100" velocity="2.9670" />
         </joint>
-        <joint name="${prefix}joint_e" type="revolute">
-            <parent link="${prefix}link_l"/>
-            <child link="${prefix}link_e"/>
+        <joint name="${prefix}joint_3" type="revolute">
+            <parent link="${prefix}link_2"/>
+            <child link="${prefix}link_3"/>
             <origin xyz="0 0 0.36" rpy="0 0 0"/>
             <axis xyz="0 0 1" />
             <limit lower="-2.9670" upper="2.9670" effort="100" velocity="2.9670" />
         </joint>
-        <joint name="${prefix}joint_u" type="revolute">
-            <parent link="${prefix}link_e"/>
-            <child link="${prefix}link_u"/>
+        <joint name="${prefix}joint_4" type="revolute">
+            <parent link="${prefix}link_3"/>
+            <child link="${prefix}link_4"/>
             <origin xyz="0 0 0" rpy="0 0 0"/>
             <axis xyz="0 -1 0" />
             <limit lower="-2.3561" upper="2.3561" effort="100" velocity="2.9670" />
         </joint>
-        <joint name="${prefix}joint_r" type="revolute">
-            <parent link="${prefix}link_u"/>
-            <child link="${prefix}link_r"/>
+        <joint name="${prefix}joint_5" type="revolute">
+            <parent link="${prefix}link_4"/>
+            <child link="${prefix}link_5"/>
             <origin xyz="0 0 0.360" rpy="0 0 0"/>
             <axis xyz="0 0 -1" />
             <limit lower="-3.1415" upper="3.1415" effort="100" velocity="3.4906" />
         </joint>
-        <joint name="${prefix}joint_b" type="revolute">
-            <parent link="${prefix}link_r"/>
-            <child link="${prefix}link_b"/>
+        <joint name="${prefix}joint_6" type="revolute">
+            <parent link="${prefix}link_5"/>
+            <child link="${prefix}link_6"/>
             <origin xyz="0 0 0" rpy="0 0 0"/>
             <axis xyz="0 -1 0" />
             <limit lower="-1.9198" upper="1.9198" effort="100" velocity="3.4906" />
         </joint>
-        <joint name="${prefix}joint_t" type="revolute">
-            <parent link="${prefix}link_b"/>
-            <child link="${prefix}link_t"/>
+        <joint name="${prefix}joint_7" type="revolute">
+            <parent link="${prefix}link_6"/>
+            <child link="${prefix}link_7"/>
             <origin xyz="0 0 0.155" rpy="0 0 0"/>
             <axis xyz="0 0 -1" />
@@ -195,7 +195,7 @@
         <!-- ROS-Industrial 'flange' frame: attachment point for EEF models -->
         <link name="${prefix}flange"/>
-        <joint name="${prefix}joint_t-flange" type="fixed">
+        <joint name="${prefix}joint_7-flange" type="fixed">
             <origin xyz="0 0 0" rpy="0 -1.57079632679 0"/>
-            <parent link="${prefix}link_t"/>
+            <parent link="${prefix}link_7"/>
             <child link="${prefix}flange"/>
         </joint>

File: motoman_sia5d_support/urdf/sia5d_macro.xacro (robot description, xacro)
@@ -18,5 +18,5 @@
     </collision>
   </link>
-  <link name="${prefix}link_s">
+  <link name="${prefix}link_1">
     <visual>
       <origin xyz="0 0 0" rpy="0 0 0" />
@@ -32,12 +32,12 @@
     </collision>
   </link>
-  <joint name="${prefix}joint_s" type="revolute">
+  <joint name="${prefix}joint_1" type="revolute">
     <origin xyz="0 0 0.31" rpy="0 0 0" /> <!--r=${90*deg}-->
     <parent link="${prefix}base_link" />
-    <child link="${prefix}link_s" />
+    <child link="${prefix}link_1" />
     <axis xyz="0 0 1" />
     <limit lower="${-180*deg}" upper="${180*deg}" effort="0" velocity="${200*deg}" />
   </joint>
-  <link name="${prefix}link_l">
+  <link name="${prefix}link_2">
     <visual>
       <origin xyz="0 0 0" rpy="0 0 0" />
@@ -53,12 +53,12 @@
     </collision>
   </link>
-  <joint name="${prefix}joint_l" type="revolute">
+  <joint name="${prefix}joint_2" type="revolute">
     <origin xyz="0 0 0" rpy="0 0 0" />
-    <parent link="${prefix}link_s" />
-    <child link="${prefix}link_l" />
+    <parent link="${prefix}link_1" />
+    <child link="${prefix}link_2" />
     <axis xyz="0 1 0" />
     <limit lower="${-110*deg}" upper="${110*deg}" effort="0" velocity="${200*deg}" />
   </joint>
-  <link name="${prefix}link_e">
+  <link name="${prefix}link_3">
     <visual>
       <origin xyz="0 0 0" rpy="0 0 0" />
@@ -74,12 +74,12 @@
     </collision>
   </link>
-  <joint name="${prefix}joint_e" type="revolute">
+  <joint name="${prefix}joint_3" type="revolute">
     <origin xyz="0 0 0.27" rpy="0 0 0" />
-    <parent link="${prefix}link_l" />
-    <child link="${prefix}link_e" />
+    <parent link="${prefix}link_2" />
+    <child link="${prefix}link_3" />
     <axis xyz="0 0 1" />
     <limit lower="${-170*deg}" upper="${170*deg}" effort="0" velocity="${200*deg}" />
   </joint>
-  <link name="${prefix}link_u">
+  <link name="${prefix}link_4">
     <visual>
       <origin xyz="0 0 0" rpy="0 0 0" />
@@ -95,12 +95,12 @@
     </collision>
   </link>
-  <joint name="${prefix}joint_u" type="revolute">
+  <joint name="${prefix}joint_4" type="revolute">
     <origin xyz="0.085 0 0" rpy="0 0 0" />
-    <parent link="${prefix}link_e" />
-    <child link="${prefix}link_u" />
+    <parent link="${prefix}link_3" />
+    <child link="${prefix}link_4" />
     <axis xyz="0 -1 0" />
     <limit lower="${-90*deg}" upper="${115*deg}" effort="0"  velocity="${200*deg}" />
   </joint>
-  <link name="${prefix}link_r">
+  <link name="${prefix}link_5">
     <visual>
       <origin xyz="0 0 0" rpy="0 0 0" />
@@ -116,12 +116,12 @@
     </collision>
   </link>
-  <joint name="${prefix}joint_r" type="revolute">
+  <joint name="${prefix}joint_5" type="revolute">
     <origin xyz="0.27 0 0.06" rpy="0 0 0" />
-    <parent link="${prefix}link_u" />
-    <child link="${prefix}link_r" />
+    <parent link="${prefix}link_4" />
+    <child link="${prefix}link_5" />
     <axis xyz="-1 0 0" />
     <limit lower="${-90*deg}" upper="${90*deg}" effort="0" velocity="${200*deg}" />
   </joint>
-  <link name="${prefix}link_b">
+  <link name="${prefix}link_6">
     <visual>
       <origin xyz="0 0 0" rpy="0 0 0" />
@@ -137,12 +137,12 @@
     </collision>
   </link>
-  <joint name="${prefix}joint_b" type="revolute">
+  <joint name="${prefix}joint_6" type="revolute">
     <origin xyz="0 0 0" rpy="0 0 0" />
-    <parent link="${prefix}link_r" />
-    <child link="${prefix}link_b" />
+    <parent link="${prefix}link_5" />
+    <child link="${prefix}link_6" />
     <axis xyz="0 -1 0" />
     <limit lower="${-110*deg}" upper="${110*deg}" effort="0" velocity="${230*deg}" />
   </joint>
-  <link name="${prefix}link_t">
+  <link name="${prefix}link_7">
     <visual>
       <origin xyz="0 0 0" rpy="0 0 0" />
@@ -158,8 +158,8 @@
     </collision>
   </link>
-  <joint name="${prefix}joint_t" type="revolute">
+  <joint name="${prefix}joint_7" type="revolute">
     <origin xyz="0.134 0 0" rpy="0 0 0" />
-    <parent link="${prefix}link_b" />
-    <child link="${prefix}link_t" />
+    <parent link="${prefix}link_6" />
+    <child link="${prefix}link_7" />
     <axis xyz="-1 0 0" />
     <limit lower="${-90*deg}" upper="${90*deg}" effort="0" velocity="${350*deg}" />
@@ -175,7 +175,7 @@
   <!-- ROS-Industrial 'flange' frame: attachment point for EEF models -->
   <link name="${prefix}flange"/>
-  <joint name="${prefix}joint_t-flange" type="fixed">
+  <joint name="${prefix}joint_7-flange" type="fixed">
     <origin xyz="0.011 0 0" rpy="0 0 0"/>
-    <parent link="${prefix}link_t"/>
+    <parent link="${prefix}link_7"/>
     <child link="${prefix}flange"/>
   </joint>

Commit message: Fixup

File: motoman_gp225_support/urdf/gp225_macro.xacro (robot description, xacro)
@@ -140,21 +140,21 @@
     </joint>
     <!-- balancer -->
-    <link name="${prefix}balancer_1">
-        <visual>
-            <geometry>
-                <mesh filename="package://motoman_gp225_support/meshes/gp225/visual/balancer_1.dae"/>
-            </geometry>
-            <xacro:material_yaskawa_blue/>
-        </visual>
-        <collision>
-            <geometry>
-                <mesh filename="package://motoman_gp225_support/meshes/gp225/collision/balancer_1.stl"/>
-            </geometry>
-        </collision>
-    </link>
-    <link name="${prefix}balancer_2">
-        <visual>
-            <geometry>
-                <mesh filename="package://motoman_gp225_support/meshes/gp225/visual/balancer_2.dae"/>
+    <link name="${prefix}balancer_link_1">
+        <visual>
+            <geometry>
+                <mesh filename="package://motoman_gp225_support/meshes/gp225/visual/balancer_link_1.dae"/>
+            </geometry>
+            <xacro:material_yaskawa_blue/>
+        </visual>
+        <collision>
+            <geometry>
+                <mesh filename="package://motoman_gp225_support/meshes/gp225/collision/balancer_link_1.stl"/>
+            </geometry>
+        </collision>
+    </link>
+    <link name="${prefix}balancer_link_2">
+        <visual>
+            <geometry>
+                <mesh filename="package://motoman_gp225_support/meshes/gp225/visual/balancer_link_2.dae"/>
             </geometry>
             <xacro:material_yaskawa_blue/>
@@ -164,5 +164,5 @@
     <joint name="${prefix}balancer_joint_1" type="revolute">
         <parent link="${prefix}link_1"/>
-        <child link="${prefix}balancer_1"/>
+        <child link="${prefix}balancer_link_1"/>
         <origin xyz="0.3989 0 -0.2576" rpy="0 0 0" />
         <axis xyz="0 1 0" />
@@ -172,5 +172,5 @@
     <joint name="${prefix}balancer_joint_2" type="revolute">
         <parent link="${prefix}link_2"/>
-        <child link="${prefix}balancer_2"/>
+        <child link="${prefix}balancer_link_2"/>
         <origin xyz="0 0 0.720" rpy="0 0 0" />
         <axis xyz="0 1 0" />

Commit message: Separated GP225 link 3 collision mesh into 2 convex hulls

File: motoman_gp225_support/urdf/gp225_macro.xacro (robot description, xacro)
@@ -53,4 +53,9 @@
             <geometry>
                 <mesh filename="package://motoman_gp225_support/meshes/gp225/collision/link_3_u.stl"/>
+            </geometry>
+        </collision>
+        <collision>
+            <geometry>
+                <mesh filename="package://motoman_gp225_support/meshes/gp225/collision/link_3_u_2.stl"/>
             </geometry>
         </collision>
