Commit message: move '-' inside of 'radians(...)'

File: motoman_mh5_support/urdf/mh5_macro.xacro (robot description, xacro)
@@ -118,5 +118,5 @@
       <origin xyz="0 0 0.330" rpy="0 0 0"/>
       <axis xyz="0 0 1" />
-      <limit lower="-${radians(170)}" upper="${radians(170)}" effort="215.6" velocity="${radians(376)}" />
+      <limit lower="${radians(-170)}" upper="${radians(170)}" effort="215.6" velocity="${radians(376)}" />
     </joint>
     <joint name="${prefix}joint_2" type="revolute">
@@ -125,5 +125,5 @@
       <origin xyz="0.0880 0 0.00" rpy="0 0 0"/>
       <axis xyz="0 1 0" />
-      <limit lower="-${radians(65)}" upper="${radians(150)}" effort="176.4" velocity="${radians(350)}" />
+      <limit lower="${radians(-65)}" upper="${radians(150)}" effort="176.4" velocity="${radians(350)}" />
     </joint>
     <joint name="${prefix}joint_3" type="revolute">
@@ -132,5 +132,5 @@
       <origin xyz="0 0 0.310" rpy="0 0 0"/>
       <axis xyz="0 -1 0" />
-      <limit lower="-${radians(70)}" upper="${radians(190)}" effort="76.8" velocity="${radians(400)}" />
+      <limit lower="${radians(-70)}" upper="${radians(190)}" effort="76.8" velocity="${radians(400)}" />
     </joint>
     <joint name="${prefix}joint_4" type="revolute">
@@ -139,5 +139,5 @@
       <origin xyz="0 0 0.040" rpy="0 0 0"/>
       <axis xyz="-1 0 0" />
-      <limit lower="-${radians(190)}" upper="${radians(190)}" effort="44.7" velocity="${radians(450)}" />
+      <limit lower="${radians(-190)}" upper="${radians(190)}" effort="44.7" velocity="${radians(450)}" />
     </joint>
     <joint name="${prefix}joint_5" type="revolute">
@@ -146,5 +146,5 @@
       <origin xyz="0.305 0 0" rpy="0 0 0"/>
       <axis xyz="0 -1 0" />
-      <limit lower="-${radians(135)}" upper="${radians(135)}" effort="18.0" velocity="${radians(450)}" />
+      <limit lower="${radians(-135)}" upper="${radians(135)}" effort="18.0" velocity="${radians(450)}" />
     </joint>
     <joint name="${prefix}joint_6" type="revolute">
@@ -153,5 +153,5 @@
       <origin xyz="0.080 0 0" rpy="0 0 0"/>
       <axis xyz="-1 0 0" />
-      <limit lower="-${radians(360)}" upper="${radians(360)}" effort="18.0" velocity="${radians(720)}" />
+      <limit lower="${radians(-360)}" upper="${radians(360)}" effort="18.0" velocity="${radians(720)}" />
     </joint>
     <!-- end of joint list -->

File: motoman_mh5_support/urdf/mh5l_macro.xacro (robot description, xacro)
@@ -116,12 +116,12 @@
       <origin xyz="0 0 0.330" rpy="0 0 0"/>
       <axis xyz="0 0 1" />
-      <limit lower="-${radians(170)}" upper="${radians(170)}" effort="303.8" velocity="${radians(270)}" />
+      <limit lower="${radians(-170)}" upper="${radians(170)}" effort="303.8" velocity="${radians(270)}" />
     </joint>
     <joint name="${prefix}joint_2" type="revolute">
       <parent link="${prefix}link_1"/>
       <child link="${prefix}link_2"/>
-      <origin xyz="0.0880 0 0.00" rpy="0 0 0"/>
+      <origin xyz="0.088 0 0" rpy="0 0 0"/>
       <axis xyz="0 1 0" />
-      <limit lower="-${radians(65)}" upper="${radians(150)}" effort="205.8" velocity="${radians(280)}" />
+      <limit lower="${radians(-65)}" upper="${radians(150)}" effort="205.8" velocity="${radians(280)}" />
     </joint>
     <joint name="${prefix}joint_3" type="revolute">
@@ -130,5 +130,5 @@
       <origin xyz="0 0 0.400" rpy="0 0 0"/>
       <axis xyz="0 -1 0" />
-      <limit lower="-${radians(70)}" upper="${radians(190)}" effort="85.5" velocity="${radians(300)}" />
+      <limit lower="${radians(-70)}" upper="${radians(190)}" effort="85.5" velocity="${radians(300)}" />
     </joint>
     <joint name="${prefix}joint_4" type="revolute">
@@ -137,5 +137,5 @@
       <origin xyz="0 0 0.040" rpy="0 0 0"/>
       <axis xyz="-1 0 0" />
-      <limit lower="-${radians(190)}" upper="${radians(190)}" effort="44.7" velocity="${radians(450)}" />
+      <limit lower="${radians(-190)}" upper="${radians(190)}" effort="44.7" velocity="${radians(450)}" />
     </joint>
     <joint name="${prefix}joint_5" type="revolute">
@@ -144,5 +144,5 @@
       <origin xyz="0.405 0 0" rpy="0 0 0"/>
       <axis xyz="0 -1 0" />
-      <limit lower="-${radians(135)}" upper="${radians(135)}" effort="18.0" velocity="${radians(450)}" />
+      <limit lower="${radians(-135)}" upper="${radians(135)}" effort="18.0" velocity="${radians(450)}" />
     </joint>
     <joint name="${prefix}joint_6" type="revolute">
@@ -151,5 +151,5 @@
       <origin xyz="0.080 0 0" rpy="0 0 0"/>
       <axis xyz="-1 0 0" />
-      <limit lower="-${radians(360)}" upper="${radians(360)}" effort="18.0" velocity="${radians(720)}" />
+      <limit lower="${radians(-360)}" upper="${radians(360)}" effort="18.0" velocity="${radians(720)}" />
     </joint>
     <!-- end of joint list -->
