Commit message: remove many unnecessary trailing zeros

File: motoman_gp20hl_support/urdf/gp20hl_macro.xacro (robot description, xacro)
@@ -102,5 +102,5 @@
       <origin xyz="0 0 0.540" rpy="0 0 0" />
       <axis xyz="0 0 1" />
-      <limit lower="${radians(-180)}" upper="${radians(180)}" effort="5516.2" velocity="${radians(180.0)}"/>
+      <limit lower="${radians(-180)}" upper="${radians(180)}" effort="5516.2" velocity="${radians(180)}"/>
     </joint>
     <joint name="${prefix}joint_2" type="revolute">
@@ -109,5 +109,5 @@
       <origin xyz="0.145 0 0" rpy="0 0 0" />
       <axis xyz="0 1 0" />
-      <limit lower="${radians(-90)}" upper="${radians(135)}" effort="7060.7" velocity="${radians(180.0)}"/>
+      <limit lower="${radians(-90)}" upper="${radians(135)}" effort="7060.7" velocity="${radians(180)}"/>
     </joint>
     <joint name="${prefix}joint_3" type="revolute">
@@ -116,5 +116,5 @@
       <origin xyz="0 0 1.150" rpy="0 0 0" />
       <axis xyz="0 -1 0" />
-      <limit lower="${radians(-80)}" upper="${radians(206)}" effort="3089.0" velocity="${radians(180.0)}"/>
+      <limit lower="${radians(-80)}" upper="${radians(206)}" effort="3089.0" velocity="${radians(180)}"/>
     </joint>
     <joint name="${prefix}joint_4" type="revolute">

File: motoman_gp215_support/urdf/gp215_macro.xacro (robot description, xacro)
@@ -102,5 +102,5 @@
       <origin xyz="0 0 0.650" rpy="0 0 0" />
       <axis xyz="0 0 1" />
-      <limit lower="${radians(-180)}" upper="${radians(180)}" effort="9316.2" velocity="${radians(100.0)}"/>
+      <limit lower="${radians(-180)}" upper="${radians(180)}" effort="9316.2" velocity="${radians(100)}"/>
     </joint>
     <joint name="${prefix}joint_2" type="revolute">
@@ -109,5 +109,5 @@
       <origin xyz="0.285 0 0" rpy="0 0 0" />
       <axis xyz="0 1 0" />
-      <limit lower="${radians(-60)}" upper="${radians(76)}" effort="10591.1" velocity="${radians(90.0)}"/>
+      <limit lower="${radians(-60)}" upper="${radians(76)}" effort="10591.1" velocity="${radians(90)}"/>
     </joint>
     <joint name="${prefix}joint_3" type="revolute">
@@ -116,5 +116,5 @@
       <origin xyz="0 0 1.150" rpy="0 0 0" />
       <axis xyz="0 -1 0" />
-      <limit lower="${radians(-77.8)}" upper="${radians(197)}" effort="9929.2" velocity="${radians(97.0)}"/>
+      <limit lower="${radians(-77.8)}" upper="${radians(197)}" effort="9929.2" velocity="${radians(97)}"/>
     </joint>
     <joint name="${prefix}joint_4" type="revolute">

File: motoman_gp250_support/urdf/gp250_macro.xacro (robot description, xacro)
@@ -102,5 +102,5 @@
       <origin xyz="0 0 0.650" rpy="0 0 0" />
       <axis xyz="0 0 1" />
-      <limit lower="${radians(-180)}" upper="${radians(180)}" effort="9316.2" velocity="${radians(100.0)}"/>
+      <limit lower="${radians(-180)}" upper="${radians(180)}" effort="9316.2" velocity="${radians(100)}"/>
     </joint>
     <joint name="${prefix}joint_2" type="revolute">
@@ -109,5 +109,5 @@
       <origin xyz="0.285 0 0" rpy="0 0 0" />
       <axis xyz="0 1 0" />
-      <limit lower="${radians(-60)}" upper="${radians(76)}" effort="10591.1" velocity="${radians(90.0)}"/>
+      <limit lower="${radians(-60)}" upper="${radians(76)}" effort="10591.1" velocity="${radians(90)}"/>
     </joint>
     <joint name="${prefix}joint_3" type="revolute">
@@ -116,5 +116,5 @@
       <origin xyz="0 0 1.150" rpy="0 0 0" />
       <axis xyz="0 -1 0" />
-      <limit lower="${radians(-77.8)}" upper="${radians(197)}" effort="9929.2" velocity="${radians(97.0)}"/>
+      <limit lower="${radians(-77.8)}" upper="${radians(197)}" effort="9929.2" velocity="${radians(97)}"/>
     </joint>
     <joint name="${prefix}joint_4" type="revolute">

File: motoman_gp35l_support/urdf/gp35l_macro.xacro (robot description, xacro)
@@ -102,5 +102,5 @@
       <origin xyz="0 0 0.540" rpy="0 0 0" />
       <axis xyz="0 0 1" />
-      <limit lower="${radians(-180)}" upper="${radians(180)}" effort="5516.2" velocity="${radians(180.0)}"/>
+      <limit lower="${radians(-180)}" upper="${radians(180)}" effort="5516.2" velocity="${radians(180)}"/>
     </joint>
     <joint name="${prefix}joint_2" type="revolute">
@@ -109,5 +109,5 @@
       <origin xyz="0.145 0 0" rpy="0 0 0" />
       <axis xyz="0 1 0" />
-      <limit lower="${radians(-90)}" upper="${radians(135)}" effort="7060.7" velocity="${radians(140.0)}"/>
+      <limit lower="${radians(-90)}" upper="${radians(135)}" effort="7060.7" velocity="${radians(140)}"/>
     </joint>
     <joint name="${prefix}joint_3" type="revolute">
@@ -116,5 +116,5 @@
       <origin xyz="0 0 1.150" rpy="0 0 0" />
       <axis xyz="0 -1 0" />
-      <limit lower="${radians(-80)}" upper="${radians(206)}" effort="3089.0" velocity="${radians(178.0)}"/>
+      <limit lower="${radians(-80)}" upper="${radians(206)}" effort="3089.0" velocity="${radians(178)}"/>
     </joint>
     <joint name="${prefix}joint_4" type="revolute">

File: motoman_gp70l_support/urdf/gp70l_macro.xacro (robot description, xacro)
@@ -102,5 +102,5 @@
       <origin xyz="0 0 0.540" rpy="0 0 0" />
       <axis xyz="0 0 1" />
-      <limit lower="${radians(-180)}" upper="${radians(180)}" effort="3983.9" velocity="${radians(180.0)}"/>
+      <limit lower="${radians(-180)}" upper="${radians(180)}" effort="3983.9" velocity="${radians(180)}"/>
     </joint>
     <joint name="${prefix}joint_2" type="revolute">
@@ -109,5 +109,5 @@
       <origin xyz="0.320 0 0" rpy="0 0 0" />
       <axis xyz="0 1 0" />
-      <limit lower="${radians(-90)}" upper="${radians(155)}" effort="10174.4" velocity="${radians(123.0)}"/>
+      <limit lower="${radians(-90)}" upper="${radians(155)}" effort="10174.4" velocity="${radians(123)}"/>
     </joint>
     <joint name="${prefix}joint_3" type="revolute">
@@ -116,5 +116,5 @@
       <origin xyz="0 0 1.165" rpy="0 0 0" />
       <axis xyz="0 -1 0" />
-      <limit lower="${radians(-80)}" upper="${radians(90)}" effort="5148.4" velocity="${radians(160.0)}"/>
+      <limit lower="${radians(-80)}" upper="${radians(90)}" effort="5148.4" velocity="${radians(160)}"/>
     </joint>
     <joint name="${prefix}joint_4" type="revolute">

File: motoman_sda10f_support/urdf/arm_macro.xacro (robot description, xacro)
@@ -109,5 +109,5 @@
       <parent link="${parent}"/>
       <child link="${prefix}link_1"/>
-      <origin xyz="0.100 ${reflect*0.265} 0.0" rpy="${radians(90)} 0.0 ${(reflect-1)*radians(90)}"/>
+      <origin xyz="0.100 ${reflect*0.265} 0" rpy="${radians(90)} 0 ${(reflect-1)*radians(90)}"/>
       <axis xyz="0 0 ${-reflect}" />
       <limit lower="${radians(-180)}" upper="${radians(180)}" effort="0" velocity="${radians(170)}" />
@@ -116,5 +116,5 @@
       <parent link="${prefix}link_1"/>
       <child link="${prefix}link_2"/>
-      <origin xyz="0.0 0.0 0.0" rpy="${radians(-90)} 0.0 0.0"/>
+      <origin xyz="0 0 0" rpy="${radians(-90)} 0 0"/>
       <axis xyz="0 0 ${-reflect}" />
       <limit lower="${radians(-110)}" upper="${radians(110)}" effort="0" velocity="${radians(170)}" />
@@ -123,5 +123,5 @@
       <parent link="${prefix}link_2"/>
       <child link="${prefix}link_3"/>
-      <origin xyz="0.0 0.360 0.0" rpy="${radians(90)} 0.0 0.0"/>
+      <origin xyz="0 0.360 0" rpy="${radians(90)} 0 0"/>
       <axis xyz="0 0 ${-reflect}" />
       <limit lower="${radians(-170)}" upper="${radians(170)}" effort="0" velocity="${radians(170)}" />
@@ -130,5 +130,5 @@
       <parent link="${prefix}link_3"/>
       <child link="${prefix}link_4"/>
-      <origin xyz="0.0 0.0 0.0" rpy="${radians(-90)} 0.0 0.0"/>
+      <origin xyz="0 0 0" rpy="${radians(-90)} 0 0"/>
       <axis xyz="0 0 ${reflect}" />
       <limit lower="${radians(-135)}" upper="${radians(135)}" effort="0" velocity="${radians(170)}" />
@@ -137,5 +137,5 @@
       <parent link="${prefix}link_4"/>
       <child link="${prefix}link_5"/>
-      <origin xyz="0.0 0.360 0.0" rpy="${radians(90)} 0.0 0.0"/>
+      <origin xyz="0 0.360 0" rpy="${radians(90)} 0 0"/>
       <axis xyz="0 0 ${reflect}" />
       <limit lower="${radians(-180)}" upper="${radians(180)}" effort="0" velocity="${radians(200)}" />
@@ -144,5 +144,5 @@
       <parent link="${prefix}link_5"/>
       <child link="${prefix}link_6"/>
-      <origin xyz="0.0 0.0 0.0" rpy="${radians(-90)} 0.0 0.0"/>
+      <origin xyz="0 0 0" rpy="${radians(-90)} 0 0"/>
       <axis xyz="0 0 ${reflect}" />
       <limit lower="${radians(-110)}" upper="${radians(110)}" effort="0" velocity="${radians(200)}" />
@@ -151,5 +151,5 @@
       <parent link="${prefix}link_6"/>
       <child link="${prefix}link_7"/>
-      <origin xyz="0.0 0.155 0.0" rpy="${radians(-90)} 0.0 0.0"/>
+      <origin xyz="0 0.155 0" rpy="${radians(-90)} 0 0"/>
       <axis xyz="0 0 ${-reflect}" />
       <limit lower="${radians(-180)}" upper="${radians(180)}" effort="0" velocity="${radians(400)}" />

File: motoman_sda10f_support/urdf/csda10f_arm_macro.xacro (robot description, xacro)
@@ -109,5 +109,5 @@
       <parent link="${parent}"/>
       <child link="${prefix}link_1"/>
-      <origin xyz="0.100 ${reflect*0.265} 0.0" rpy="${radians(90)} 0.0 ${(reflect-1)*radians(90)}"/>
+      <origin xyz="0.100 ${reflect*0.265} 0" rpy="${radians(90)} 0 ${(reflect-1)*radians(90)}"/>
       <axis xyz="0 0 ${-reflect}" />
       <limit lower="${radians(-170)}" upper="${radians(170)}" effort="268.36" velocity="${radians(170)}" />
@@ -116,5 +116,5 @@
       <parent link="${prefix}link_1"/>
       <child link="${prefix}link_2"/>
-      <origin xyz="0.0 0.0 0.0" rpy="${radians(-90)} 0.0 0.0"/>
+      <origin xyz="0 0 0" rpy="${radians(-90)} 0 0"/>
       <axis xyz="0 0 ${-reflect}" />
       <limit lower="${radians(-110)}" upper="${radians(110)}" effort="268.36" velocity="${radians(170)}" />
@@ -123,5 +123,5 @@
       <parent link="${prefix}link_2"/>
       <child link="${prefix}link_3"/>
-      <origin xyz="0.0 0.360 0.0" rpy="${radians(90)} 0.0 0.0"/>
+      <origin xyz="0 0.360 0" rpy="${radians(90)} 0 0"/>
       <axis xyz="0 0 ${-reflect}" />
       <limit lower="${radians(-170)}" upper="${radians(170)}" effort="122.89" velocity="${radians(170)}" />
@@ -130,5 +130,5 @@
       <parent link="${prefix}link_3"/>
       <child link="${prefix}link_4"/>
-      <origin xyz="0.0 0.0 0.0" rpy="${radians(-90)} 0.0 0.0"/>
+      <origin xyz="0 0 0" rpy="${radians(-90)} 0 0"/>
       <axis xyz="0 0 ${reflect}" />
       <limit lower="${radians(-135)}" upper="${radians(135)}" effort="122.89" velocity="${radians(170)}" />
@@ -137,5 +137,5 @@
       <parent link="${prefix}link_4"/>
       <child link="${prefix}link_5"/>
-      <origin xyz="0.0 0.360 0.0" rpy="${radians(90)} 0.0 0.0"/>
+      <origin xyz="0 0.360 0" rpy="${radians(90)} 0 0"/>
       <axis xyz="0 0 ${reflect}" />
       <limit lower="${radians(-180)}" upper="${radians(180)}" effort="44.34" velocity="${radians(200)}" />
@@ -144,5 +144,5 @@
       <parent link="${prefix}link_5"/>
       <child link="${prefix}link_6"/>
-      <origin xyz="0.0 0.0 0.0" rpy="${radians(-90)} 0.0 0.0"/>
+      <origin xyz="0 0 0" rpy="${radians(-90)} 0 0"/>
       <axis xyz="0 0 ${reflect}" />
       <limit lower="${radians(-110)}" upper="${radians(110)}" effort="44.34" velocity="${radians(200)}" />
@@ -151,5 +151,5 @@
       <parent link="${prefix}link_6"/>
       <child link="${prefix}link_7"/>
-      <origin xyz="0.0 0.175 0.0" rpy="${radians(-90)} 0.0 0.0"/>
+      <origin xyz="0 0.175 0" rpy="${radians(-90)} 0 0"/>
       <axis xyz="0 0 ${-reflect}" />
       <limit lower="${radians(-180)}" upper="${radians(180)}" effort="39.04" velocity="${radians(400)}" />
