Commit message: remove unnecessary trailing spaces

File: motoman_ms210_support/urdf/ms210_macro.xacro (robot description, xacro)
@@ -171,5 +171,5 @@
   <link name="${prefix}tool0"/>
   <joint name="${prefix}flange-tool0" type="fixed">
-    <origin xyz="0 0 0 " rpy="${radians(180)} ${radians(-90)} 0"/>
+    <origin xyz="0 0 0" rpy="${radians(180)} ${radians(-90)} 0"/>
     <parent link="${prefix}flange"/>
     <child link="${prefix}tool0"/>

File: motoman_sda10f_support/urdf/sda10f_macro.xacro (robot description, xacro)
@@ -4,5 +4,5 @@
   <xacro:include filename="$(find motoman_sda10f_support)/urdf/common_torso_macro.xacro" />
   <xacro:include filename="$(find motoman_sda10f_support)/urdf/arm_macro.xacro" />
-  <xacro:macro name="motoman_sda10f" params="prefix left_arm_prefix right_arm_prefix left_base_prefix right_base_prefix ">
+  <xacro:macro name="motoman_sda10f" params="prefix left_arm_prefix right_arm_prefix left_base_prefix right_base_prefix">
     <xacro:torso name="${prefix}torso" prefix="${prefix}"  left_base_prefix="${left_base_prefix}" right_base_prefix="${right_base_prefix}"/>
     <xacro:motoman_arm name="${prefix}${left_arm_prefix}arm" prefix="${prefix}${left_arm_prefix}" parent="${prefix}${left_base_prefix}base_link" reflect="1">

File: motoman_sia30d_support/urdf/sia30d_macro.xacro (robot description, xacro)
@@ -177,5 +177,5 @@
     <link name="${prefix}tool0"/>
     <joint name="${prefix}flange-tool0" type="fixed">
-        <origin xyz="0 0 0 " rpy="0 ${radians(-90)} ${radians(180)}"/>
+        <origin xyz="0 0 0" rpy="0 ${radians(-90)} ${radians(180)}"/>
         <parent link="${prefix}flange"/>
         <child link="${prefix}tool0"/>

File: motoman_sia50_support/urdf/sia50_macro.xacro (robot description, xacro)
@@ -197,5 +197,5 @@
     <link name="${prefix}tool0"/>
     <joint name="${prefix}flange-tool0" type="fixed">
-        <origin xyz="0 0 0 " rpy="${radians(180)} ${radians(-90)} 0"/>
+        <origin xyz="0 0 0" rpy="${radians(180)} ${radians(-90)} 0"/>
         <parent link="${prefix}flange"/>
         <child link="${prefix}tool0"/>
