Commit message: replace radian values with degree values

File: motoman_ar2010_support/urdf/ar2010_macro.xacro (robot description, xacro)
@@ -108,5 +108,5 @@
       <parent link="${prefix}link_1"/>
       <child link="${prefix}link_2"/>
-      <origin xyz="0.150 0 0" rpy="${pi/2} ${-pi/2} ${-pi}"/>
+      <origin xyz="0.150 0 0" rpy="${radians(90)} ${radians(-90)} ${radians(-180)}"/>
       <axis xyz="0 0 1"/>
       <limit lower="${radians(-105)}" upper="${radians(155)}" effort="3087" velocity="${radians(210)}"/>
@@ -115,5 +115,5 @@
       <parent link="${prefix}link_2"/>
       <child link="${prefix}link_3"/>
-      <origin xyz="0.760 0 0" rpy="${pi} 0 0"/>
+      <origin xyz="0.760 0 0" rpy="${radians(180)} 0 0"/>
       <axis xyz="0 0 1"/>
       <limit lower="${radians(-86)}" upper="${radians(160)}" effort="926.1" velocity="${radians(220)}"/>
@@ -122,5 +122,5 @@
       <parent link="${prefix}link_3"/>
       <child link="${prefix}link_4"/>
-      <origin xyz="0.200 -1.082 0" rpy="${-pi/2} 0 0"/>
+      <origin xyz="0.200 -1.082 0" rpy="${radians(-90)} 0 0"/>
       <axis xyz="0 0 1"/>
       <limit lower="${radians(-150)}" upper="${radians(150)}" effort="78.4" velocity="${radians(435)}"/>
@@ -129,5 +129,5 @@
       <parent link="${prefix}link_4"/>
       <child link="${prefix}link_5"/>
-      <origin xyz="0 0 0" rpy="${pi/2} 0 0"/>
+      <origin xyz="0 0 0" rpy="${radians(90)} 0 0"/>
       <axis xyz="0 0 1"/>
       <limit lower="${radians(-135)}" upper="${radians(90)}" effort="67.03" velocity="${radians(435)}"/>
@@ -136,5 +136,5 @@
       <parent link="${prefix}link_5"/>
       <child link="${prefix}link_6"/>
-      <origin xyz="0 -0.100 0" rpy="${-pi/2} 0 0"/>
+      <origin xyz="0 -0.100 0" rpy="${radians(-90)} 0 0"/>
       <axis xyz="0 0 1"/>
       <limit lower="${radians(-210)}" upper="${radians(210)}" effort="33.3" velocity="${radians(700)}"/>
@@ -151,5 +151,5 @@
     <link name="${prefix}flange"/>
     <joint name="${prefix}joint_6-flange" type="fixed">
-      <origin xyz="0 0 0" rpy="0 ${pi/2} 0"/>
+      <origin xyz="0 0 0" rpy="0 ${radians(90)} 0"/>
       <parent link="${prefix}link_6"/>
       <child link="${prefix}flange"/>
@@ -158,5 +158,5 @@
     <link name="${prefix}tool0"/>
     <joint name="${prefix}flange-tool0" type="fixed">
-      <origin xyz="0 0 0" rpy="${pi} ${-pi/2.0} 0"/>
+      <origin xyz="0 0 0" rpy="${radians(180)} ${radians(-90)} 0"/>
       <parent link="${prefix}flange"/>
       <child link="${prefix}tool0"/>

File: motoman_gp12_support/urdf/gp12_macro.xacro (robot description, xacro)
@@ -102,5 +102,5 @@
         <origin xyz="0 0 0.450" rpy="0 0 0" />
         <axis xyz="0 0 1" />
-        <limit lower="-2.9670" upper="2.9670" effort="926.10" velocity="4.5355"/>
+        <limit lower="${radians(-170)}" upper="${radians(170)}" effort="926.10" velocity="${radians(260)}"/>
     </joint>
     <joint name="${prefix}joint_2" type="revolute">
@@ -109,5 +109,5 @@
         <origin xyz="0.155 0 0" rpy="0 0 0" />
         <axis xyz="0 1 0" />
-        <limit lower="-1.5708" upper="2.7052" effort="1029.00" velocity="4.0132"/>
+        <limit lower="${radians(-90)}" upper="${radians(155)}" effort="1029.00" velocity="${radians(230)}"/>
     </joint>
     <joint name="${prefix}joint_3" type="revolute">
@@ -116,5 +116,5 @@
         <origin xyz="0 0 0.614" rpy="0 0 0" />
         <axis xyz="0 -1 0" />
-        <limit lower="-1.4835" upper="2.6179" effort="551.25" velocity="4.5375"/>
+        <limit lower="${radians(-85)}" upper="${radians(150)}" effort="551.25" velocity="${radians(260)}"/>
     </joint>
     <joint name="${prefix}joint_4" type="revolute">
@@ -123,5 +123,5 @@
         <origin xyz="0.640 0 0.200" rpy="0 0 0" />
         <axis xyz="-1 0 0" />
-        <limit lower="-3.4906" upper="3.4906" effort="89.96" velocity="8.2007"/>
+        <limit lower="${radians(-200)}" upper="${radians(200)}" effort="89.96" velocity="${radians(470)}"/>
     </joint>
     <joint name="${prefix}joint_5" type="revolute">
@@ -130,5 +130,5 @@
         <origin xyz="0 0 0" rpy="0 0 0" />
         <axis xyz="0 -1 0" />
-        <limit lower="-2.6179" upper="2.6179" effort="67.03" velocity="8.1992"/>
+        <limit lower="${radians(-150)}" upper="${radians(150)}" effort="67.03" velocity="${radians(470)}"/>
     </joint>
     <joint name="${prefix}joint_6" type="revolute">
@@ -137,5 +137,5 @@
         <origin xyz="0 0 0" rpy="0 0 0" />
         <axis xyz="-1 0 0" />
-        <limit lower="-7.9412" upper="7.9412" effort="33.30" velocity="12.2143"/>
+        <limit lower="${radians(-455)}" upper="${radians(455)}" effort="33.30" velocity="${radians(700)}"/>
     </joint>
     <!-- end of joint list -->
@@ -157,5 +157,5 @@
     <link name="${prefix}tool0"/>
     <joint name="${prefix}flange-tool0" type="fixed">
-      <origin xyz="0 0 0" rpy="3.1415926 -1.570796 0"/>
+      <origin xyz="0 0 0" rpy="${radians(180)} ${radians(-90)} 0"/>
       <parent link="${prefix}flange"/>
       <child link="${prefix}tool0"/>

File: motoman_gp180_support/urdf/gp180_macro.xacro (robot description, xacro)
@@ -167,5 +167,5 @@
     <link name="${prefix}tool0" />
     <joint name="${prefix}flange-tool0" type="fixed">
-        <origin xyz="0 0 0" rpy="${pi} ${-pi/2.0} 0" />
+        <origin xyz="0 0 0" rpy="${radians(180)} ${radians(-90)} 0" />
         <parent link="${prefix}flange" />
         <child link="${prefix}tool0" />

File: motoman_hc20_support/urdf/hc30pl_macro.xacro (robot description, xacro)
@@ -74,5 +74,5 @@
           <mesh filename="package://motoman_hc20_support/meshes/hc20dtp/visual/link_5.dae"/>
         </geometry>
-        <origin rpy="0 1.57075 0"/>
+        <origin rpy="0 ${radians(90)} 0"/>
         <xacro:material_yaskawa_white/>
       </visual>
@@ -81,5 +81,5 @@
           <mesh filename="package://motoman_hc20_support/meshes/hc20dtp/collision/link_5.stl"/>
         </geometry>
-        <origin rpy="0 1.57075 0"/>
+        <origin rpy="0 ${radians(90)} 0"/>
       </collision>
     </link>
@@ -89,5 +89,5 @@
           <mesh filename="package://motoman_hc20_support/meshes/hc20dtp/visual/link_6.dae"/>
         </geometry>
-        <origin rpy="0 1.57075 0"/>
+        <origin rpy="0 ${radians(90)} 0"/>
         <xacro:material_yaskawa_white/>
       </visual>
@@ -96,5 +96,5 @@
           <mesh filename="package://motoman_hc20_support/meshes/hc20dtp/collision/link_6.stl"/>
         </geometry>
-        <origin rpy="0 1.57075 0"/>
+        <origin rpy="0 ${radians(90)} 0"/>
       </collision>
     </link>

File: motoman_ma2010_support/urdf/ma2010_macro.xacro (robot description, xacro)
@@ -102,5 +102,5 @@
       <origin xyz="0 0 0.505" rpy="0 0 0" />
       <axis xyz="0 0 1" />
-      <limit lower="-3.1416" upper="3.1416" effort="3087" velocity="3.4383"/>
+      <limit lower="${radians(-180)}" upper="${radians(180)}" effort="3087" velocity="${radians(197)}"/>
     </joint>
     <joint name="${prefix}joint_2" type="revolute">
@@ -109,5 +109,5 @@
       <origin xyz="0.150 0 0" rpy="0 0 0" />
       <axis xyz="0 1 0" />
-      <limit lower="-1.8326" upper="2.7052" effort="2744" velocity="3.3161"/>
+      <limit lower="${radians(-105)}" upper="${radians(155)}" effort="2744" velocity="${radians(190)}"/>
     </joint>
     <joint name="${prefix}joint_3" type="revolute">
@@ -116,5 +116,5 @@
       <origin xyz="0 0 0.760" rpy="0 0 0" />
       <axis xyz="0 -1 0" />
-      <limit lower="-1.5009" upper="2.7925" effort="874.65" velocity="3.6652"/>
+      <limit lower="${radians(-86)}" upper="${radians(160)}" effort="874.65" velocity="${radians(210)}"/>
     </joint>
     <joint name="${prefix}joint_4" type="revolute">
@@ -123,5 +123,5 @@
       <origin xyz="0 0 0.200" rpy="0 0 0" />
       <axis xyz="-1 0 0" />
-      <limit lower="-2.6180" upper="2.6180" effort="78.4" velocity="7.1558"/>
+      <limit lower="${radians(-150)}" upper="${radians(150)}" effort="78.4" velocity="${radians(410)}"/>
     </joint>
     <joint name="${prefix}joint_5" type="revolute">
@@ -130,5 +130,5 @@
       <origin xyz="1.082 0 0" rpy="0 0 0" />
       <axis xyz="0 -1 0" />
-      <limit lower="-2.3562" upper="1.5708" effort="59.58" velocity="7.1558"/>
+      <limit lower="${radians(-135)}" upper="${radians(90)}" effort="59.58" velocity="${radians(410)}"/>
     </joint>
     <joint name="${prefix}joint_6" type="revolute">
@@ -137,5 +137,5 @@
       <origin xyz="0 0 0" rpy="0 0 0" />
       <axis xyz="-1 0 0" />
-      <limit lower="-3.6652" upper="3.6652" effort="29.6" velocity="10.6465"/>
+      <limit lower="${radians(-210)}" upper="${radians(210)}" effort="29.6" velocity="${radians(610)}"/>
     </joint>
     <!-- end of joint list -->
@@ -157,5 +157,5 @@
     <link name="${prefix}tool0"/>
     <joint name="${prefix}flange-tool0" type="fixed">
-      <origin xyz="0 0 0" rpy="3.1415926 -1.5707963 0"/>
+      <origin xyz="0 0 0" rpy="${radians(180)} ${radians(-90)} 0"/>
       <parent link="${prefix}flange"/>
       <child link="${prefix}tool0"/>

File: motoman_mh12_support/urdf/mh12_macro.xacro (robot description, xacro)
@@ -157,5 +157,5 @@
     <link name="${prefix}tool0"/>
     <joint name="${prefix}flange-tool0" type="fixed">
-      <origin xyz="0 0 0" rpy="3.1415926 -1.570796 0"/>
+      <origin xyz="0 0 0" rpy="${radians(180)} ${radians(-90)} 0"/>
       <parent link="${prefix}flange"/>
       <child link="${prefix}tool0"/>

File: motoman_mh50_support/urdf/mh50_macro.xacro (robot description, xacro)
@@ -102,5 +102,5 @@
         <origin xyz="0 0 0.540" rpy="0 0 0" />
         <axis xyz="0 0 1" />
-        <limit lower="-3.14159" upper="3.14159" effort="4903.32" velocity="3.141"/>
+        <limit lower="${radians(-180)}" upper="${radians(180)}" effort="4903.32" velocity="${radians(180)}"/>
     </joint>
     <joint name="${prefix}joint_2" type="revolute">
@@ -109,5 +109,5 @@
         <origin xyz="0.145 0 0" rpy="0 0 0" />
         <axis xyz="0 1 0" />
-        <limit lower="-1.57079" upper="2.35619" effort="6276.26" velocity="3.103"/>
+        <limit lower="${radians(-90)}" upper="${radians(135)}" effort="6276.26" velocity="${radians(178)}"/>
     </joint>
     <joint name="${prefix}joint_3" type="revolute">
@@ -116,5 +116,5 @@
         <origin xyz="0 0 0.870" rpy="0 0 0" />
         <axis xyz="0 -1 0" />
-        <limit lower="-1.39626" upper="3.59538" effort="2745.86" velocity="3.106"/>
+        <limit lower="${radians(-80)}" upper="${radians(206)}" effort="2745.86" velocity="${radians(178)}"/>
     </joint>
     <joint name="${prefix}joint_4" type="revolute">
@@ -123,5 +123,5 @@
         <origin xyz="1.025 0 0.210" rpy="0 0 0"/>
         <axis xyz="-1 0 0" />
-        <limit lower="-6.28319" upper="6.28319" effort="823.76" velocity="4.363"/>
+        <limit lower="${radians(-360)}" upper="${radians(360)}" effort="823.76" velocity="${radians(250)}"/>
     </joint>
     <joint name="${prefix}joint_5" type="revolute">
@@ -130,5 +130,5 @@
         <origin xyz="0 0 0" rpy="0 0 0" />
         <axis xyz="0 -1 0" />
-        <limit lower="-2.18167" upper="2.18167" effort="706.08" velocity="4.363"/>
+        <limit lower="${radians(-125)}" upper="${radians(125)}" effort="706.08" velocity="${radians(250)}"/>
     </joint>
     <joint name="${prefix}joint_6" type="revolute">
@@ -137,5 +137,5 @@
         <origin xyz="0 0 0" rpy="0 0 0" />
         <axis xyz="-1 0 0" />
-        <limit lower="-6.2831" upper="6.2831" effort="333.43" velocity="6.283"/>
+        <limit lower="${radians(-360)}" upper="${radians(360)}" effort="333.43" velocity="${radians(360)}"/>
     </joint>
     <!-- end of joint list -->
@@ -157,5 +157,5 @@
     <link name="${prefix}tool0"/>
     <joint name="${prefix}flange-tool0" type="fixed">
-      <origin xyz="0 0 0" rpy="3.1415926 -1.570796 0"/>
+      <origin xyz="0 0 0" rpy="${radians(180)} ${radians(-90)} 0"/>
       <parent link="${prefix}flange"/>
       <child link="${prefix}tool0"/>

File: motoman_motomini_support/urdf/motomini_macro.xacro (robot description, xacro)
@@ -102,5 +102,5 @@
     <origin xyz="0 0 0.103" rpy="0 0 0" />
     <axis xyz="0 0 1" />
-    <limit lower="-2.9670" upper="2.9670" effort="0.12" velocity="5.4977"/>
+    <limit lower="${radians(-170)}" upper="${radians(170)}" effort="0.12" velocity="${radians(315)}"/>
   </joint>
   <joint name="${prefix}joint_2" type="revolute">
@@ -109,5 +109,5 @@
     <origin xyz="0.020 0 0" rpy="0 0 0" />
     <axis xyz="0 1 0" />
-    <limit lower="-1.4835" upper="1.5707" effort="0.12" velocity="5.4977"/>
+    <limit lower="${radians(-85)}" upper="${radians(90)}" effort="0.12" velocity="${radians(315)}"/>
   </joint>
   <joint name="${prefix}joint_3" type="revolute">
@@ -116,5 +116,5 @@
     <origin xyz="0 0 0.165" rpy="0 0 0" />
     <axis xyz="0 -1 0" />
-    <limit lower="-0.8726" upper="1.5707" effort="0.12" velocity="7.3304"/>
+    <limit lower="${radians(-50)}" upper="${radians(90)}" effort="0.12" velocity="${radians(420)}"/>
   </joint>
   <joint name="${prefix}joint_4" type="revolute">
@@ -123,5 +123,5 @@
     <origin xyz="0.165 0 0" rpy="0 0 0" />
     <axis xyz="-1 0 0" />
-    <limit lower="-2.4434" upper="2.4434" effort="0.07" velocity="10.4719"/>
+    <limit lower="${radians(-140)}" upper="${radians(140)}" effort="0.07" velocity="${radians(600)}"/>
   </joint>
   <joint name="${prefix}joint_5" type="revolute">
@@ -130,5 +130,5 @@
     <origin xyz="0 0 0" rpy="0 0 0" />
     <axis xyz="0 -1 0" />
-    <limit lower="-0.5235" upper="3.6651" effort="0.07" velocity="10.4719"/>
+    <limit lower="${radians(-30)}" upper="${radians(210)}" effort="0.07" velocity="${radians(600)}"/>
   </joint>
   <joint name="${prefix}joint_6" type="revolute">
@@ -137,5 +137,5 @@
     <origin xyz="0 0 0" rpy="0 0 0" />
     <axis xyz="0 0 1" />
-    <limit lower="-6.2831" upper="6.2831" effort="0.07" velocity="10.4719"/>
+    <limit lower="${radians(-360)}" upper="${radians(360)}" effort="0.07" velocity="${radians(600)}"/>
   </joint>
     <!-- end of joint list -->
@@ -150,5 +150,5 @@
     <link name="${prefix}flange"/>
     <joint name="${prefix}joint_6-flange" type="fixed">
-      <origin xyz="0 0 -0.040" rpy="0 ${pi/2} 0"/>
+      <origin xyz="0 0 -0.040" rpy="0 ${radians(90)} 0"/>
       <parent link="${prefix}link_6"/>
       <child link="${prefix}flange"/>
@@ -157,5 +157,5 @@
     <link name="${prefix}tool0"/>
     <joint name="${prefix}flange-tool0" type="fixed">
-      <origin xyz="0 0 0 " rpy="${pi} ${-pi/2} 0"/>
+      <origin xyz="0 0 0" rpy="${radians(180)} ${radians(-90)} 0"/>
       <parent link="${prefix}flange"/>
       <child link="${prefix}tool0"/>

File: motoman_motopos_d500_support/urdf/motopos_d500_macro.xacro (robot description, xacro)
@@ -50,5 +50,5 @@
       <origin xyz="0 0 0.380" rpy="0 0 0" />
       <axis xyz="0 -1 0" />
-      <limit lower="-2.3561" upper="2.3561" effort="1274" velocity="1.3962"/>
+      <limit lower="${radians(-135)}" upper="${radians(135)}" effort="1274" velocity="${radians(80)}"/>
     </joint>
     <joint name="${prefix}joint_2" type="revolute">
@@ -57,5 +57,5 @@
       <origin xyz="0 0 0" rpy="0 0 0" />
       <axis xyz="0 0 -1" />
-      <limit lower="-3.4906" upper="3.4906" effort="392" velocity="2.7925"/>
+      <limit lower="${radians(-200)}" upper="${radians(200)}" effort="392" velocity="${radians(160)}"/>
     </joint>
     <!-- end of joint list -->
@@ -70,5 +70,5 @@
     <link name="${prefix}flange"/>
     <joint name="${prefix}joint_2-flange" type="fixed">
-      <origin xyz="0 0 0.150 " rpy="0 -1.57079632679 0"/>
+      <origin xyz="0 0 0.150" rpy="0 ${radians(-90)} 0"/>
       <parent link="${prefix}link_2"/>
       <child link="${prefix}flange"/>
@@ -77,5 +77,5 @@
     <link name="${prefix}tool0"/>
     <joint name="${prefix}flange-tool0" type="fixed">
-      <origin xyz="0 0 0 " rpy="0 -1.57079632679 3.14159265359"/>
+      <origin xyz="0 0 0" rpy="0 ${radians(-90)} ${radians(180)}"/>
       <parent link="${prefix}flange"/>
       <child link="${prefix}tool0"/>

File: motoman_motopos_mh1655_support/urdf/motopos_mh1655_macro.xacro (robot description, xacro)
@@ -55,5 +55,5 @@
       <!-- NOTE: the velocity limit is a conservative conversion from the stated
            limit in the manual: 10.8 rpm (in section 3.2.1) -->
-      <limit lower="${-2*pi}" upper="${2*pi}" effort="1274" velocity="1.1309"/>
+      <limit lower="${radians(-360)}" upper="${radians(360)}" effort="1274" velocity="${radians(65)}"/>
     </joint>
     <!-- end of joint list -->
@@ -75,5 +75,5 @@
     <link name="${prefix}tool0"/>
     <joint name="${prefix}flange-tool0" type="fixed">
-      <origin xyz="0 0 0" rpy="${pi} ${-pi/2} 0"/>
+      <origin xyz="0 0 0" rpy="${radians(180)} ${radians(-90)} 0"/>
       <parent link="${prefix}flange"/>
       <child link="${prefix}tool0"/>
