Commit message: replace radian values with degree values

File: motoman_sia10d_support/urdf/sia10d_macro.xacro (robot description, xacro)
@@ -37,5 +37,5 @@
         <link name="${prefix}link_2">
             <visual>
-                <origin rpy="1.57 3.1416 0" xyz="0 0 0"/>
+                <origin rpy="${radians(90)} ${radians(180)} 0" xyz="0 0 0"/>
                 <geometry>
                     <mesh filename="package://motoman_sia10d_support/meshes/sia10d/visual/link_2.stl"/>
@@ -44,5 +44,5 @@
             </visual>
             <collision>
-                <origin rpy="1.57 3.1416 0" xyz="0 0 0"/>
+                <origin rpy="${radians(90)} ${radians(180)} 0" xyz="0 0 0"/>
                 <geometry>
                     <mesh filename="package://motoman_sia10d_support/meshes/sia10d/collision/link_2.stl" />
@@ -53,5 +53,5 @@
         <link name="${prefix}link_3">
             <visual>
-                <origin rpy="0 0 3.1415" xyz="0 0 0"/>
+                <origin rpy="0 0 ${radians(180)}" xyz="0 0 0"/>
                 <geometry>
                     <mesh filename="package://motoman_sia10d_support/meshes/sia10d/visual/link_3.stl"/>
@@ -60,5 +60,5 @@
             </visual>
             <collision>
-                <origin rpy="0 0 3.1415" xyz="0 0 0"/>
+                <origin rpy="0 0 ${radians(180)}" xyz="0 0 0"/>
                 <geometry>
                     <mesh filename="package://motoman_sia10d_support/meshes/sia10d/collision/link_3.stl" />
@@ -69,5 +69,5 @@
         <link name="${prefix}link_4">
             <visual>
-                <origin rpy="1.57 -3.1415 0" xyz="0 0 0"/>
+                <origin rpy="${radians(90)} ${radians(-180)} 0" xyz="0 0 0"/>
                 <geometry>
                     <mesh filename="package://motoman_sia10d_support/meshes/sia10d/visual/link_4.stl"/>
@@ -76,5 +76,5 @@
             </visual>
             <collision>
-                <origin rpy="1.57 -3.1415 0" xyz="0 0 0"/>
+                <origin rpy="${radians(90)} ${radians(-180)} 0" xyz="0 0 0"/>
                 <geometry>
                     <mesh filename="package://motoman_sia10d_support/meshes/sia10d/collision/link_4.stl" />
@@ -85,5 +85,5 @@
         <link name="${prefix}link_5">
             <visual>
-                <origin rpy="0 0 3.1416" xyz="0 0 0"/>
+                <origin rpy="0 0 ${radians(180)}" xyz="0 0 0"/>
                 <geometry>
                     <mesh filename="package://motoman_sia10d_support/meshes/sia10d/visual/link_5.stl"/>
@@ -92,5 +92,5 @@
             </visual>
             <collision>
-                <origin rpy="0 0 3.1416" xyz="0 0 0"/>
+                <origin rpy="0 0 ${radians(180)}" xyz="0 0 0"/>
                 <geometry>
                     <mesh filename="package://motoman_sia10d_support/meshes/sia10d/collision/link_5.stl" />
@@ -101,5 +101,5 @@
         <link name="${prefix}link_6">
             <visual>
-                <origin rpy="-1.57 0 3.1416" xyz="0 0 0"/>
+                <origin rpy="${radians(-90)} 0 ${radians(180)}" xyz="0 0 0"/>
                 <geometry>
                     <mesh filename="package://motoman_sia10d_support/meshes/sia10d/visual/link_6.stl"/>
@@ -108,5 +108,5 @@
             </visual>
             <collision>
-                <origin rpy="-1.57 0 3.1416" xyz="0 0 0"/>
+                <origin rpy="${radians(-90)} 0 ${radians(180)}" xyz="0 0 0"/>
                 <geometry>
                     <mesh filename="package://motoman_sia10d_support/meshes/sia10d/collision/link_6.stl" />
@@ -141,5 +141,5 @@
             <origin xyz="0 0 0.36" rpy="0 0 0"/>
             <axis xyz="0 0 1" />
-            <limit lower="-3.1415" upper="3.1415" effort="100" velocity="2.9670" />
+            <limit lower="${radians(-180)}" upper="${radians(180)}" effort="100" velocity="${radians(170)}" />
         </joint>
         <joint name="${prefix}joint_2" type="revolute">
@@ -148,5 +148,5 @@
             <origin xyz="0 0 0" rpy="0 0 0"/>
             <axis xyz="0 1 0" />
-            <limit lower="-1.9198" upper="1.9198" effort="100" velocity="2.9670" />
+            <limit lower="${radians(-110)}" upper="${radians(110)}" effort="100" velocity="${radians(170)}" />
         </joint>
         <joint name="${prefix}joint_3" type="revolute">
@@ -155,5 +155,5 @@
             <origin xyz="0 0 0.36" rpy="0 0 0"/>
             <axis xyz="0 0 1" />
-            <limit lower="-2.9670" upper="2.9670" effort="100" velocity="2.9670" />
+            <limit lower="${radians(-170)}" upper="${radians(170)}" effort="100" velocity="${radians(170)}" />
         </joint>
         <joint name="${prefix}joint_4" type="revolute">
@@ -162,5 +162,5 @@
             <origin xyz="0 0 0" rpy="0 0 0"/>
             <axis xyz="0 -1 0" />
-            <limit lower="-2.3561" upper="2.3561" effort="100" velocity="2.9670" />
+            <limit lower="${radians(-135)}" upper="${radians(135)}" effort="100" velocity="${radians(170)}" />
         </joint>
         <joint name="${prefix}joint_5" type="revolute">
@@ -169,5 +169,5 @@
             <origin xyz="0 0 0.360" rpy="0 0 0"/>
             <axis xyz="0 0 -1" />
-            <limit lower="-3.1415" upper="3.1415" effort="100" velocity="3.4906" />
+            <limit lower="${radians(-180)}" upper="${radians(180)}" effort="100" velocity="${radians(200)}" />
         </joint>
         <joint name="${prefix}joint_6" type="revolute">
@@ -176,5 +176,5 @@
             <origin xyz="0 0 0" rpy="0 0 0"/>
             <axis xyz="0 -1 0" />
-            <limit lower="-1.9198" upper="1.9198" effort="100" velocity="3.4906" />
+            <limit lower="${radians(-110)}" upper="${radians(110)}" effort="100" velocity="${radians(200)}" />
         </joint>
         <joint name="${prefix}joint_7" type="revolute">
@@ -183,5 +183,5 @@
             <origin xyz="0 0 0.155" rpy="0 0 0"/>
             <axis xyz="0 0 -1" />
-            <limit lower="-3.1415" upper="3.1415" effort="100" velocity="6.9813" />
+            <limit lower="${radians(-180)}" upper="${radians(180)}" effort="100" velocity="${radians(400)}" />
         </joint>
         <!-- end of joint list -->
@@ -196,5 +196,5 @@
         <link name="${prefix}flange"/>
         <joint name="${prefix}joint_7-flange" type="fixed">
-            <origin xyz="0 0 0" rpy="0 -1.57079632679 0"/>
+            <origin xyz="0 0 0" rpy="0 ${radians(-90)} 0"/>
             <parent link="${prefix}link_7"/>
             <child link="${prefix}flange"/>
@@ -203,5 +203,5 @@
         <link name="${prefix}tool0"/>
         <joint name="${prefix}flange-tool0" type="fixed">
-            <origin xyz="0 0 0 " rpy="0 -1.57079632679 3.1415296"/>
+            <origin xyz="0 0 0" rpy="0 ${radians(-90)} ${radians(180)}"/>
             <parent link="${prefix}flange"/>
             <child link="${prefix}tool0"/>

File: motoman_sia10f_support/urdf/sia10f_macro.xacro (robot description, xacro)
@@ -36,5 +36,5 @@
         <link name="${prefix}link_2">
             <visual>
-                <origin rpy="1.57 3.1416 0" xyz="0 0 0"/>
+                <origin rpy="${radians(90)} ${radians(180)} 0" xyz="0 0 0"/>
                 <geometry>
                     <mesh filename="package://motoman_sia10f_support/meshes/sia10f/visual/link_2.stl"/>
@@ -43,5 +43,5 @@
             </visual>
             <collision>
-                <origin rpy="1.57 3.1416 0" xyz="0 0 0"/>
+                <origin rpy="${radians(90)} ${radians(180)} 0" xyz="0 0 0"/>
                 <geometry>
                     <mesh filename="package://motoman_sia10f_support/meshes/sia10f/collision/link_2.stl" />
@@ -52,5 +52,5 @@
         <link name="${prefix}link_3">
             <visual>
-                <origin rpy="0 0 3.1415" xyz="0 0 0"/>
+                <origin rpy="0 0 ${radians(180)}" xyz="0 0 0"/>
                 <geometry>
                     <mesh filename="package://motoman_sia10f_support/meshes/sia10f/visual/link_3.stl"/>
@@ -59,5 +59,5 @@
             </visual>
             <collision>
-                <origin rpy="0 0 3.1415" xyz="0 0 0"/>
+                <origin rpy="0 0 ${radians(180)}" xyz="0 0 0"/>
                 <geometry>
                     <mesh filename="package://motoman_sia10f_support/meshes/sia10f/collision/link_3.stl" />
@@ -68,5 +68,5 @@
         <link name="${prefix}link_4">
             <visual>
-                <origin rpy="1.57 -3.1415 0" xyz="0 0 0"/>
+                <origin rpy="${radians(90)} ${radians(-180)} 0" xyz="0 0 0"/>
                 <geometry>
                     <mesh filename="package://motoman_sia10f_support/meshes/sia10f/visual/link_4.stl"/>
@@ -75,5 +75,5 @@
             </visual>
             <collision>
-                <origin rpy="1.57 -3.1415 0" xyz="0 0 0"/>
+                <origin rpy="${radians(90)} ${radians(-180)} 0" xyz="0 0 0"/>
                 <geometry>
                     <mesh filename="package://motoman_sia10f_support/meshes/sia10f/collision/link_4.stl" />
@@ -84,5 +84,5 @@
         <link name="${prefix}link_5">
             <visual>
-                <origin rpy="0 0 3.1416" xyz="0 0 0"/>
+                <origin rpy="0 0 ${radians(180)}" xyz="0 0 0"/>
                 <geometry>
                     <mesh filename="package://motoman_sia10f_support/meshes/sia10f/visual/link_5.stl"/>
@@ -91,5 +91,5 @@
             </visual>
             <collision>
-                <origin rpy="0 0 3.1416" xyz="0 0 0"/>
+                <origin rpy="0 0 ${radians(180)}" xyz="0 0 0"/>
                 <geometry>
                     <mesh filename="package://motoman_sia10f_support/meshes/sia10f/collision/link_5.stl" />
@@ -100,5 +100,5 @@
         <link name="${prefix}link_6">
             <visual>
-                <origin rpy="-1.57 0 3.1416" xyz="0 0 0"/>
+                <origin rpy="${radians(-90)} 0 ${radians(180)}" xyz="0 0 0"/>
                 <geometry>
                     <mesh filename="package://motoman_sia10f_support/meshes/sia10f/visual/link_6.stl"/>
@@ -107,5 +107,5 @@
             </visual>
             <collision>
-                <origin rpy="-1.57 0 3.1416" xyz="0 0 0"/>
+                <origin rpy="${radians(-90)} 0 ${radians(180)}" xyz="0 0 0"/>
                 <geometry>
                     <mesh filename="package://motoman_sia10f_support/meshes/sia10f/collision/link_6.stl" />
@@ -135,5 +135,5 @@
             <origin xyz="0 0 0.36" rpy="0 0 0"/>
             <axis xyz="0 0 1" />
-            <limit lower="-3.1415" upper="3.1415" effort="0" velocity="2.9670" />
+            <limit lower="${radians(-180)}" upper="${radians(180)}" effort="0" velocity="${radians(170)}" />
         </joint>
         <joint name="${prefix}joint_2" type="revolute">
@@ -142,5 +142,5 @@
             <origin xyz="0 0 0" rpy="0 0 0"/>
             <axis xyz="0 1 0" />
-            <limit lower="-1.9198" upper="1.9198" effort="0" velocity="2.9670" />
+            <limit lower="${radians(-110)}" upper="${radians(110)}" effort="0" velocity="${radians(170)}" />
         </joint>
         <joint name="${prefix}joint_3" type="revolute">
@@ -149,5 +149,5 @@
             <origin xyz="0 0 0.36" rpy="0 0 0"/>
             <axis xyz="0 0 1" />
-            <limit lower="-2.9670" upper="2.9670" effort="0" velocity="2.9670" />
+            <limit lower="${radians(-170)}" upper="${radians(170)}" effort="0" velocity="${radians(170)}" />
         </joint>
         <joint name="${prefix}joint_4" type="revolute">
@@ -156,5 +156,5 @@
             <origin xyz="0 0 0" rpy="0 0 0"/>
             <axis xyz="0 -1 0" />
-            <limit lower="-2.3561" upper="2.3561" effort="0" velocity="2.9670" />
+            <limit lower="${radians(-135)}" upper="${radians(135)}" effort="0" velocity="${radians(170)}" />
         </joint>
         <joint name="${prefix}joint_5" type="revolute">
@@ -163,5 +163,5 @@
             <origin xyz="0 0 0.360" rpy="0 0 0"/>
             <axis xyz="0 0 -1" />
-            <limit lower="-3.1415" upper="3.1415" effort="0" velocity="3.4906" />
+            <limit lower="${radians(-180)}" upper="${radians(180)}" effort="0" velocity="${radians(200)}" />
         </joint>
         <joint name="${prefix}joint_6" type="revolute">
@@ -170,5 +170,5 @@
             <origin xyz="0 0 0" rpy="0 0 0"/>
             <axis xyz="0 -1 0" />
-            <limit lower="-1.9198" upper="1.9198" effort="0" velocity="3.4906" />
+            <limit lower="${radians(-110)}" upper="${radians(110)}" effort="0" velocity="${radians(200)}" />
         </joint>
         <joint name="${prefix}joint_7" type="revolute">
@@ -177,5 +177,5 @@
             <origin xyz="0 0 0.155" rpy="0 0 0"/>
             <axis xyz="0 0 -1" />
-            <limit lower="-3.1415" upper="3.1415" effort="0" velocity="6.9813" />
+            <limit lower="${radians(-180)}" upper="${radians(180)}" effort="0" velocity="${radians(400)}" />
         </joint>
         <!-- end of joint list -->
@@ -190,5 +190,5 @@
         <link name="${prefix}flange"/>
         <joint name="${prefix}joint_7-flange" type="fixed">
-            <origin xyz="0 0 0" rpy="0 -1.57079632679 0"/>
+            <origin xyz="0 0 0" rpy="0 ${radians(-90)} 0"/>
             <parent link="${prefix}link_7"/>
             <child link="${prefix}flange"/>
@@ -197,5 +197,5 @@
         <link name="${prefix}tool0"/>
         <joint name="${prefix}flange-tool0" type="fixed">
-            <origin xyz="0 0 0 " rpy="0 -1.57079632679 3.1415296"/>
+            <origin xyz="0 0 0" rpy="0 ${radians(-90)} ${radians(180)}"/>
             <parent link="${prefix}flange"/>
             <child link="${prefix}tool0"/>

File: motoman_sia20d_support/urdf/sia20d_macro.xacro (robot description, xacro)
@@ -20,5 +20,5 @@
         <link name="${prefix}link_1">
             <visual>
-                <origin rpy="0 0 3.1416" xyz="0 0 0"/>
+                <origin rpy="0 0 ${radians(180)}" xyz="0 0 0"/>
                 <geometry>
                     <mesh filename="package://motoman_sia20d_support/meshes/sia20d/visual/link_1.stl"/>
@@ -27,5 +27,5 @@
             </visual>
             <collision>
-                <origin rpy="0 0 3.1416" xyz="0 0 0"/>
+                <origin rpy="0 0 ${radians(180)}" xyz="0 0 0"/>
                 <geometry>
                     <mesh filename="package://motoman_sia20d_support/meshes/sia20d/collision/link_1.stl" />
@@ -36,5 +36,5 @@
         <link name="${prefix}link_2">
             <visual>
-                <origin rpy="1.57 3.1416 3.1416" xyz="0 0 0"/>
+                <origin rpy="${radians(90)} ${radians(180)} ${radians(180)}" xyz="0 0 0"/>
                 <geometry>
                     <mesh filename="package://motoman_sia20d_support/meshes/sia20d/visual/link_2.stl"/>
@@ -43,5 +43,5 @@
             </visual>
             <collision>
-                <origin rpy="1.57 3.1416 3.1416" xyz="0 0 0"/>
+                <origin rpy="${radians(90)} ${radians(180)} ${radians(180)}" xyz="0 0 0"/>
                 <geometry>
                     <mesh filename="package://motoman_sia20d_support/meshes/sia20d/collision/link_2.stl"/>
@@ -68,5 +68,5 @@
         <link name="${prefix}link_4">
             <visual>
-                <origin rpy="1.57 -3.1415 3.1416" xyz="0 0 0"/>
+                <origin rpy="${radians(90)} ${radians(-180)} ${radians(180)}" xyz="0 0 0"/>
                 <geometry>
                     <mesh filename="package://motoman_sia20d_support/meshes/sia20d/visual/link_4.stl"/>
@@ -75,5 +75,5 @@
             </visual>
             <collision>
-                <origin rpy="1.57 -3.1415 3.1416" xyz="0 0 0"/>
+                <origin rpy="${radians(90)} ${radians(-180)} ${radians(180)}" xyz="0 0 0"/>
                 <geometry>
                     <mesh filename="package://motoman_sia20d_support/meshes/sia20d/collision/link_4.stl"/>
@@ -100,5 +100,5 @@
         <link name="${prefix}link_6">
             <visual>
-                <origin rpy="-1.57 0 0" xyz="0 0 0"/>
+                <origin rpy="${radians(-90)} 0 0" xyz="0 0 0"/>
                 <geometry>
                     <mesh filename="package://motoman_sia20d_support/meshes/sia20d/visual/link_6.stl"/>
@@ -107,5 +107,5 @@
             </visual>
             <collision>
-                <origin rpy="-1.57 0 0" xyz="0 0 0"/>
+                <origin rpy="${radians(-90)} 0 0" xyz="0 0 0"/>
                 <geometry>
                     <mesh filename="package://motoman_sia20d_support/meshes/sia20d/collision/link_6.stl"/>
@@ -135,5 +135,5 @@
             <origin xyz="0 0 0.41" rpy="0 0 0"/>
             <axis xyz="0 0 1" />
-            <limit lower="-3.1415" upper="3.1415" effort="100" velocity="2.2689" />
+            <limit lower="${radians(-180)}" upper="${radians(180)}" effort="100" velocity="${radians(130)}" />
         </joint>
         <joint name="${prefix}joint_2" type="revolute">
@@ -142,5 +142,5 @@
             <origin xyz="0 0 0" rpy="0 0 0"/>
             <axis xyz="0 1 0" />
-            <limit lower="-1.9198" upper="1.9198" effort="100" velocity="2.2689" />
+            <limit lower="${radians(-110)}" upper="${radians(110)}" effort="100" velocity="${radians(130)}" />
         </joint>
         <joint name="${prefix}joint_3" type="revolute">
@@ -149,5 +149,5 @@
             <origin xyz="0 0 0.49" rpy="0 0 0"/>
             <axis xyz="0 0 1" />
-            <limit lower="-2.9670" upper="2.9670" effort="100" velocity="2.9670" />
+            <limit lower="${radians(-170)}" upper="${radians(170)}" effort="100" velocity="${radians(170)}" />
         </joint>
         <joint name="${prefix}joint_4" type="revolute">
@@ -156,5 +156,5 @@
             <origin xyz="0 0 0" rpy="0 0 0"/>
             <axis xyz="0 -1 0" />
-            <limit lower="-2.2689" upper="2.2689" effort="100" velocity="2.9670" />
+            <limit lower="${radians(-130)}" upper="${radians(130)}" effort="100" velocity="${radians(170)}" />
         </joint>
         <joint name="${prefix}joint_5" type="revolute">
@@ -163,5 +163,5 @@
             <origin xyz="0 0 0.420" rpy="0 0 0"/>
             <axis xyz="0 0 -1" />
-            <limit lower="-3.1415" upper="3.1415" effort="100" velocity="3.4906" />
+            <limit lower="${radians(-180)}" upper="${radians(180)}" effort="100" velocity="${radians(200)}" />
         </joint>
         <joint name="${prefix}joint_6" type="revolute">
@@ -170,5 +170,5 @@
             <origin xyz="0 0 0" rpy="0 0 0"/>
             <axis xyz="0 -1 0" />
-            <limit lower="-1.9198" upper="1.9198" effort="100" velocity="3.4906" />
+            <limit lower="${radians(-110)}" upper="${radians(110)}" effort="100" velocity="${radians(200)}" />
         </joint>
         <joint name="${prefix}joint_7" type="revolute">
@@ -177,5 +177,5 @@
             <origin xyz="0 0 0.18" rpy="0 0 0"/>
             <axis xyz="0 0 -1" />
-            <limit lower="-3.1415" upper="3.1415" effort="100" velocity="6.9813" />
+            <limit lower="${radians(-180)}" upper="${radians(180)}" effort="100" velocity="${radians(400)}" />
         </joint>
         <!-- end of joint list -->
@@ -190,5 +190,5 @@
         <link name="${prefix}flange"/>
         <joint name="${prefix}joint_7-flange" type="fixed">
-            <origin xyz="0 0 0" rpy="0 -1.57079632679 0"/>
+            <origin xyz="0 0 0" rpy="0 ${radians(-90)} 0"/>
             <parent link="${prefix}link_7"/>
             <child link="${prefix}flange"/>
@@ -197,5 +197,5 @@
         <link name="${prefix}tool0"/>
         <joint name="${prefix}flange-tool0" type="fixed">
-            <origin xyz="0 0 0 " rpy="0 -1.57079632679 3.1415296"/>
+            <origin xyz="0 0 0" rpy="0 ${radians(-90)} ${radians(180)}"/>
             <parent link="${prefix}flange"/>
             <child link="${prefix}tool0"/>

File: motoman_sia5d_support/urdf/sia5d_macro.xacro (robot description, xacro)
@@ -37,5 +37,5 @@
     <child link="${prefix}link_1" />
     <axis xyz="0 0 1" />
-    <limit lower="${-180*deg}" upper="${180*deg}" effort="0" velocity="${200*deg}" />
+    <limit lower="${radians(-180)}" upper="${radians(180)}" effort="0" velocity="${radians(200)}" />
   </joint>
   <link name="${prefix}link_2">
@@ -58,5 +58,5 @@
     <child link="${prefix}link_2" />
     <axis xyz="0 1 0" />
-    <limit lower="${-110*deg}" upper="${110*deg}" effort="0" velocity="${200*deg}" />
+    <limit lower="${radians(-110)}" upper="${radians(110)}" effort="0" velocity="${radians(200)}" />
   </joint>
   <link name="${prefix}link_3">
@@ -79,5 +79,5 @@
     <child link="${prefix}link_3" />
     <axis xyz="0 0 1" />
-    <limit lower="${-170*deg}" upper="${170*deg}" effort="0" velocity="${200*deg}" />
+    <limit lower="${radians(-170)}" upper="${radians(170)}" effort="0" velocity="${radians(200)}" />
   </joint>
   <link name="${prefix}link_4">
@@ -100,5 +100,5 @@
     <child link="${prefix}link_4" />
     <axis xyz="0 -1 0" />
-    <limit lower="${-90*deg}" upper="${115*deg}" effort="0"  velocity="${200*deg}" />
+    <limit lower="${radians(-90)}" upper="${radians(115)}" effort="0" velocity="${radians(200)}" />
   </joint>
   <link name="${prefix}link_5">
@@ -121,5 +121,5 @@
     <child link="${prefix}link_5" />
     <axis xyz="-1 0 0" />
-    <limit lower="${-90*deg}" upper="${90*deg}" effort="0" velocity="${200*deg}" />
+    <limit lower="${radians(-90)}" upper="${radians(90)}" effort="0" velocity="${radians(200)}" />
   </joint>
   <link name="${prefix}link_6">
@@ -142,5 +142,5 @@
     <child link="${prefix}link_6" />
     <axis xyz="0 -1 0" />
-    <limit lower="${-110*deg}" upper="${110*deg}" effort="0" velocity="${230*deg}" />
+    <limit lower="${radians(-110)}" upper="${radians(110)}" effort="0" velocity="${radians(230)}" />
   </joint>
   <link name="${prefix}link_7">
@@ -163,5 +163,5 @@
     <child link="${prefix}link_7" />
     <axis xyz="-1 0 0" />
-    <limit lower="${-90*deg}" upper="${90*deg}" effort="0" velocity="${350*deg}" />
+    <limit lower="${radians(-90)}" upper="${radians(90)}" effort="0" velocity="${radians(350)}" />
   </joint>
   <!-- end of joint list -->
@@ -183,5 +183,5 @@
   <link name="${prefix}tool0"/>
   <joint name="${prefix}flange-tool0" type="fixed">
-    <origin xyz="0 0 0 " rpy="${180*deg} ${-90*deg} 0"/>
+    <origin xyz="0 0 0" rpy="${radians(180)} ${radians(-90)} 0"/>
     <parent link="${prefix}flange"/>
     <child link="${prefix}tool0"/>
