Commit message: Fix ar2010 joint limits

File: motoman_ar2010_support/urdf/ar2010_macro.xacro (robot description, xacro)
@@ -124,5 +124,5 @@
       <origin xyz="0.200 -1.082 0" rpy="${radians(-90)} 0 0"/>
       <axis xyz="0 0 1"/>
-      <limit lower="${radians(-150)}" upper="${radians(150)}" effort="78.4" velocity="${radians(435)}"/>
+      <limit lower="${radians(-200)}" upper="${radians(200)}" effort="78.4" velocity="${radians(435)}"/>
     </joint>
     <joint name="${prefix}joint_5" type="revolute">
@@ -131,5 +131,5 @@
       <origin xyz="0 0 0" rpy="${radians(90)} 0 0"/>
       <axis xyz="0 0 1"/>
-      <limit lower="${radians(-135)}" upper="${radians(90)}" effort="67.03" velocity="${radians(435)}"/>
+      <limit lower="${radians(-150)}" upper="${radians(150)}" effort="67.03" velocity="${radians(435)}"/>
     </joint>
     <joint name="${prefix}joint_6" type="revolute">
@@ -138,5 +138,5 @@
       <origin xyz="0 -0.100 0" rpy="${radians(-90)} 0 0"/>
       <axis xyz="0 0 1"/>
-      <limit lower="${radians(-210)}" upper="${radians(210)}" effort="33.3" velocity="${radians(700)}"/>
+      <limit lower="${radians(-455)}" upper="${radians(455)}" effort="33.3" velocity="${radians(700)}"/>
     </joint>
     <!-- end of joint list -->
