Commit message: replace 'radians(0)' with 0

File: motoman_gp180_support/urdf/gp180_macro.xacro (robot description, xacro)
@@ -32,5 +32,5 @@
     <link name="${prefix}link_2">
         <visual>
-            <origin rpy="${radians(90)} ${radians(0)} ${radians(90)}" />
+            <origin rpy="${radians(90)} 0 ${radians(90)}" />
             <geometry>
                 <mesh filename="package://motoman_gp180_support/meshes/gp180_120/visual/link_2.stl"/>
@@ -39,5 +39,5 @@
         </visual>
         <collision>
-            <origin rpy="${radians(90)} ${radians(0)} ${radians(90)}" />
+            <origin rpy="${radians(90)} 0 ${radians(90)}" />
             <geometry>
                 <mesh filename="package://motoman_gp180_support/meshes/gp180_120/collision/link_2.stl"/>
@@ -47,5 +47,5 @@
     <link name="${prefix}link_3">
         <visual>
-            <origin rpy="${radians(-90)} ${radians(0)} ${radians(-90)}" />
+            <origin rpy="${radians(-90)} 0 ${radians(-90)}" />
             <geometry>
                 <mesh filename="package://motoman_gp180_support/meshes/gp180/visual/link_3.stl"/>
@@ -54,5 +54,5 @@
         </visual>
         <collision>
-            <origin rpy="${radians(-90)} ${radians(0)} ${radians(-90)}" />
+            <origin rpy="${radians(-90)} 0 ${radians(-90)}" />
             <geometry>
                 <mesh filename="package://motoman_gp180_support/meshes/gp180/collision/link_3.stl"/>
@@ -62,5 +62,5 @@
     <link name="${prefix}link_4">
         <visual>
-            <origin rpy="${radians(0)} ${radians(90)} ${radians(0)}" xyz="0 0 1.225"/>
+            <origin rpy="0 ${radians(90)} 0" xyz="0 0 1.225"/>
             <geometry>
                 <mesh filename="package://motoman_gp180_support/meshes/gp180/visual/link_4.stl"/>
@@ -69,5 +69,5 @@
         </visual>
         <collision>
-            <origin rpy="${radians(0)} ${radians(90)} ${radians(0)}" xyz="0 0 1.225"/>
+            <origin rpy="0 ${radians(90)} 0" xyz="0 0 1.225"/>
             <geometry>
                 <mesh filename="package://motoman_gp180_support/meshes/gp180/collision/link_4.stl"/>
@@ -77,5 +77,5 @@
     <link name="${prefix}link_5">
         <visual>
-            <origin rpy="${radians(-90)} ${radians(0)} ${radians(-90)}" />
+            <origin rpy="${radians(-90)} 0 ${radians(-90)}" />
             <geometry>
                 <mesh filename="package://motoman_gp180_support/meshes/gp180_120/visual/link_5.stl"/>
@@ -84,5 +84,5 @@
         </visual>
         <collision>
-            <origin rpy="${radians(-90)} ${radians(0)} ${radians(-90)}" />
+            <origin rpy="${radians(-90)} 0 ${radians(-90)}" />
             <geometry>
                 <mesh filename="package://motoman_gp180_support/meshes/gp180_120/collision/link_5.stl"/>
@@ -92,5 +92,5 @@
     <link name="${prefix}link_6">
         <visual>
-            <origin rpy="${radians(0)} ${radians(90)} ${radians(0)}" />
+            <origin rpy="0 ${radians(90)} 0" />
             <geometry>
                 <mesh filename="package://motoman_gp180_support/meshes/gp180_120/visual/link_6.stl"/>
@@ -99,5 +99,5 @@
         </visual>
         <collision>
-            <origin rpy="${radians(0)} ${radians(90)} ${radians(0)}" />
+            <origin rpy="0 ${radians(90)} 0" />
             <geometry>
                 <mesh filename="package://motoman_gp180_support/meshes/gp180_120/collision/link_6.stl"/>

Commit message: Fix gp180 effort

File: motoman_gp180_support/urdf/gp180_macro.xacro (robot description, xacro)
@@ -140,5 +140,5 @@
         <origin xyz="0 0 0" rpy="${radians(90)} 0 0" />
         <axis xyz="0 0 1" />
-        <limit lower="${radians(-130)}" upper="${radians(130)}" effort="1081.18" velocity="${radians(175)}"/>
+        <limit lower="${radians(-130)}" upper="${radians(130)}" effort="1765.20" velocity="${radians(175)}"/>
     </joint>
     <joint name="${prefix}joint_6" type="revolute">
@@ -147,5 +147,5 @@
         <origin xyz="0 -0.225 0" rpy="${radians(-90)} 0 0" />
         <axis xyz="0 0 1" />
-        <limit lower="${radians(-360)}" upper="${radians(360)}" effort="926.73" velocity="${radians(265)}"/>
+        <limit lower="${radians(-360)}" upper="${radians(360)}" effort="1081.18" velocity="${radians(265)}"/>
     </joint>
     <!-- end of joint list -->
