Commit message: Fix gp200r joint limits

File: motoman_gp200r_support/urdf/gp200r_macro.xacro (robot description, xacro)
@@ -124,5 +124,5 @@
         <origin xyz="0.250 0 0" rpy="0 ${radians(90)} 0" />
         <axis xyz="-1 0 0" />
-        <limit lower="${radians(-180)}" upper="${radians(180)}" effort="2621.3" velocity="${radians(120)}"/>
+        <limit lower="${radians(-360)}" upper="${radians(360)}" effort="2621.3" velocity="${radians(120)}"/>
     </joint>
     <joint name="${prefix}joint_5" type="revolute">
@@ -131,5 +131,5 @@
         <origin xyz="1.225 0 0" rpy="0 0 0" />
         <axis xyz="0 -1 0" />
-        <limit lower="${radians(-125)}" upper="${radians(180)}" effort="3530.38" velocity="${radians(120)}"/>
+        <limit lower="${radians(-125)}" upper="${radians(125)}" effort="3530.38" velocity="${radians(120)}"/>
     </joint>
     <joint name="${prefix}joint_6" type="revolute">
@@ -138,5 +138,5 @@
         <origin xyz="0.250 0 0" rpy="0 0 0" />
         <axis xyz="1 0 0" />
-        <limit lower="${radians(-180)}" upper="${radians(180)}" effort="1765.19" velocity="${radians(190)}"/>
+        <limit lower="${radians(-360)}" upper="${radians(360)}" effort="1765.19" velocity="${radians(190)}"/>
     </joint>
     <!-- end of joint list -->
