Commit message: Add flange to gp88

File: motoman_gp88_support/urdf/gp88_macro.xacro (robot description, xacro)
@@ -147,9 +147,16 @@
       <child link="${prefix}base"/>
     </joint>
+    <!-- ROS-Industrial 'flange' frame: attachment point for EEF models -->
+    <link name="${prefix}flange" />
+    <joint name="${prefix}joint_6_t-flange" type="fixed">
+        <origin xyz="0.175 0 0" rpy="0 0 0" />
+        <parent link="${prefix}link_6_t" />
+        <child link="${prefix}flange" />
+    </joint>
     <!-- ROS-Industrial 'tool0' frame: all-zeros tool frame -->
     <link name="${prefix}tool0"/>
-    <joint name="${prefix}joint_6_t-tool0" type="fixed">
-      <origin xyz="0.175 0 0" rpy="${radians(180)} ${radians(-90)} 0"/>
-      <parent link="${prefix}link_6_t"/>
+    <joint name="${prefix}flange-tool0" type="fixed">
+      <origin xyz="0 0 0" rpy="${radians(180)} ${radians(-90)} 0"/>
+      <parent link="${prefix}flange"/>
       <child link="${prefix}tool0"/>
     </joint>

Commit message: Fix GP88 effort

File: motoman_gp88_support/urdf/gp88_macro.xacro (robot description, xacro)
@@ -109,5 +109,5 @@
       <origin xyz="0.320 0 0" rpy="0 0 0" />
       <axis xyz="0 1 0" />
-      <limit lower="${radians(-90)}" upper="${radians(155)}" effort="7353.05" velocity="${radians(140)}"/>
+      <limit lower="${radians(-90)}" upper="${radians(155)}" effort="7453.05" velocity="${radians(140)}"/>
     </joint>
     <joint name="${prefix}joint_3" type="revolute">
