Commit message: Fix MH12 `joint_4` axis limits

File: motoman_mh12_support/urdf/mh12_macro.xacro (robot description, xacro)
@@ -124,5 +124,5 @@
         <origin xyz="0.640 0 0.200" rpy="0 0 0" />
         <axis xyz="-1 0 0" />
-        <limit lower="${radians(-180)}" upper="${radians(-180)}" effort="74.97" velocity="${radians(410)}"/>
+        <limit lower="${radians(-180)}" upper="${radians(180)}" effort="74.97" velocity="${radians(410)}"/>
     </joint>
     <joint name="${prefix}joint_5_b" type="revolute">

Commit message: Add `flange` and `tool0` for single-arm robots and positioners

File: motoman_mh12_support/urdf/mh12_macro.xacro (robot description, xacro)
@@ -95,5 +95,4 @@
         </collision>
     </link>
-    <link name="${prefix}tool0"/>
     <!-- end of link list -->
     <!-- joint list -->
@@ -124,5 +123,5 @@
         <origin xyz="0.640 0 0.200" rpy="0 0 0" />
         <axis xyz="-1 0 0" />
-        <limit lower="${radians(-180)}" upper="${radians(180)}" effort="74.97" velocity="${radians(410)}"/>
+        <limit lower="${radians(-180)}" upper="${radians(-180)}" effort="74.97" velocity="${radians(410)}"/>
     </joint>
     <joint name="${prefix}joint_5_b" type="revolute">
@@ -140,8 +139,17 @@
         <limit lower="${radians(-360)}" upper="${radians(360)}" effort="14.80" velocity="${radians(610)}"/>
     </joint>
-    <joint name="${prefix}joint_6_t-tool0" type="fixed">
-        <origin xyz="0.100 0 0" rpy="3.1415926 -1.570796 0"/>
-        <parent link="${prefix}link_6_t"/>
-        <child link="${prefix}tool0"/>
+    <!-- ROS-Industrial 'flange' frame: attachment point for EEF models -->
+    <link name="${prefix}flange"/>
+    <joint name="${prefix}joint_6_t-flange" type="fixed">
+      <origin xyz="0.100 0 0" rpy="0 0 0"/>
+      <parent link="${prefix}link_6_t"/>
+      <child link="${prefix}flange"/>
+    </joint>
+    <!-- ROS-Industrial 'tool0' frame: all-zeros tool frame -->
+    <link name="${prefix}tool0"/>
+    <joint name="${prefix}flange-tool0" type="fixed">
+      <origin xyz="0 0 0" rpy="3.1415926 -1.570796 0"/>
+      <parent link="${prefix}flange"/>
+      <child link="${prefix}tool0"/>
     </joint>
     <!-- end of joint list -->

Commit message: Fix inaccurate link_3 ranges

File: motoman_mh12_support/urdf/mh12_macro.xacro (robot description, xacro)
@@ -116,5 +116,5 @@
         <origin xyz="0 0 0.614" rpy="0 0 0" />
         <axis xyz="0 -1 0" />
-        <limit lower="${radians(-175)}" upper="${radians(240)}" effort="257.25" velocity="${radians(220)}"/>
+        <limit lower="${radians(-85)}" upper="${radians(150)}" effort="257.25" velocity="${radians(220)}"/>
     </joint>
     <joint name="${prefix}joint_4" type="revolute">

File: motoman_ms210_support/urdf/ms210_macro.xacro (robot description, xacro)
@@ -130,5 +130,5 @@
     <origin xyz="0 0 1.150" rpy="0 0 0" />
     <axis xyz="0 -1 0" />
-    <limit lower="${radians(-147)}" upper="${radians(90)}" effort="9806.65" velocity="${radians(115)}" />
+    <limit lower="${radians(-86)}" upper="${radians(90)}" effort="9806.65" velocity="${radians(115)}" />
   </joint>
   <joint name="${prefix}joint_4" type="revolute">
