Commit message: fix hc10 and hc10dt effort values

File: motoman_hc10_support/urdf/hc10_macro.xacro (robot description, xacro)
@@ -123,5 +123,5 @@
       <origin xyz="0 0 -0.500" rpy="0 0 0" />
       <axis xyz="0 0 1" />
-      <limit lower="${radians(-180)}" upper="${radians(180)}" effort="39.20" velocity="${radians(180)}"/>
+      <limit lower="${radians(-180)}" upper="${radians(180)}" effort="31.36" velocity="${radians(180)}"/>
     </joint>
     <joint name="${prefix}joint_5" type="revolute">

File: motoman_hc10_support/urdf/hc10dt_macro.xacro (robot description, xacro)
@@ -123,5 +123,5 @@
       <origin xyz="0 0 -0.500" rpy="0 0 0" />
       <axis xyz="0 0 1" />
-      <limit lower="${radians(-180)}" upper="${radians(180)}" effort="39.20" velocity="${radians(180)}"/>
+      <limit lower="${radians(-180)}" upper="${radians(180)}" effort="31.36" velocity="${radians(180)}"/>
     </joint>
     <joint name="${prefix}joint_5" type="revolute">
