Commit message: rename hc20 to hc20dt

File: motoman_hc20_support/urdf/hc20dt_macro.xacro (robot description, xacro)
@@ -1,5 +1,5 @@
 <?xml version="1.0" ?>
 <robot xmlns:xacro="http://ros.org/wiki/xacro">
-  <xacro:macro name="motoman_hc20" params="prefix">
+  <xacro:macro name="motoman_hc20dt" params="prefix">
     <xacro:include filename="$(find motoman_resources)/urdf/common_materials.xacro"/>
     <!-- link list -->
@@ -7,5 +7,5 @@
       <visual>
         <geometry>
-          <mesh filename="package://motoman_hc20_support/meshes/hc20/visual/base_link.dae"/>
+          <mesh filename="package://motoman_hc20_support/meshes/hc20dt/visual/base_link.dae"/>
         </geometry>
         <xacro:material_yaskawa_white/>
@@ -13,5 +13,5 @@
       <collision>
         <geometry>
-          <mesh filename="package://motoman_hc20_support/meshes/hc20/collision/base_link.stl"/>
+          <mesh filename="package://motoman_hc20_support/meshes/hc20dt/collision/base_link.stl"/>
         </geometry>
       </collision>
@@ -20,5 +20,5 @@
       <visual>
         <geometry>
-          <mesh filename="package://motoman_hc20_support/meshes/hc20/visual/link_1.dae"/>
+          <mesh filename="package://motoman_hc20_support/meshes/hc20dt/visual/link_1.dae"/>
         </geometry>
         <xacro:material_yaskawa_white/>
@@ -26,5 +26,5 @@
       <collision>
         <geometry>
-          <mesh filename="package://motoman_hc20_support/meshes/hc20/collision/link_1.stl"/>
+          <mesh filename="package://motoman_hc20_support/meshes/hc20dt/collision/link_1.stl"/>
         </geometry>
       </collision>
@@ -33,5 +33,5 @@
       <visual>
         <geometry>
-          <mesh filename="package://motoman_hc20_support/meshes/hc20/visual/link_2.dae"/>
+          <mesh filename="package://motoman_hc20_support/meshes/hc20dt/visual/link_2.dae"/>
         </geometry>
         <xacro:material_yaskawa_white/>
@@ -39,5 +39,5 @@
       <collision>
         <geometry>
-          <mesh filename="package://motoman_hc20_support/meshes/hc20/collision/link_2.stl"/>
+          <mesh filename="package://motoman_hc20_support/meshes/hc20dt/collision/link_2.stl"/>
         </geometry>
       </collision>
@@ -46,5 +46,5 @@
       <visual>
         <geometry>
-          <mesh filename="package://motoman_hc20_support/meshes/hc20/visual/link_3.dae"/>
+          <mesh filename="package://motoman_hc20_support/meshes/hc20dt/visual/link_3.dae"/>
         </geometry>
         <xacro:material_yaskawa_white/>
@@ -52,5 +52,5 @@
       <collision>
         <geometry>
-          <mesh filename="package://motoman_hc20_support/meshes/hc20/collision/link_3.stl"/>
+          <mesh filename="package://motoman_hc20_support/meshes/hc20dt/collision/link_3.stl"/>
         </geometry>
       </collision>
@@ -59,5 +59,5 @@
       <visual>
         <geometry>
-          <mesh filename="package://motoman_hc20_support/meshes/hc20/visual/link_4.dae"/>
+          <mesh filename="package://motoman_hc20_support/meshes/hc20dt/visual/link_4.dae"/>
         </geometry>
         <xacro:material_yaskawa_white/>
@@ -65,5 +65,5 @@
       <collision>
         <geometry>
-          <mesh filename="package://motoman_hc20_support/meshes/hc20/collision/link_4.stl"/>
+          <mesh filename="package://motoman_hc20_support/meshes/hc20dt/collision/link_4.stl"/>
         </geometry>
       </collision>
@@ -72,5 +72,5 @@
       <visual>
         <geometry>
-          <mesh filename="package://motoman_hc20_support/meshes/hc20/visual/link_5.dae"/>
+          <mesh filename="package://motoman_hc20_support/meshes/hc20dt/visual/link_5.dae"/>
         </geometry>
         <xacro:material_yaskawa_white/>
@@ -78,5 +78,5 @@
       <collision>
         <geometry>
-          <mesh filename="package://motoman_hc20_support/meshes/hc20/collision/link_5.stl"/>
+          <mesh filename="package://motoman_hc20_support/meshes/hc20dt/collision/link_5.stl"/>
         </geometry>
       </collision>
@@ -85,5 +85,5 @@
       <visual>
         <geometry>
-          <mesh filename="package://motoman_hc20_support/meshes/hc20/visual/link_6.dae"/>
+          <mesh filename="package://motoman_hc20_support/meshes/hc20dt/visual/link_6.dae"/>
         </geometry>
         <xacro:material_yaskawa_white/>
@@ -91,5 +91,5 @@
       <collision>
         <geometry>
-          <mesh filename="package://motoman_hc20_support/meshes/hc20/collision/link_6.stl"/>
+          <mesh filename="package://motoman_hc20_support/meshes/hc20dt/collision/link_6.stl"/>
         </geometry>
       </collision>

File: motoman_hc20_support/urdf/hc20dtp_macro.xacro (robot description, xacro)
@@ -7,5 +7,5 @@
       <visual>
         <geometry>
-          <mesh filename="package://motoman_hc20_support/meshes/hc20/visual/base_link.dae"/>
+          <mesh filename="package://motoman_hc20_support/meshes/hc20dt/visual/base_link.dae"/>
         </geometry>
         <xacro:material_yaskawa_white/>
@@ -13,5 +13,5 @@
       <collision>
         <geometry>
-          <mesh filename="package://motoman_hc20_support/meshes/hc20/collision/base_link.stl"/>
+          <mesh filename="package://motoman_hc20_support/meshes/hc20dt/collision/base_link.stl"/>
         </geometry>
       </collision>
@@ -20,5 +20,5 @@
       <visual>
         <geometry>
-          <mesh filename="package://motoman_hc20_support/meshes/hc20/visual/link_1.dae"/>
+          <mesh filename="package://motoman_hc20_support/meshes/hc20dt/visual/link_1.dae"/>
         </geometry>
         <xacro:material_yaskawa_white/>
@@ -26,5 +26,5 @@
       <collision>
         <geometry>
-          <mesh filename="package://motoman_hc20_support/meshes/hc20/collision/link_1.stl"/>
+          <mesh filename="package://motoman_hc20_support/meshes/hc20dt/collision/link_1.stl"/>
         </geometry>
       </collision>
@@ -33,5 +33,5 @@
       <visual>
         <geometry>
-          <mesh filename="package://motoman_hc20_support/meshes/hc20/visual/link_2.dae"/>
+          <mesh filename="package://motoman_hc20_support/meshes/hc20dt/visual/link_2.dae"/>
         </geometry>
         <xacro:material_yaskawa_white/>
@@ -39,5 +39,5 @@
       <collision>
         <geometry>
-          <mesh filename="package://motoman_hc20_support/meshes/hc20/collision/link_2.stl"/>
+          <mesh filename="package://motoman_hc20_support/meshes/hc20dt/collision/link_2.stl"/>
         </geometry>
       </collision>
@@ -46,5 +46,5 @@
       <visual>
         <geometry>
-          <mesh filename="package://motoman_hc20_support/meshes/hc20/visual/link_3.dae"/>
+          <mesh filename="package://motoman_hc20_support/meshes/hc20dt/visual/link_3.dae"/>
         </geometry>
         <xacro:material_yaskawa_white/>
@@ -52,5 +52,5 @@
       <collision>
         <geometry>
-          <mesh filename="package://motoman_hc20_support/meshes/hc20/collision/link_3.stl"/>
+          <mesh filename="package://motoman_hc20_support/meshes/hc20dt/collision/link_3.stl"/>
         </geometry>
       </collision>
@@ -59,5 +59,5 @@
       <visual>
         <geometry>
-          <mesh filename="package://motoman_hc20_support/meshes/hc20/visual/link_4.dae"/>
+          <mesh filename="package://motoman_hc20_support/meshes/hc20dt/visual/link_4.dae"/>
         </geometry>
         <xacro:material_yaskawa_white/>
@@ -65,5 +65,5 @@
       <collision>
         <geometry>
-          <mesh filename="package://motoman_hc20_support/meshes/hc20/collision/link_4.stl"/>
+          <mesh filename="package://motoman_hc20_support/meshes/hc20dt/collision/link_4.stl"/>
         </geometry>
       </collision>

File: motoman_hc20_support/urdf/hc30pl_macro.xacro (robot description, xacro)
@@ -7,5 +7,5 @@
       <visual>
         <geometry>
-          <mesh filename="package://motoman_hc20_support/meshes/hc20/visual/base_link.dae"/>
+          <mesh filename="package://motoman_hc20_support/meshes/hc20dt/visual/base_link.dae"/>
         </geometry>
         <xacro:material_yaskawa_white/>
@@ -13,5 +13,5 @@
       <collision>
         <geometry>
-          <mesh filename="package://motoman_hc20_support/meshes/hc20/collision/base_link.stl"/>
+          <mesh filename="package://motoman_hc20_support/meshes/hc20dt/collision/base_link.stl"/>
         </geometry>
       </collision>
@@ -20,5 +20,5 @@
       <visual>
         <geometry>
-          <mesh filename="package://motoman_hc20_support/meshes/hc20/visual/link_1.dae"/>
+          <mesh filename="package://motoman_hc20_support/meshes/hc20dt/visual/link_1.dae"/>
         </geometry>
         <xacro:material_yaskawa_white/>
@@ -26,5 +26,5 @@
       <collision>
         <geometry>
-          <mesh filename="package://motoman_hc20_support/meshes/hc20/collision/link_1.stl"/>
+          <mesh filename="package://motoman_hc20_support/meshes/hc20dt/collision/link_1.stl"/>
         </geometry>
       </collision>
@@ -33,5 +33,5 @@
       <visual>
         <geometry>
-          <mesh filename="package://motoman_hc20_support/meshes/hc20/visual/link_2.dae"/>
+          <mesh filename="package://motoman_hc20_support/meshes/hc20dt/visual/link_2.dae"/>
         </geometry>
         <xacro:material_yaskawa_white/>
@@ -39,5 +39,5 @@
       <collision>
         <geometry>
-          <mesh filename="package://motoman_hc20_support/meshes/hc20/collision/link_2.stl"/>
+          <mesh filename="package://motoman_hc20_support/meshes/hc20dt/collision/link_2.stl"/>
         </geometry>
       </collision>
@@ -46,5 +46,5 @@
       <visual>
         <geometry>
-          <mesh filename="package://motoman_hc20_support/meshes/hc20/visual/link_3.dae"/>
+          <mesh filename="package://motoman_hc20_support/meshes/hc20dt/visual/link_3.dae"/>
         </geometry>
         <xacro:material_yaskawa_white/>
@@ -52,5 +52,5 @@
       <collision>
         <geometry>
-          <mesh filename="package://motoman_hc20_support/meshes/hc20/collision/link_3.stl"/>
+          <mesh filename="package://motoman_hc20_support/meshes/hc20dt/collision/link_3.stl"/>
         </geometry>
       </collision>
@@ -59,5 +59,5 @@
       <visual>
         <geometry>
-          <mesh filename="package://motoman_hc20_support/meshes/hc20/visual/link_4.dae"/>
+          <mesh filename="package://motoman_hc20_support/meshes/hc20dt/visual/link_4.dae"/>
         </geometry>
         <xacro:material_yaskawa_white/>
@@ -65,5 +65,5 @@
       <collision>
         <geometry>
-          <mesh filename="package://motoman_hc20_support/meshes/hc20/collision/link_4.stl"/>
+          <mesh filename="package://motoman_hc20_support/meshes/hc20dt/collision/link_4.stl"/>
         </geometry>
       </collision>
