Commit message: Fix hc30pl flange

File: motoman_hc20_support/urdf/hc30pl_macro.xacro (robot description, xacro)
@@ -156,5 +156,5 @@
     <link name="${prefix}flange"/>
     <joint name="${prefix}joint_6-flange" type="fixed">
-      <origin xyz="0 0 -0.200" rpy="0 0 0"/>
+      <origin xyz="0 0 -0.200" rpy="0 ${radians(90)} 0"/>
       <parent link="${prefix}link_6"/>
       <child link="${prefix}flange"/>
@@ -163,5 +163,5 @@
     <link name="${prefix}tool0"/>
     <joint name="${prefix}flange-tool0" type="fixed">
-      <origin xyz="0 0 0" rpy="0 ${radians(180)} ${radians(180)}"/>
+      <origin xyz="0 0 0" rpy="${radians(180)} ${radians(-90)} 0"/>
       <parent link="${prefix}flange"/>
       <child link="${prefix}tool0"/>
