Commit message: Remove `world` link and transform

File: motoman_sia10d_support/urdf/sia10d_macro.xacro (robot description, xacro)
@@ -4,7 +4,4 @@
         <xacro:include filename="$(find motoman_resources)/urdf/common_materials.xacro"/>
         <!-- link list -->
-        <link name="world">
-            <origin xyz="0 0 0" rpy="0 0 0"/>
-        </link>
         <link name="${prefix}base_link">
             <visual>
@@ -131,9 +128,4 @@
         <!-- end of link list -->
         <!-- joint list -->
-        <joint name="world-base" type="fixed">
-            <origin xyz="0 0 0" rpy="0 0 0"/>
-            <parent link="world" />
-            <child link="base_link"/>
-        </joint>
         <joint name="${prefix}joint_1" type="revolute">
             <parent link="${prefix}base_link"/>

Commit message: Remove mass and inertial properties

File: motoman_sia10d_support/urdf/sia10d_macro.xacro (robot description, xacro)
@@ -20,8 +20,4 @@
                 <xacro:material_yaskawa_yellow/>
             </collision>
-            <inertial>
-                    <mass value="400" />  <!-- Arbitrarily large value, to simulate bolting down in case of absence of fixed joint -->
-                    <inertia ixx="1.0" ixy="0.0" ixz="0.0" iyy="1.0" iyz="0.0" izz="1.0"/>
-                </inertial>
         </link>
         <gazebo reference="${prefix}base_link">
@@ -43,9 +39,4 @@
                 <xacro:material_yaskawa_yellow/>
             </collision>
-            <inertial>
-                    <mass value="13.746057" />
-                    <inertia ixx="0.070027808" ixy="0.0" ixz="0.0" iyy="0.077808312" iyz="0.0" izz="0.043654657"/>
-                <origin xyz="0.0 0.0046451930 -0.018976267" rpy="0.0 0.0 0.0"/>
-                </inertial>
         </link>
         <gazebo reference="${prefix}link_s">
@@ -69,9 +60,4 @@
                 <xacro:material_yaskawa_yellow/>
             </collision>
-            <inertial>
-                    <mass value="5.227999" />
-                    <inertia ixx="0.016063413" ixy="0.0" ixz="0.0" iyy="0.10522920" iyz="0.0" izz="0.10250891"/>
-                <origin xyz="0.11422130 0.0 0.018935113" rpy="0.0 0.0 0.0"/>
-                </inertial>
         </link>
         <gazebo reference="${prefix}link_l">
@@ -95,9 +81,4 @@
                 <xacro:material_yaskawa_yellow/>
             </collision>
-            <inertial>
-                    <mass value="4.7092004" />
-                    <inertia ixx="0.030190273" ixy="0.0" ixz="0.0" iyy="0.030943336" iyz="0.0" izz="0.0096760191"/>
-                <origin xyz="0.0 -0.011901001 -0.036023969" rpy="0.0 0.0 0.0"/>
-                </inertial>
         </link>
         <gazebo reference="${prefix}link_e">
@@ -121,9 +102,4 @@
                 <xacro:material_yaskawa_yellow/>
             </collision>
-            <inertial>
-                    <mass value="3.1488649" />
-                    <inertia ixx="0.083840132" ixy="0.0" ixz="0.0" iyy="0.0061641860" iyz="0.0" izz="0.083291837"/>
-                <origin xyz="0.0 -0.015659426 0.13525753" rpy="0.0 0.0 0.0"/>
-                </inertial>
         </link>
         <gazebo reference="${prefix}link_u">
@@ -147,9 +123,4 @@
                 <xacro:material_yaskawa_yellow/>
             </collision>
-            <inertial>
-                    <mass value="3.0270943" />
-                    <inertia ixx="0.017471059" ixy="0.0" ixz="0.0" iyy="0.017175292" iyz="0.0" izz="0.0049008824"/>
-                <origin xyz="0.0 -0.011271807 -0.0416" rpy="0.0 0.0 0.0"/>
-                </inertial>
         </link>
         <gazebo reference="${prefix}link_r">
@@ -173,9 +144,4 @@
                 <xacro:material_yaskawa_yellow/>
             </collision>
-            <inertial>
-                    <mass value="2.3902999" />
-                    <inertia ixx="0.080" ixy="0.0" ixz="0.0" iyy="0.0038377449" iyz="0.0" izz="0.080"/>
-                <origin xyz="0.0 0.0074364051 0.078721289" rpy="0.0 0.0 0.0"/>
-                </inertial>
         </link>
         <gazebo reference="${prefix}link_b">
@@ -197,9 +163,4 @@
                 <xacro:material_yaskawa_yellow/>
             </collision>
-            <inertial>
-                    <mass value="0.63670412" />
-                    <inertia ixx="0.00058471221" ixy="0.0" ixz="0.0" iyy="0.0005929671" iyz="0.0" izz="0.001081389"/>
-                <origin xyz="0.0 0.0 0.0" rpy="0.0 0.0 0.0"/>
-                </inertial>
         </link>
         <gazebo reference="${prefix}link_t">

Commit message: Remove gazebo tags

File: motoman_sia10d_support/urdf/sia10d_macro.xacro (robot description, xacro)
@@ -21,9 +21,4 @@
             </collision>
         </link>
-        <gazebo reference="${prefix}base_link">
-                <turnGravityOff>false</turnGravityOff>
-                <selfCollide>true</selfCollide>
-            <material>Gazebo/Blue</material>
-        </gazebo>
         <link name="${prefix}link_s">
             <visual>
@@ -40,9 +35,4 @@
             </collision>
         </link>
-        <gazebo reference="${prefix}link_s">
-                <turnGravityOff>false</turnGravityOff>
-                <selfCollide>true</selfCollide>
-            <material>Gazebo/White</material>
-        </gazebo>
         <link name="${prefix}link_l">
             <visual>
@@ -61,9 +51,4 @@
             </collision>
         </link>
-        <gazebo reference="${prefix}link_l">
-                <turnGravityOff>false</turnGravityOff>
-                <selfCollide>true</selfCollide>
-            <material>Gazebo/Blue</material>
-        </gazebo>
         <link name="${prefix}link_e">
             <visual>
@@ -82,9 +67,4 @@
             </collision>
         </link>
-        <gazebo reference="${prefix}link_e">
-                <turnGravityOff>false</turnGravityOff>
-                <selfCollide>true</selfCollide>
-            <material>Gazebo/White</material>
-        </gazebo>
         <link name="${prefix}link_u">
             <visual>
@@ -103,9 +83,4 @@
             </collision>
         </link>
-        <gazebo reference="${prefix}link_u">
-                <turnGravityOff>false</turnGravityOff>
-                <selfCollide>true</selfCollide>
-            <material>Gazebo/Blue</material>
-        </gazebo>
         <link name="${prefix}link_r">
             <visual>
@@ -124,9 +99,4 @@
             </collision>
         </link>
-        <gazebo reference="${prefix}link_r">
-                <turnGravityOff>false</turnGravityOff>
-                <selfCollide>true</selfCollide>
-            <material>Gazebo/White</material>
-        </gazebo>
         <link name="${prefix}link_b">
             <visual>
@@ -145,9 +115,4 @@
             </collision>
         </link>
-        <gazebo reference="${prefix}link_b">
-                <turnGravityOff>false</turnGravityOff>
-                <selfCollide>true</selfCollide>
-            <material>Gazebo/Blue</material>
-        </gazebo>
         <link name="${prefix}link_t">
             <visual>
@@ -164,9 +129,4 @@
             </collision>
         </link>
-        <gazebo reference="${prefix}link_t">
-                <turnGravityOff>false</turnGravityOff>
-                <selfCollide>true</selfCollide>
-            <material>Gazebo/White</material>
-        </gazebo>
         <!-- end of link list -->
         <!-- joint list -->

Commit message: add missing SIA effort values

File: motoman_sia10d_support/urdf/sia10d_macro.xacro (robot description, xacro)
@@ -141,5 +141,5 @@
             <origin xyz="0 0 0.36" rpy="0 0 0"/>
             <axis xyz="0 0 1" />
-            <limit lower="${radians(-180)}" upper="${radians(180)}" effort="100" velocity="${radians(170)}" />
+            <limit lower="${radians(-180)}" upper="${radians(180)}" effort="268.36" velocity="${radians(170)}" />
         </joint>
         <joint name="${prefix}joint_2" type="revolute">
@@ -148,5 +148,5 @@
             <origin xyz="0 0 0" rpy="0 0 0"/>
             <axis xyz="0 1 0" />
-            <limit lower="${radians(-110)}" upper="${radians(110)}" effort="100" velocity="${radians(170)}" />
+            <limit lower="${radians(-110)}" upper="${radians(110)}" effort="268.36" velocity="${radians(170)}" />
         </joint>
         <joint name="${prefix}joint_3" type="revolute">
@@ -155,5 +155,5 @@
             <origin xyz="0 0 0.36" rpy="0 0 0"/>
             <axis xyz="0 0 1" />
-            <limit lower="${radians(-170)}" upper="${radians(170)}" effort="100" velocity="${radians(170)}" />
+            <limit lower="${radians(-170)}" upper="${radians(170)}" effort="122.89" velocity="${radians(170)}" />
         </joint>
         <joint name="${prefix}joint_4" type="revolute">
@@ -162,5 +162,5 @@
             <origin xyz="0 0 0" rpy="0 0 0"/>
             <axis xyz="0 -1 0" />
-            <limit lower="${radians(-135)}" upper="${radians(135)}" effort="100" velocity="${radians(170)}" />
+            <limit lower="${radians(-135)}" upper="${radians(135)}" effort="122.89" velocity="${radians(170)}" />
         </joint>
         <joint name="${prefix}joint_5" type="revolute">
@@ -169,5 +169,5 @@
             <origin xyz="0 0 0.360" rpy="0 0 0"/>
             <axis xyz="0 0 -1" />
-            <limit lower="${radians(-180)}" upper="${radians(180)}" effort="100" velocity="${radians(200)}" />
+            <limit lower="${radians(-180)}" upper="${radians(180)}" effort="44.34" velocity="${radians(200)}" />
         </joint>
         <joint name="${prefix}joint_6" type="revolute">
@@ -176,5 +176,5 @@
             <origin xyz="0 0 0" rpy="0 0 0"/>
             <axis xyz="0 -1 0" />
-            <limit lower="${radians(-110)}" upper="${radians(110)}" effort="100" velocity="${radians(200)}" />
+            <limit lower="${radians(-110)}" upper="${radians(110)}" effort="44.34" velocity="${radians(200)}" />
         </joint>
         <joint name="${prefix}joint_7" type="revolute">
@@ -183,5 +183,5 @@
             <origin xyz="0 0 0.155" rpy="0 0 0"/>
             <axis xyz="0 0 -1" />
-            <limit lower="${radians(-180)}" upper="${radians(180)}" effort="100" velocity="${radians(400)}" />
+            <limit lower="${radians(-180)}" upper="${radians(180)}" effort="39.04" velocity="${radians(400)}" />
         </joint>
         <!-- end of joint list -->

File: motoman_sia10f_support/urdf/sia10f_macro.xacro (robot description, xacro)
@@ -135,5 +135,5 @@
             <origin xyz="0 0 0.36" rpy="0 0 0"/>
             <axis xyz="0 0 1" />
-            <limit lower="${radians(-180)}" upper="${radians(180)}" effort="0" velocity="${radians(170)}" />
+            <limit lower="${radians(-180)}" upper="${radians(180)}" effort="268.36" velocity="${radians(170)}" />
         </joint>
         <joint name="${prefix}joint_2" type="revolute">
@@ -142,5 +142,5 @@
             <origin xyz="0 0 0" rpy="0 0 0"/>
             <axis xyz="0 1 0" />
-            <limit lower="${radians(-110)}" upper="${radians(110)}" effort="0" velocity="${radians(170)}" />
+            <limit lower="${radians(-110)}" upper="${radians(110)}" effort="268.36" velocity="${radians(170)}" />
         </joint>
         <joint name="${prefix}joint_3" type="revolute">
@@ -149,5 +149,5 @@
             <origin xyz="0 0 0.36" rpy="0 0 0"/>
             <axis xyz="0 0 1" />
-            <limit lower="${radians(-170)}" upper="${radians(170)}" effort="0" velocity="${radians(170)}" />
+            <limit lower="${radians(-170)}" upper="${radians(170)}" effort="122.89" velocity="${radians(170)}" />
         </joint>
         <joint name="${prefix}joint_4" type="revolute">
@@ -156,5 +156,5 @@
             <origin xyz="0 0 0" rpy="0 0 0"/>
             <axis xyz="0 -1 0" />
-            <limit lower="${radians(-135)}" upper="${radians(135)}" effort="0" velocity="${radians(170)}" />
+            <limit lower="${radians(-135)}" upper="${radians(135)}" effort="122.89" velocity="${radians(170)}" />
         </joint>
         <joint name="${prefix}joint_5" type="revolute">
@@ -163,5 +163,5 @@
             <origin xyz="0 0 0.360" rpy="0 0 0"/>
             <axis xyz="0 0 -1" />
-            <limit lower="${radians(-180)}" upper="${radians(180)}" effort="0" velocity="${radians(200)}" />
+            <limit lower="${radians(-180)}" upper="${radians(180)}" effort="44.34" velocity="${radians(200)}" />
         </joint>
         <joint name="${prefix}joint_6" type="revolute">
@@ -170,5 +170,5 @@
             <origin xyz="0 0 0" rpy="0 0 0"/>
             <axis xyz="0 -1 0" />
-            <limit lower="${radians(-110)}" upper="${radians(110)}" effort="0" velocity="${radians(200)}" />
+            <limit lower="${radians(-110)}" upper="${radians(110)}" effort="44.34" velocity="${radians(200)}" />
         </joint>
         <joint name="${prefix}joint_7" type="revolute">
@@ -177,5 +177,5 @@
             <origin xyz="0 0 0.155" rpy="0 0 0"/>
             <axis xyz="0 0 -1" />
-            <limit lower="${radians(-180)}" upper="${radians(180)}" effort="0" velocity="${radians(400)}" />
+            <limit lower="${radians(-180)}" upper="${radians(180)}" effort="39.04" velocity="${radians(400)}" />
         </joint>
         <!-- end of joint list -->

File: motoman_sia20d_support/urdf/sia20d_macro.xacro (robot description, xacro)
@@ -135,5 +135,5 @@
             <origin xyz="0 0 0.41" rpy="0 0 0"/>
             <axis xyz="0 0 1" />
-            <limit lower="${radians(-180)}" upper="${radians(180)}" effort="100" velocity="${radians(130)}" />
+            <limit lower="${radians(-180)}" upper="${radians(180)}" effort="611.76" velocity="${radians(130)}" />
         </joint>
         <joint name="${prefix}joint_2" type="revolute">
@@ -142,5 +142,5 @@
             <origin xyz="0 0 0" rpy="0 0 0"/>
             <axis xyz="0 1 0" />
-            <limit lower="${radians(-110)}" upper="${radians(110)}" effort="100" velocity="${radians(130)}" />
+            <limit lower="${radians(-110)}" upper="${radians(110)}" effort="611.76" velocity="${radians(130)}" />
         </joint>
         <joint name="${prefix}joint_3" type="revolute">
@@ -149,5 +149,5 @@
             <origin xyz="0 0 0.49" rpy="0 0 0"/>
             <axis xyz="0 0 1" />
-            <limit lower="${radians(-170)}" upper="${radians(170)}" effort="100" velocity="${radians(170)}" />
+            <limit lower="${radians(-170)}" upper="${radians(170)}" effort="246.00" velocity="${radians(170)}" />
         </joint>
         <joint name="${prefix}joint_4" type="revolute">
@@ -156,5 +156,5 @@
             <origin xyz="0 0 0" rpy="0 0 0"/>
             <axis xyz="0 -1 0" />
-            <limit lower="${radians(-130)}" upper="${radians(130)}" effort="100" velocity="${radians(170)}" />
+            <limit lower="${radians(-130)}" upper="${radians(130)}" effort="246.00" velocity="${radians(170)}" />
         </joint>
         <joint name="${prefix}joint_5" type="revolute">
@@ -163,5 +163,5 @@
             <origin xyz="0 0 0.420" rpy="0 0 0"/>
             <axis xyz="0 0 -1" />
-            <limit lower="${radians(-180)}" upper="${radians(180)}" effort="100" velocity="${radians(200)}" />
+            <limit lower="${radians(-180)}" upper="${radians(180)}" effort="87.96" velocity="${radians(200)}" />
         </joint>
         <joint name="${prefix}joint_6" type="revolute">
@@ -170,5 +170,5 @@
             <origin xyz="0 0 0" rpy="0 0 0"/>
             <axis xyz="0 -1 0" />
-            <limit lower="${radians(-110)}" upper="${radians(110)}" effort="100" velocity="${radians(200)}" />
+            <limit lower="${radians(-110)}" upper="${radians(110)}" effort="87.96" velocity="${radians(200)}" />
         </joint>
         <joint name="${prefix}joint_7" type="revolute">
@@ -177,5 +177,5 @@
             <origin xyz="0 0 0.18" rpy="0 0 0"/>
             <axis xyz="0 0 -1" />
-            <limit lower="${radians(-180)}" upper="${radians(180)}" effort="100" velocity="${radians(400)}" />
+            <limit lower="${radians(-180)}" upper="${radians(180)}" effort="37.93" velocity="${radians(400)}" />
         </joint>
         <!-- end of joint list -->

File: motoman_sia5d_support/urdf/sia5d_macro.xacro (robot description, xacro)
@@ -36,5 +36,5 @@
     <child link="${prefix}link_1" />
     <axis xyz="0 0 1" />
-    <limit lower="${radians(-180)}" upper="${radians(180)}" effort="0" velocity="${radians(200)}" />
+    <limit lower="${radians(-180)}" upper="${radians(180)}" effort="129.36" velocity="${radians(200)}" />
   </joint>
   <link name="${prefix}link_2">
@@ -57,5 +57,5 @@
     <child link="${prefix}link_2" />
     <axis xyz="0 1 0" />
-    <limit lower="${radians(-110)}" upper="${radians(110)}" effort="0" velocity="${radians(200)}" />
+    <limit lower="${radians(-110)}" upper="${radians(110)}" effort="129.36" velocity="${radians(200)}" />
   </joint>
   <link name="${prefix}link_3">
@@ -78,5 +78,5 @@
     <child link="${prefix}link_3" />
     <axis xyz="0 0 1" />
-    <limit lower="${radians(-170)}" upper="${radians(170)}" effort="0" velocity="${radians(200)}" />
+    <limit lower="${radians(-170)}" upper="${radians(170)}" effort="129.36" velocity="${radians(200)}" />
   </joint>
   <link name="${prefix}link_4">
@@ -99,5 +99,5 @@
     <child link="${prefix}link_4" />
     <axis xyz="0 -1 0" />
-    <limit lower="${radians(-90)}" upper="${radians(115)}" effort="0" velocity="${radians(200)}" />
+    <limit lower="${radians(-90)}" upper="${radians(115)}" effort="85.26" velocity="${radians(200)}" />
   </joint>
   <link name="${prefix}link_5">
@@ -120,5 +120,5 @@
     <child link="${prefix}link_5" />
     <axis xyz="-1 0 0" />
-    <limit lower="${radians(-180)}" upper="${radians(180)}" effort="0" velocity="${radians(200)}" />
+    <limit lower="${radians(-180)}" upper="${radians(180)}" effort="77.08" velocity="${radians(200)}" />
   </joint>
   <link name="${prefix}link_6">
@@ -141,5 +141,5 @@
     <child link="${prefix}link_6" />
     <axis xyz="0 -1 0" />
-    <limit lower="${radians(-110)}" upper="${radians(110)}" effort="0" velocity="${radians(230)}" />
+    <limit lower="${radians(-110)}" upper="${radians(110)}" effort="38.44" velocity="${radians(230)}" />
   </joint>
   <link name="${prefix}link_7">
@@ -162,5 +162,5 @@
     <child link="${prefix}link_7" />
     <axis xyz="-1 0 0" />
-    <limit lower="${radians(-180)}" upper="${radians(180)}" effort="0" velocity="${radians(350)}" />
+    <limit lower="${radians(-180)}" upper="${radians(180)}" effort="72.52" velocity="${radians(350)}" />
   </joint>
   <!-- end of joint list -->
