Commit message: Various changes

File: motoman_gp250_support/urdf/gp250_macro.xacro (robot description, xacro)
@@ -102,5 +102,5 @@
       <origin xyz="0 0 0.650" rpy="0 0 0" />
       <axis xyz="0 0 1" />
-      <limit lower="${radians(-180)}" upper="${radians(180)}" effort="9316.2" velocity="${radians(100)}"/>
+      <limit lower="${radians(-180)}" upper="${radians(180)}" effort="9806.54" velocity="${radians(100)}"/>
     </joint>
     <joint name="${prefix}joint_2" type="revolute">
@@ -109,5 +109,5 @@
       <origin xyz="0.285 0 0" rpy="0 0 0" />
       <axis xyz="0 1 0" />
-      <limit lower="${radians(-60)}" upper="${radians(76)}" effort="10591.1" velocity="${radians(90)}"/>
+      <limit lower="${radians(-60)}" upper="${radians(76)}" effort="11804.75" velocity="${radians(90)}"/>
     </joint>
     <joint name="${prefix}joint_3" type="revolute">
@@ -116,5 +116,5 @@
       <origin xyz="0 0 1.150" rpy="0 0 0" />
       <axis xyz="0 -1 0" />
-      <limit lower="${radians(-77.8)}" upper="${radians(197)}" effort="9929.2" velocity="${radians(97)}"/>
+      <limit lower="${radians(-77.8)}" upper="${radians(197)}" effort="10811.83" velocity="${radians(97)}"/>
     </joint>
     <joint name="${prefix}joint_4" type="revolute">
@@ -123,5 +123,5 @@
       <origin xyz="1.285 0 0.250" rpy="0 0 0" />
       <axis xyz="-1 0 0" />
-      <limit lower="${radians(-360)}" upper="${radians(360)}" effort="2758.0" velocity="${radians(120)}"/>
+      <limit lower="${radians(-360)}" upper="${radians(360)}" effort="2911.32" velocity="${radians(120)}"/>
     </joint>
     <joint name="${prefix}joint_5" type="revolute">

File: motoman_hc10_support/urdf/hc10_macro.xacro (robot description, xacro)
@@ -123,5 +123,5 @@
       <origin xyz="0 0 -0.500" rpy="0 0 0" />
       <axis xyz="0 0 1" />
-      <limit lower="${radians(-180)}" upper="${radians(180)}" effort="39.20" velocity="${radians(180)}"/>
+      <limit lower="${radians(-180)}" upper="${radians(180)}" effort="31.36" velocity="${radians(180)}"/>
     </joint>
     <joint name="${prefix}joint_5" type="revolute">

File: motoman_hc10_support/urdf/hc10dt_macro.xacro (robot description, xacro)
@@ -123,5 +123,5 @@
       <origin xyz="0 0 -0.500" rpy="0 0 0" />
       <axis xyz="0 0 1" />
-      <limit lower="${radians(-180)}" upper="${radians(180)}" effort="39.20" velocity="${radians(180)}"/>
+      <limit lower="${radians(-180)}" upper="${radians(180)}" effort="31.36" velocity="${radians(180)}"/>
     </joint>
     <joint name="${prefix}joint_5" type="revolute">

File: motoman_hc20_support/urdf/hc20dt_macro.xacro (robot description, xacro)
@@ -7,5 +7,5 @@
       <visual>
         <geometry>
-          <mesh filename="package://motoman_hc20_support/meshes/hc20/visual/base_link.dae"/>
+          <mesh filename="package://motoman_hc20_support/meshes/hc20dt/visual/base_link.dae"/>
         </geometry>
         <xacro:material_yaskawa_white/>
@@ -13,5 +13,5 @@
       <collision>
         <geometry>
-          <mesh filename="package://motoman_hc20_support/meshes/hc20/collision/base_link.stl"/>
+          <mesh filename="package://motoman_hc20_support/meshes/hc20dt/collision/base_link.stl"/>
         </geometry>
       </collision>
@@ -20,5 +20,5 @@
       <visual>
         <geometry>
-          <mesh filename="package://motoman_hc20_support/meshes/hc20/visual/link_1.dae"/>
+          <mesh filename="package://motoman_hc20_support/meshes/hc20dt/visual/link_1.dae"/>
         </geometry>
         <xacro:material_yaskawa_white/>
@@ -26,5 +26,5 @@
       <collision>
         <geometry>
-          <mesh filename="package://motoman_hc20_support/meshes/hc20/collision/link_1.stl"/>
+          <mesh filename="package://motoman_hc20_support/meshes/hc20dt/collision/link_1.stl"/>
         </geometry>
       </collision>
@@ -33,5 +33,5 @@
       <visual>
         <geometry>
-          <mesh filename="package://motoman_hc20_support/meshes/hc20/visual/link_2.dae"/>
+          <mesh filename="package://motoman_hc20_support/meshes/hc20dt/visual/link_2.dae"/>
         </geometry>
         <xacro:material_yaskawa_white/>
@@ -39,5 +39,5 @@
       <collision>
         <geometry>
-          <mesh filename="package://motoman_hc20_support/meshes/hc20/collision/link_2.stl"/>
+          <mesh filename="package://motoman_hc20_support/meshes/hc20dt/collision/link_2.stl"/>
         </geometry>
       </collision>
@@ -46,5 +46,5 @@
       <visual>
         <geometry>
-          <mesh filename="package://motoman_hc20_support/meshes/hc20/visual/link_3.dae"/>
+          <mesh filename="package://motoman_hc20_support/meshes/hc20dt/visual/link_3.dae"/>
         </geometry>
         <xacro:material_yaskawa_white/>
@@ -52,5 +52,5 @@
       <collision>
         <geometry>
-          <mesh filename="package://motoman_hc20_support/meshes/hc20/collision/link_3.stl"/>
+          <mesh filename="package://motoman_hc20_support/meshes/hc20dt/collision/link_3.stl"/>
         </geometry>
       </collision>
@@ -59,5 +59,5 @@
       <visual>
         <geometry>
-          <mesh filename="package://motoman_hc20_support/meshes/hc20/visual/link_4.dae"/>
+          <mesh filename="package://motoman_hc20_support/meshes/hc20dt/visual/link_4.dae"/>
         </geometry>
         <xacro:material_yaskawa_white/>
@@ -65,5 +65,5 @@
       <collision>
         <geometry>
-          <mesh filename="package://motoman_hc20_support/meshes/hc20/collision/link_4.stl"/>
+          <mesh filename="package://motoman_hc20_support/meshes/hc20dt/collision/link_4.stl"/>
         </geometry>
       </collision>
@@ -72,5 +72,5 @@
       <visual>
         <geometry>
-          <mesh filename="package://motoman_hc20_support/meshes/hc20/visual/link_5.dae"/>
+          <mesh filename="package://motoman_hc20_support/meshes/hc20dt/visual/link_5.dae"/>
         </geometry>
         <xacro:material_yaskawa_white/>
@@ -78,5 +78,5 @@
       <collision>
         <geometry>
-          <mesh filename="package://motoman_hc20_support/meshes/hc20/collision/link_5.stl"/>
+          <mesh filename="package://motoman_hc20_support/meshes/hc20dt/collision/link_5.stl"/>
         </geometry>
       </collision>
@@ -85,5 +85,5 @@
       <visual>
         <geometry>
-          <mesh filename="package://motoman_hc20_support/meshes/hc20/visual/link_6.dae"/>
+          <mesh filename="package://motoman_hc20_support/meshes/hc20dt/visual/link_6.dae"/>
         </geometry>
         <xacro:material_yaskawa_white/>
@@ -91,5 +91,5 @@
       <collision>
         <geometry>
-          <mesh filename="package://motoman_hc20_support/meshes/hc20/collision/link_6.stl"/>
+          <mesh filename="package://motoman_hc20_support/meshes/hc20dt/collision/link_6.stl"/>
         </geometry>
       </collision>

File: motoman_hc20_support/urdf/hc20dtp_macro.xacro (robot description, xacro)
@@ -7,5 +7,5 @@
       <visual>
         <geometry>
-          <mesh filename="package://motoman_hc20_support/meshes/hc20/visual/base_link.dae"/>
+          <mesh filename="package://motoman_hc20_support/meshes/hc20dt/visual/base_link.dae"/>
         </geometry>
         <xacro:material_yaskawa_white/>
@@ -13,5 +13,5 @@
       <collision>
         <geometry>
-          <mesh filename="package://motoman_hc20_support/meshes/hc20/collision/base_link.stl"/>
+          <mesh filename="package://motoman_hc20_support/meshes/hc20dt/collision/base_link.stl"/>
         </geometry>
       </collision>
@@ -20,5 +20,5 @@
       <visual>
         <geometry>
-          <mesh filename="package://motoman_hc20_support/meshes/hc20/visual/link_1.dae"/>
+          <mesh filename="package://motoman_hc20_support/meshes/hc20dt/visual/link_1.dae"/>
         </geometry>
         <xacro:material_yaskawa_white/>
@@ -26,5 +26,5 @@
       <collision>
         <geometry>
-          <mesh filename="package://motoman_hc20_support/meshes/hc20/collision/link_1.stl"/>
+          <mesh filename="package://motoman_hc20_support/meshes/hc20dt/collision/link_1.stl"/>
         </geometry>
       </collision>
@@ -33,5 +33,5 @@
       <visual>
         <geometry>
-          <mesh filename="package://motoman_hc20_support/meshes/hc20/visual/link_2.dae"/>
+          <mesh filename="package://motoman_hc20_support/meshes/hc20dt/visual/link_2.dae"/>
         </geometry>
         <xacro:material_yaskawa_white/>
@@ -39,5 +39,5 @@
       <collision>
         <geometry>
-          <mesh filename="package://motoman_hc20_support/meshes/hc20/collision/link_2.stl"/>
+          <mesh filename="package://motoman_hc20_support/meshes/hc20dt/collision/link_2.stl"/>
         </geometry>
       </collision>
@@ -46,5 +46,5 @@
       <visual>
         <geometry>
-          <mesh filename="package://motoman_hc20_support/meshes/hc20/visual/link_3.dae"/>
+          <mesh filename="package://motoman_hc20_support/meshes/hc20dt/visual/link_3.dae"/>
         </geometry>
         <xacro:material_yaskawa_white/>
@@ -52,5 +52,5 @@
       <collision>
         <geometry>
-          <mesh filename="package://motoman_hc20_support/meshes/hc20/collision/link_3.stl"/>
+          <mesh filename="package://motoman_hc20_support/meshes/hc20dt/collision/link_3.stl"/>
         </geometry>
       </collision>
@@ -59,5 +59,5 @@
       <visual>
         <geometry>
-          <mesh filename="package://motoman_hc20_support/meshes/hc20/visual/link_4.dae"/>
+          <mesh filename="package://motoman_hc20_support/meshes/hc20dt/visual/link_4.dae"/>
         </geometry>
         <xacro:material_yaskawa_white/>
@@ -65,5 +65,5 @@
       <collision>
         <geometry>
-          <mesh filename="package://motoman_hc20_support/meshes/hc20/collision/link_4.stl"/>
+          <mesh filename="package://motoman_hc20_support/meshes/hc20dt/collision/link_4.stl"/>
         </geometry>
       </collision>

File: motoman_hc20_support/urdf/hc30pl_macro.xacro (robot description, xacro)
@@ -7,5 +7,5 @@
       <visual>
         <geometry>
-          <mesh filename="package://motoman_hc20_support/meshes/hc20/visual/base_link.dae"/>
+          <mesh filename="package://motoman_hc20_support/meshes/hc20dt/visual/base_link.dae"/>
         </geometry>
         <xacro:material_yaskawa_white/>
@@ -13,5 +13,5 @@
       <collision>
         <geometry>
-          <mesh filename="package://motoman_hc20_support/meshes/hc20/collision/base_link.stl"/>
+          <mesh filename="package://motoman_hc20_support/meshes/hc20dt/collision/base_link.stl"/>
         </geometry>
       </collision>
@@ -20,5 +20,5 @@
       <visual>
         <geometry>
-          <mesh filename="package://motoman_hc20_support/meshes/hc20/visual/link_1.dae"/>
+          <mesh filename="package://motoman_hc20_support/meshes/hc20dt/visual/link_1.dae"/>
         </geometry>
         <xacro:material_yaskawa_white/>
@@ -26,5 +26,5 @@
       <collision>
         <geometry>
-          <mesh filename="package://motoman_hc20_support/meshes/hc20/collision/link_1.stl"/>
+          <mesh filename="package://motoman_hc20_support/meshes/hc20dt/collision/link_1.stl"/>
         </geometry>
       </collision>
@@ -33,5 +33,5 @@
       <visual>
         <geometry>
-          <mesh filename="package://motoman_hc20_support/meshes/hc20/visual/link_2.dae"/>
+          <mesh filename="package://motoman_hc20_support/meshes/hc20dt/visual/link_2.dae"/>
         </geometry>
         <xacro:material_yaskawa_white/>
@@ -39,5 +39,5 @@
       <collision>
         <geometry>
-          <mesh filename="package://motoman_hc20_support/meshes/hc20/collision/link_2.stl"/>
+          <mesh filename="package://motoman_hc20_support/meshes/hc20dt/collision/link_2.stl"/>
         </geometry>
       </collision>
@@ -46,5 +46,5 @@
       <visual>
         <geometry>
-          <mesh filename="package://motoman_hc20_support/meshes/hc20/visual/link_3.dae"/>
+          <mesh filename="package://motoman_hc20_support/meshes/hc20dt/visual/link_3.dae"/>
         </geometry>
         <xacro:material_yaskawa_white/>
@@ -52,5 +52,5 @@
       <collision>
         <geometry>
-          <mesh filename="package://motoman_hc20_support/meshes/hc20/collision/link_3.stl"/>
+          <mesh filename="package://motoman_hc20_support/meshes/hc20dt/collision/link_3.stl"/>
         </geometry>
       </collision>
@@ -59,5 +59,5 @@
       <visual>
         <geometry>
-          <mesh filename="package://motoman_hc20_support/meshes/hc20/visual/link_4.dae"/>
+          <mesh filename="package://motoman_hc20_support/meshes/hc20dt/visual/link_4.dae"/>
         </geometry>
         <xacro:material_yaskawa_white/>
@@ -65,5 +65,5 @@
       <collision>
         <geometry>
-          <mesh filename="package://motoman_hc20_support/meshes/hc20/collision/link_4.stl"/>
+          <mesh filename="package://motoman_hc20_support/meshes/hc20dt/collision/link_4.stl"/>
         </geometry>
       </collision>

File: motoman_mh12_support/urdf/mh12_macro.xacro (robot description, xacro)
@@ -116,5 +116,5 @@
         <origin xyz="0 0 0.614" rpy="0 0 0" />
         <axis xyz="0 -1 0" />
-        <limit lower="${radians(-175)}" upper="${radians(240)}" effort="257.25" velocity="${radians(220)}"/>
+        <limit lower="${radians(-85)}" upper="${radians(150)}" effort="257.25" velocity="${radians(220)}"/>
     </joint>
     <joint name="${prefix}joint_4" type="revolute">

File: motoman_motomini_support/urdf/motomini_macro.xacro (robot description, xacro)
@@ -102,5 +102,5 @@
     <origin xyz="0 0 0.103" rpy="0 0 0" />
     <axis xyz="0 0 1" />
-    <limit lower="${radians(-170)}" upper="${radians(170)}" effort="0.12" velocity="${radians(315)}"/>
+    <limit lower="${radians(-170)}" upper="${radians(170)}" effort="18.40" velocity="${radians(315)}"/>
   </joint>
   <joint name="${prefix}joint_2" type="revolute">
@@ -109,5 +109,5 @@
     <origin xyz="0.020 0 0" rpy="0 0 0" />
     <axis xyz="0 1 0" />
-    <limit lower="${radians(-85)}" upper="${radians(90)}" effort="0.12" velocity="${radians(315)}"/>
+    <limit lower="${radians(-85)}" upper="${radians(90)}" effort="18.40" velocity="${radians(315)}"/>
   </joint>
   <joint name="${prefix}joint_3" type="revolute">
@@ -116,5 +116,5 @@
     <origin xyz="0 0 0.165" rpy="0 0 0" />
     <axis xyz="0 -1 0" />
-    <limit lower="${radians(-50)}" upper="${radians(90)}" effort="0.12" velocity="${radians(420)}"/>
+    <limit lower="${radians(-50)}" upper="${radians(90)}" effort="6.64" velocity="${radians(420)}"/>
   </joint>
   <joint name="${prefix}joint_4" type="revolute">
@@ -123,5 +123,5 @@
     <origin xyz="0.165 0 0" rpy="0 0 0" />
     <axis xyz="-1 0 0" />
-    <limit lower="${radians(-140)}" upper="${radians(140)}" effort="0.07" velocity="${radians(600)}"/>
+    <limit lower="${radians(-140)}" upper="${radians(140)}" effort="1.80" velocity="${radians(600)}"/>
   </joint>
   <joint name="${prefix}joint_5" type="revolute">
@@ -130,5 +130,5 @@
     <origin xyz="0 0 0" rpy="0 0 0" />
     <axis xyz="0 -1 0" />
-    <limit lower="${radians(-30)}" upper="${radians(210)}" effort="0.07" velocity="${radians(600)}"/>
+    <limit lower="${radians(-30)}" upper="${radians(210)}" effort="1.80" velocity="${radians(600)}"/>
   </joint>
   <joint name="${prefix}joint_6" type="revolute">
@@ -137,5 +137,5 @@
     <origin xyz="0 0 0" rpy="0 0 0" />
     <axis xyz="0 0 1" />
-    <limit lower="${radians(-360)}" upper="${radians(360)}" effort="0.07" velocity="${radians(600)}"/>
+    <limit lower="${radians(-360)}" upper="${radians(360)}" effort="1.44" velocity="${radians(600)}"/>
   </joint>
     <!-- end of joint list -->

File: motoman_ms210_support/urdf/ms210_macro.xacro (robot description, xacro)
@@ -130,5 +130,5 @@
     <origin xyz="0 0 1.150" rpy="0 0 0" />
     <axis xyz="0 -1 0" />
-    <limit lower="${radians(-147)}" upper="${radians(90)}" effort="9806.65" velocity="${radians(115)}" />
+    <limit lower="${radians(-86)}" upper="${radians(90)}" effort="9806.65" velocity="${radians(115)}" />
   </joint>
   <joint name="${prefix}joint_4" type="revolute">

File: motoman_sda10f_support/urdf/csda10f_arm_macro.xacro (robot description, xacro)
@@ -111,5 +111,5 @@
       <origin xyz="0.100 ${reflect*0.265} 0" rpy="${radians(90)} 0 ${(reflect-1)*radians(90)}"/>
       <axis xyz="0 0 ${-reflect}" />
-      <limit lower="${radians(-170)}" upper="${radians(170)}" effort="268.36" velocity="${radians(170)}" />
+      <limit lower="${radians(-180)}" upper="${radians(180)}" effort="268.36" velocity="${radians(170)}" />
     </joint>
     <joint name="${prefix}joint_2" type="revolute">

File: motoman_sia10d_support/urdf/sia10d_macro.xacro (robot description, xacro)
@@ -141,5 +141,5 @@
             <origin xyz="0 0 0.36" rpy="0 0 0"/>
             <axis xyz="0 0 1" />
-            <limit lower="${radians(-180)}" upper="${radians(180)}" effort="100" velocity="${radians(170)}" />
+            <limit lower="${radians(-180)}" upper="${radians(180)}" effort="268.36" velocity="${radians(170)}" />
         </joint>
         <joint name="${prefix}joint_2" type="revolute">
@@ -148,5 +148,5 @@
             <origin xyz="0 0 0" rpy="0 0 0"/>
             <axis xyz="0 1 0" />
-            <limit lower="${radians(-110)}" upper="${radians(110)}" effort="100" velocity="${radians(170)}" />
+            <limit lower="${radians(-110)}" upper="${radians(110)}" effort="268.36" velocity="${radians(170)}" />
         </joint>
         <joint name="${prefix}joint_3" type="revolute">
@@ -155,5 +155,5 @@
             <origin xyz="0 0 0.36" rpy="0 0 0"/>
             <axis xyz="0 0 1" />
-            <limit lower="${radians(-170)}" upper="${radians(170)}" effort="100" velocity="${radians(170)}" />
+            <limit lower="${radians(-170)}" upper="${radians(170)}" effort="122.89" velocity="${radians(170)}" />
         </joint>
         <joint name="${prefix}joint_4" type="revolute">
@@ -162,5 +162,5 @@
             <origin xyz="0 0 0" rpy="0 0 0"/>
             <axis xyz="0 -1 0" />
-            <limit lower="${radians(-135)}" upper="${radians(135)}" effort="100" velocity="${radians(170)}" />
+            <limit lower="${radians(-135)}" upper="${radians(135)}" effort="122.89" velocity="${radians(170)}" />
         </joint>
         <joint name="${prefix}joint_5" type="revolute">
@@ -169,5 +169,5 @@
             <origin xyz="0 0 0.360" rpy="0 0 0"/>
             <axis xyz="0 0 -1" />
-            <limit lower="${radians(-180)}" upper="${radians(180)}" effort="100" velocity="${radians(200)}" />
+            <limit lower="${radians(-180)}" upper="${radians(180)}" effort="44.34" velocity="${radians(200)}" />
         </joint>
         <joint name="${prefix}joint_6" type="revolute">
@@ -176,5 +176,5 @@
             <origin xyz="0 0 0" rpy="0 0 0"/>
             <axis xyz="0 -1 0" />
-            <limit lower="${radians(-110)}" upper="${radians(110)}" effort="100" velocity="${radians(200)}" />
+            <limit lower="${radians(-110)}" upper="${radians(110)}" effort="44.34" velocity="${radians(200)}" />
         </joint>
         <joint name="${prefix}joint_7" type="revolute">
@@ -183,5 +183,5 @@
             <origin xyz="0 0 0.155" rpy="0 0 0"/>
             <axis xyz="0 0 -1" />
-            <limit lower="${radians(-180)}" upper="${radians(180)}" effort="100" velocity="${radians(400)}" />
+            <limit lower="${radians(-180)}" upper="${radians(180)}" effort="39.04" velocity="${radians(400)}" />
         </joint>
         <!-- end of joint list -->

File: motoman_sia10f_support/urdf/sia10f_macro.xacro (robot description, xacro)
@@ -135,5 +135,5 @@
             <origin xyz="0 0 0.36" rpy="0 0 0"/>
             <axis xyz="0 0 1" />
-            <limit lower="${radians(-180)}" upper="${radians(180)}" effort="0" velocity="${radians(170)}" />
+            <limit lower="${radians(-180)}" upper="${radians(180)}" effort="268.36" velocity="${radians(170)}" />
         </joint>
         <joint name="${prefix}joint_2" type="revolute">
@@ -142,5 +142,5 @@
             <origin xyz="0 0 0" rpy="0 0 0"/>
             <axis xyz="0 1 0" />
-            <limit lower="${radians(-110)}" upper="${radians(110)}" effort="0" velocity="${radians(170)}" />
+            <limit lower="${radians(-110)}" upper="${radians(110)}" effort="268.36" velocity="${radians(170)}" />
         </joint>
         <joint name="${prefix}joint_3" type="revolute">
@@ -149,5 +149,5 @@
             <origin xyz="0 0 0.36" rpy="0 0 0"/>
             <axis xyz="0 0 1" />
-            <limit lower="${radians(-170)}" upper="${radians(170)}" effort="0" velocity="${radians(170)}" />
+            <limit lower="${radians(-170)}" upper="${radians(170)}" effort="122.89" velocity="${radians(170)}" />
         </joint>
         <joint name="${prefix}joint_4" type="revolute">
@@ -156,5 +156,5 @@
             <origin xyz="0 0 0" rpy="0 0 0"/>
             <axis xyz="0 -1 0" />
-            <limit lower="${radians(-135)}" upper="${radians(135)}" effort="0" velocity="${radians(170)}" />
+            <limit lower="${radians(-135)}" upper="${radians(135)}" effort="122.89" velocity="${radians(170)}" />
         </joint>
         <joint name="${prefix}joint_5" type="revolute">
@@ -163,5 +163,5 @@
             <origin xyz="0 0 0.360" rpy="0 0 0"/>
             <axis xyz="0 0 -1" />
-            <limit lower="${radians(-180)}" upper="${radians(180)}" effort="0" velocity="${radians(200)}" />
+            <limit lower="${radians(-180)}" upper="${radians(180)}" effort="44.34" velocity="${radians(200)}" />
         </joint>
         <joint name="${prefix}joint_6" type="revolute">
@@ -170,5 +170,5 @@
             <origin xyz="0 0 0" rpy="0 0 0"/>
             <axis xyz="0 -1 0" />
-            <limit lower="${radians(-110)}" upper="${radians(110)}" effort="0" velocity="${radians(200)}" />
+            <limit lower="${radians(-110)}" upper="${radians(110)}" effort="44.34" velocity="${radians(200)}" />
         </joint>
         <joint name="${prefix}joint_7" type="revolute">
@@ -177,5 +177,5 @@
             <origin xyz="0 0 0.155" rpy="0 0 0"/>
             <axis xyz="0 0 -1" />
-            <limit lower="${radians(-180)}" upper="${radians(180)}" effort="0" velocity="${radians(400)}" />
+            <limit lower="${radians(-180)}" upper="${radians(180)}" effort="39.04" velocity="${radians(400)}" />
         </joint>
         <!-- end of joint list -->
