Commit message: Various changes

File: motoman_sia20d_support/urdf/sia20d_macro.xacro (robot description, xacro)
@@ -135,5 +135,5 @@
             <origin xyz="0 0 0.41" rpy="0 0 0"/>
             <axis xyz="0 0 1" />
-            <limit lower="${radians(-180)}" upper="${radians(180)}" effort="100" velocity="${radians(130)}" />
+            <limit lower="${radians(-180)}" upper="${radians(180)}" effort="611.76" velocity="${radians(130)}" />
         </joint>
         <joint name="${prefix}joint_2" type="revolute">
@@ -142,5 +142,5 @@
             <origin xyz="0 0 0" rpy="0 0 0"/>
             <axis xyz="0 1 0" />
-            <limit lower="${radians(-110)}" upper="${radians(110)}" effort="100" velocity="${radians(130)}" />
+            <limit lower="${radians(-110)}" upper="${radians(110)}" effort="611.76" velocity="${radians(130)}" />
         </joint>
         <joint name="${prefix}joint_3" type="revolute">
@@ -149,5 +149,5 @@
             <origin xyz="0 0 0.49" rpy="0 0 0"/>
             <axis xyz="0 0 1" />
-            <limit lower="${radians(-170)}" upper="${radians(170)}" effort="100" velocity="${radians(170)}" />
+            <limit lower="${radians(-170)}" upper="${radians(170)}" effort="246.00" velocity="${radians(170)}" />
         </joint>
         <joint name="${prefix}joint_4" type="revolute">
@@ -156,5 +156,5 @@
             <origin xyz="0 0 0" rpy="0 0 0"/>
             <axis xyz="0 -1 0" />
-            <limit lower="${radians(-130)}" upper="${radians(130)}" effort="100" velocity="${radians(170)}" />
+            <limit lower="${radians(-130)}" upper="${radians(130)}" effort="246.00" velocity="${radians(170)}" />
         </joint>
         <joint name="${prefix}joint_5" type="revolute">
@@ -163,5 +163,5 @@
             <origin xyz="0 0 0.420" rpy="0 0 0"/>
             <axis xyz="0 0 -1" />
-            <limit lower="${radians(-180)}" upper="${radians(180)}" effort="100" velocity="${radians(200)}" />
+            <limit lower="${radians(-180)}" upper="${radians(180)}" effort="87.96" velocity="${radians(200)}" />
         </joint>
         <joint name="${prefix}joint_6" type="revolute">
@@ -170,5 +170,5 @@
             <origin xyz="0 0 0" rpy="0 0 0"/>
             <axis xyz="0 -1 0" />
-            <limit lower="${radians(-110)}" upper="${radians(110)}" effort="100" velocity="${radians(200)}" />
+            <limit lower="${radians(-110)}" upper="${radians(110)}" effort="87.96" velocity="${radians(200)}" />
         </joint>
         <joint name="${prefix}joint_7" type="revolute">
@@ -177,5 +177,5 @@
             <origin xyz="0 0 0.18" rpy="0 0 0"/>
             <axis xyz="0 0 -1" />
-            <limit lower="${radians(-180)}" upper="${radians(180)}" effort="100" velocity="${radians(400)}" />
+            <limit lower="${radians(-180)}" upper="${radians(180)}" effort="37.93" velocity="${radians(400)}" />
         </joint>
         <!-- end of joint list -->

File: motoman_sia5d_support/urdf/sia5d_macro.xacro (robot description, xacro)
@@ -36,5 +36,5 @@
     <child link="${prefix}link_1" />
     <axis xyz="0 0 1" />
-    <limit lower="${radians(-180)}" upper="${radians(180)}" effort="0" velocity="${radians(200)}" />
+    <limit lower="${radians(-180)}" upper="${radians(180)}" effort="129.36" velocity="${radians(200)}" />
   </joint>
   <link name="${prefix}link_2">
@@ -57,5 +57,5 @@
     <child link="${prefix}link_2" />
     <axis xyz="0 1 0" />
-    <limit lower="${radians(-110)}" upper="${radians(110)}" effort="0" velocity="${radians(200)}" />
+    <limit lower="${radians(-110)}" upper="${radians(110)}" effort="129.36" velocity="${radians(200)}" />
   </joint>
   <link name="${prefix}link_3">
@@ -78,5 +78,5 @@
     <child link="${prefix}link_3" />
     <axis xyz="0 0 1" />
-    <limit lower="${radians(-170)}" upper="${radians(170)}" effort="0" velocity="${radians(200)}" />
+    <limit lower="${radians(-170)}" upper="${radians(170)}" effort="129.36" velocity="${radians(200)}" />
   </joint>
   <link name="${prefix}link_4">
@@ -99,5 +99,5 @@
     <child link="${prefix}link_4" />
     <axis xyz="0 -1 0" />
-    <limit lower="${radians(-90)}" upper="${radians(115)}" effort="0" velocity="${radians(200)}" />
+    <limit lower="${radians(-90)}" upper="${radians(115)}" effort="85.26" velocity="${radians(200)}" />
   </joint>
   <link name="${prefix}link_5">
@@ -120,5 +120,5 @@
     <child link="${prefix}link_5" />
     <axis xyz="-1 0 0" />
-    <limit lower="${radians(-90)}" upper="${radians(90)}" effort="0" velocity="${radians(200)}" />
+    <limit lower="${radians(-180)}" upper="${radians(180)}" effort="77.08" velocity="${radians(200)}" />
   </joint>
   <link name="${prefix}link_6">
@@ -141,5 +141,5 @@
     <child link="${prefix}link_6" />
     <axis xyz="0 -1 0" />
-    <limit lower="${radians(-110)}" upper="${radians(110)}" effort="0" velocity="${radians(230)}" />
+    <limit lower="${radians(-110)}" upper="${radians(110)}" effort="38.44" velocity="${radians(230)}" />
   </joint>
   <link name="${prefix}link_7">
@@ -162,5 +162,5 @@
     <child link="${prefix}link_7" />
     <axis xyz="-1 0 0" />
-    <limit lower="${radians(-90)}" upper="${radians(90)}" effort="0" velocity="${radians(350)}" />
+    <limit lower="${radians(-180)}" upper="${radians(180)}" effort="72.52" velocity="${radians(350)}" />
   </joint>
   <!-- end of joint list -->

File: motoman_up50n_support/urdf/up50n_35_macro.xacro (robot description, xacro)
@@ -116,5 +116,5 @@
         <origin xyz="0 0 1.150" rpy="0 0 0" />
         <axis xyz="0 -1 0" />
-        <limit lower="${radians(-80)}" upper="${radians(206)}" effort="2021" velocity="${radians(140)}"/>
+        <limit lower="${radians(-77)}" upper="${radians(206)}" effort="2021" velocity="${radians(140)}"/>
     </joint>
     <joint name="${prefix}joint_4" type="revolute">

Commit message: fix gp250 effort values

File: motoman_gp250_support/urdf/gp250_macro.xacro (robot description, xacro)
@@ -102,5 +102,5 @@
       <origin xyz="0 0 0.650" rpy="0 0 0" />
       <axis xyz="0 0 1" />
-      <limit lower="${radians(-180)}" upper="${radians(180)}" effort="9316.2" velocity="${radians(100)}"/>
+      <limit lower="${radians(-180)}" upper="${radians(180)}" effort="9806.54" velocity="${radians(100)}"/>
     </joint>
     <joint name="${prefix}joint_2" type="revolute">
@@ -109,5 +109,5 @@
       <origin xyz="0.285 0 0" rpy="0 0 0" />
       <axis xyz="0 1 0" />
-      <limit lower="${radians(-60)}" upper="${radians(76)}" effort="10591.1" velocity="${radians(90)}"/>
+      <limit lower="${radians(-60)}" upper="${radians(76)}" effort="11804.75" velocity="${radians(90)}"/>
     </joint>
     <joint name="${prefix}joint_3" type="revolute">
@@ -116,5 +116,5 @@
       <origin xyz="0 0 1.150" rpy="0 0 0" />
       <axis xyz="0 -1 0" />
-      <limit lower="${radians(-77.8)}" upper="${radians(197)}" effort="9929.2" velocity="${radians(97)}"/>
+      <limit lower="${radians(-77.8)}" upper="${radians(197)}" effort="10811.83" velocity="${radians(97)}"/>
     </joint>
     <joint name="${prefix}joint_4" type="revolute">
@@ -123,5 +123,5 @@
       <origin xyz="1.285 0 0.250" rpy="0 0 0" />
       <axis xyz="-1 0 0" />
-      <limit lower="${radians(-360)}" upper="${radians(360)}" effort="2758.0" velocity="${radians(120)}"/>
+      <limit lower="${radians(-360)}" upper="${radians(360)}" effort="2911.32" velocity="${radians(120)}"/>
     </joint>
     <joint name="${prefix}joint_5" type="revolute">
