Commit message: Move `xacro` end tag in `sia5d`

File: motoman_sia5d_support/urdf/sia5d_macro.xacro (robot description, xacro)
@@ -173,5 +173,4 @@
       <child link="${prefix}base"/>
     </joint>
-    </xacro:macro>
   <!-- ROS-Industrial 'flange' frame: attachment point for EEF models -->
   <link name="${prefix}flange"/>
@@ -188,3 +187,4 @@
     <child link="${prefix}tool0"/>
   </joint>
+  </xacro:macro>
 </robot>

Commit message: remove reference to 'deg' xacro variable

File: motoman_sia5d_support/urdf/sia5d_macro.xacro (robot description, xacro)
@@ -1,5 +1,4 @@
 <?xml version="1.0" ?>
 <robot xmlns:xacro="http://ros.org/wiki/xacro">
-    <xacro:property name="deg" value="0.017453293" /> <!--degrees to radians-->
     <xacro:macro name="motoman_sia5d" params="prefix">
   <xacro:include filename="$(find motoman_resources)/urdf/common_materials.xacro"/>

Commit message: Fix sia5d joint limits

File: motoman_sia5d_support/urdf/sia5d_macro.xacro (robot description, xacro)
@@ -120,5 +120,5 @@
     <child link="${prefix}link_5" />
     <axis xyz="-1 0 0" />
-    <limit lower="${radians(-90)}" upper="${radians(90)}" effort="0" velocity="${radians(200)}" />
+    <limit lower="${radians(-180)}" upper="${radians(180)}" effort="0" velocity="${radians(200)}" />
   </joint>
   <link name="${prefix}link_6">
@@ -162,5 +162,5 @@
     <child link="${prefix}link_7" />
     <axis xyz="-1 0 0" />
-    <limit lower="${radians(-90)}" upper="${radians(90)}" effort="0" velocity="${radians(350)}" />
+    <limit lower="${radians(-180)}" upper="${radians(180)}" effort="0" velocity="${radians(350)}" />
   </joint>
   <!-- end of joint list -->
