Commit message: Fix mpx1950 joint_4 offset

File: motoman_mpx1950_support/urdf/mpx1950_macro.xacro (robot description, xacro)
@@ -121,5 +121,5 @@
       <parent link="${prefix}link_3"/>
       <child link="${prefix}link_4"/>
-      <origin xyz="0.725 0 0.015" rpy="0 0 0" />
+      <origin xyz="0.725 0 0" rpy="0 0 0" />
       <axis xyz="-1 0 0" />
       <limit lower="${radians(-200)}" upper="${radians(200)}" effort="215.6" velocity="${radians(360)}"/>
